File: kicad/VL6180ToF_20221107/VL6180ToF_20221107.kicad_sch (KiCad schematic)
At the start: 18 parts

Commit message: kicad main+kick-drib
Parts:
- J1: renamed from ?; footprint Connector_PinHeader_1.27mm:PinHeader_1x07_P1.27mm_Vertical -> 0.main.robot:Pin_1x07_P1.27mm_SMD
- gave numbers to parts that had none: 16
Changed lines of the file:
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@@
   (symbol (lib_id "VL6180ToF_20221107-rescue:Q_DUAL_NMOS_S1G1D2S2G2D1-Device") (at 119.38 119.38 90) (mirror x) (unit 1)
     (in_bom yes) (on_board yes)
-    (property "Reference" "" (id 0) (at 119.38 125.7046 90))
+    (property "Reference" "Q1" (id 0) (at 119.38 125.7046 90))
     (property "Value" "SSM6N42FE" (id 1) (at 119.38 128.016 90))
     (property "Footprint" "Package_SON:WSON-6_1.5x1.5mm_P0.5mm" (id 2) (at 119.38 124.46 0)
@@
     (pin "2")
     (pin "6")
+  )
+  (symbol (lib_id "VL6180ToF_20221107-rescue:Q_DUAL_NMOS_S1G1D2S2G2D1-Device") (at 107.95 129.54 90) (mirror x) (unit 2)
+    (in_bom yes) (on_board yes)
+    (property "Reference" "Q1" (id 0) (at 107.95 135.8646 90))
+    (property "Value" "SSM6N42FE" (id 1) (at 107.95 138.176 90))
+    (property "Footprint" "Package_SON:WSON-6_1.5x1.5mm_P0.5mm" (id 2) (at 107.95 134.62 0)
+      (effects (font (size 1.27 1.27)) hide)
+    )
+    (property "Datasheet" "~" (id 3) (at 107.95 134.62 0)
+      (effects (font (size 1.27 1.27)) hide)
+    )
     (pin "3")
     (pin "4")
     (pin "5")
   )
-  (symbol (lib_id "VL6180ToF_20221107-rescue:Q_DUAL_NMOS_S1G1D2S2G2D1-Device") (at 107.95 129.54 90) (mirror x) (unit 2)
-    (in_bom yes) (on_board yes)
-    (property "Reference" "" (id 0) (at 107.95 135.8646 90))
-    (property "Value" "SSM6N42FE" (id 1) (at 107.95 138.176 90))
-    (property "Footprint" "Package_SON:WSON-6_1.5x1.5mm_P0.5mm" (id 2) (at 107.95 134.62 0)
-      (effects (font (size 1.27 1.27)) hide)
-    )
-    (property "Datasheet" "~" (id 3) (at 107.95 134.62 0)
-      (effects (font (size 1.27 1.27)) hide)
-    )
-    (pin "1")
-    (pin "2")
-    (pin "6")
+  (symbol (lib_id "Regulator_Linear:TPS73125DBV") (at 217.17 52.07 0) (unit 1)
+    (in_bom yes) (on_board yes)
+    (property "Reference" "U1" (id 0) (at 217.17 42.7482 0))
+    (property "Value" "Si91841" (id 1) (at 217.17 45.0596 0))
+    (property "Footprint" "Package_TO_SOT_SMD:SOT-23-5" (id 2) (at 217.17 43.815 0)
+      (effects (font (size 1.27 1.27) italic) hide)
+    )
+    (property "Datasheet" "http://www.ti.com/lit/ds/symlink/tps731.pdf" (id 3) (at 217.17 53.34 0)
+      (effects (font (size 1.27 1.27)) hide)
+    )
+    (pin "1")
+    (pin "2")
     (pin "3")
     (pin "4")
     (pin "5")
   )
-  (symbol (lib_id "Regulator_Linear:TPS73125DBV") (at 217.17 52.07 0) (unit 1)
-    (in_bom yes) (on_board yes)
-    (property "Reference" "" (id 0) (at 217.17 42.7482 0))
-    (property "Value" "Si91841" (id 1) (at 217.17 45.0596 0))
-    (property "Footprint" "Package_TO_SOT_SMD:SOT-23-5" (id 2) (at 217.17 43.815 0)
-      (effects (font (size 1.27 1.27) italic) hide)
-    )
-    (property "Datasheet" "http://www.ti.com/lit/ds/symlink/tps731.pdf" (id 3) (at 217.17 53.34 0)
-      (effects (font (size 1.27 1.27)) hide)
-    )
-    (pin "1")
-    (pin "2")
-    (pin "3")
-    (pin "4")
-    (pin "5")
-  )
   (symbol (lib_id "VL6180ToF_20221107-rescue:VL6180XV0NR_1-2022-11-07_14-13-02") (at 154.94 111.76 0) (unit 1)
     (in_bom yes) (on_board yes)
-    (property "Reference" "" (id 0) (at 182.88 101.9302 0)
+    (property "Reference" "U2" (id 0) (at 182.88 101.9302 0)
       (effects (font (size 1.524 1.524)))
     )
@@
   (symbol (lib_id "Device:R") (at 148.59 92.71 0) (unit 1)
     (in_bom yes) (on_board yes)
-    (property "Reference" "" (id 0) (at 150.368 91.5416 0)
+    (property "Reference" "R6" (id 0) (at 150.368 91.5416 0)
       (effects (font (size 1.27 1.27)) (justify left))
     )
@@
   (symbol (lib_id "Device:R") (at 142.24 92.71 0) (unit 1)
     (in_bom yes) (on_board yes)
-    (property "Reference" "" (id 0) (at 144.018 91.5416 0)
+    (property "Reference" "R5" (id 0) (at 144.018 91.5416 0)
       (effects (font (size 1.27 1.27)) (justify left))
     )
@@
   (symbol (lib_id "Device:R") (at 133.35 92.71 0) (unit 1)
     (in_bom yes) (on_board yes)
-    (property "Reference" "" (id 0) (at 135.128 91.5416 0)
+    (property "Reference" "R4" (id 0) (at 135.128 91.5416 0)
       (effects (font (size 1.27 1.27)) (justify left))
     )
@@
   (symbol (lib_id "Device:R") (at 127 92.71 0) (unit 1)
     (in_bom yes) (on_board yes)
-    (property "Reference" "" (id 0) (at 128.778 91.5416 0)
+    (property "Reference" "R3" (id 0) (at 128.778 91.5416 0)
       (effects (font (size 1.27 1.27)) (justify left))
     )
@@
   (symbol (lib_id "Device:C") (at 220.98 104.14 0) (unit 1)
     (in_bom yes) (on_board yes)
-    (property "Reference" "" (id 0) (at 223.901 102.9716 0)
+    (property "Reference" "C5" (id 0) (at 223.901 102.9716 0)
       (effects (font (size 1.27 1.27)) (justify left))
     )
@@
   (symbol (lib_id "Device:C") (at 232.41 58.42 0) (unit 1)
     (in_bom yes) (on_board yes)
-    (property "Reference" "" (id 0) (at 235.331 57.2516 0)
+    (property "Reference" "C3" (id 0) (at 235.331 57.2516 0)
       (effects (font (size 1.27 1.27)) (justify left))
     )
@@
   (symbol (lib_id "Device:C") (at 242.57 58.42 0) (unit 1)
     (in_bom yes) (on_board yes)
-    (property "Reference" "" (id 0) (at 245.491 57.2516 0)
+    (property "Reference" "C4" (id 0) (at 245.491 57.2516 0)
       (effects (font (size 1.27 1.27)) (justify left))
     )
@@
   (symbol (lib_id "Device:C") (at 199.39 54.61 0) (unit 1)
     (in_bom yes) (on_board yes)
-    (property "Reference" "" (id 0) (at 202.311 53.4416 0)
+    (property "Reference" "C2" (id 0) (at 202.311 53.4416 0)
       (effects (font (size 1.27 1.27)) (justify left))
     )
@@
   (symbol (lib_id "Device:C") (at 191.77 54.61 0) (unit 1)
     (in_bom yes) (on_board yes)
-    (property "Reference" "" (id 0) (at 194.691 53.4416 0)
+    (property "Reference" "C1" (id 0) (at 194.691 53.4416 0)
       (effects (font (size 1.27 1.27)) (justify left))
     )
@@
   (symbol (lib_id "Connector_Generic:Conn_01x07") (at 54.61 99.06 0) (mirror y) (unit 1)
     (in_bom yes) (on_board yes)
-    (property "Reference" "" (id 0) (at 56.6928 85.9282 0))
+    (property "Reference" "J1" (id 0) (at 56.6928 85.9282 0))
     (property "Value" "Conn_01x07" (id 1) (at 56.6928 88.2396 0))
-    (property "Footprint" "Connector_PinHeader_1.27mm:PinHeader_1x07_P1.27mm_Vertical" (id 2) (at 54.61 99.06 0)
+    (property "Footprint" "0.main.robot:Pin_1x07_P1.27mm_SMD" (id 2) (at 54.61 99.06 0)
       (effects (font (size 1.27 1.27)) hide)
     )
@@
   (symbol (lib_id "Device:R") (at 90.17 104.14 270) (unit 1)
     (in_bom yes) (on_board yes)
-    (property "Reference" "" (id 0) (at 90.17 98.8822 90))
+    (property "Reference" "R7" (id 0) (at 90.17 98.8822 90))
     (property "Value" "1k" (id 1) (at 90.17 101.1936 90))
     (property "Footprint" "Resistor_SMD:R_0603_1608Metric" (id 2) (at 90.17 102.362 90)
@@
   (symbol (lib_id "Device:R") (at 99.06 106.68 270) (unit 1)
     (in_bom yes) (on_board yes)
-    (property "Reference" "" (id 0) (at 99.06 101.4222 90))
+    (property "Reference" "R8" (id 0) (at 99.06 101.4222 90))
     (property "Value" "1k" (id 1) (at 99.06 103.7336 90))
     (property "Footprint" "Resistor_SMD:R_0603_1608Metric" (id 2) (at 99.06 104.902 90)
@@
   (symbol (lib_id "Device:R") (at 76.2 91.44 0) (unit 1)
     (in_bom yes) (on_board yes)
-    (property "Reference" "" (id 0) (at 77.978 90.2716 0)
+    (property "Reference" "R1" (id 0) (at 77.978 90.2716 0)
       (effects (font (size 1.27 1.27)) (justify left))
     )
@@
   (symbol (lib_id "Device:R") (at 82.55 91.44 0) (unit 1)
     (in_bom yes) (on_board yes)
-    (property "Reference" "" (id 0) (at 84.328 90.2716 0)
+    (property "Reference" "R2" (id 0) (at 84.328 90.2716 0)
       (effects (font (size 1.27 1.27)) (justify left))
     )
@@
     )
     (path "/00000000-0000-0000-0000-0000636d6c25"
-      (reference "J1") (unit 1) (value "Conn_01x07") (footprint "Connector_PinHeader_1.27mm:PinHeader_1x07_P1.27mm_Vertical")
+      (reference "J1") (unit 1) (value "Conn_01x07") (footprint "0.main.robot:Pin_1x07_P1.27mm_SMD")
     )
     (path "/00000000-0000-0000-0000-0000636b6ecf"
