File: kicad/main/rp2040.kicad_sch (KiCad schematic)
At the start: 24 parts, among them SW9 BOOTSEL, U14 RP2040, U15 W25Q128JVS, Y3 12Mhz

Commit message: fix: main
Parts:
- renumbered C19 to C16, C20 to C17, C21 to C18, C22 to C19, C23 to C20, C24 to C21, C25 to C22, C26 to C23, C27 to C24, C28 to C25, C29 to C26, C30 to C27, R55 to R49, R56 to R50, R57 to R51, R58 to R52, R59 to R53, R60 to R54, R61 to R55, R62 to R56, SW9 to SW8, U14 to U11, U15 to U12

Commit message: fix: main xbee
Parts:
- renumbered C16 to C14, C17 to C15, C18 to C16, C19 to C17, C20 to C18, C21 to C19, C22 to C20, C23 to C21, C24 to C22, C25 to C23, C26 to C24, C27 to C25, R49 to R42, R50 to R43, R51 to R44, R52 to R45, R53 to R46, R54 to R47, R55 to R48, R56 to R49, SW8 to SW7, U12 to U10, U11 to U9

Commit message: no message
Parts:
- removed R42: 1k, Resistor_SMD:R_0603_1608Metric_Pad0.98x0.95mm_HandSolder, symbol Device:R
- Y3: footprint Crystal:Resonator_SMD_Murata_CSTxExxV-3Pin_3.0x1.1mm_HandSoldering -> Crystal:Resonator-3Pin_W6.0mm_H3.0mm
- renumbered C14 to C12, C15 to C13, C16 to C14, C17 to C15, C18 to C16, C19 to C17, C20 to C18, C21 to C19, C22 to C20, C23 to C21, C24 to C22, C25 to C23, R43 to R30, R44 to R31, R45 to R32, R46 to R33, R47 to R34, R48 to R35, R49 to R36, SW7 to SW3, U9 to U7, U10 to U8
