File: kicad/main/main.kicad_sch (KiCad schematic)
At the start: 98 parts, among them J1 Power IN1, J10 Drib, J11 Serial3/OpenMV, J12 LED, J13 I2C/IMU, J14 I2C_0, J15 SW1, J16 I2C_1, J17 I2C_2, J18 5V OUT, J19 Power IN, J2 AUX1, J20 LINE, J3 USB2.0_C_v3, J4 SW1, J5 MAIN, J6 I2C_3, J7 Kicker, J8 MD1, J9 MD2, Q1 AO3400A, Q2 AO3401A, SW1 GOAL, SW2 START, SW4 Reset, SW5 AUX1, SW6 IMU SET, SW7 Reset, U1 XBEE-S2C, U2 AZ1117CH-3.3, U3 AZ1117CH-3.3, U4 PCF8574PW, U5 AE-BNO055, U6 74HC32, U7 74HC04, U8 OKL-T_3-W12N-C

Commit message: fix: main
Parts:
- removed J19: Power IN, Connector_JST:JST_XH_B2B-XH-A_1x02_P2.50mm_Vertical, symbol Connector_Generic:Conn_01x02
- removed J5: MAIN, Connector_JST:JST_XH_B2B-XH-A_1x02_P2.50mm_Vertical, symbol Connector_Generic:Conn_01x02
- added J14, J15: drib-kick, 0.main.robot:JSTB4B-ZR, symbol Connector_Generic:Conn_01x04
- J5: renamed from J1; value Power IN1 -> Power IN
- renumbered C2 to C1, C7 to C10, C1 to C2, C4 to C3, C5 to C4, C6 to C5, C8 to C6, C9 to C7, C10 to C8, C3 to C9, D2 to D1, D9 to D10, D10 to D11, D4 to D2, D5 to D4, D6 to D5, D11 to D6, D13 to D7, D7 to D8, D8 to D9, J3 to J1, J14 to J11, J15 to J12, J16 to J13, J17 to J16, J18 to J17, J20 to J18, J4 to J19, J13 to J20, J6 to J3, J11 to J4, J12 to J6, R5 to R1, R17 to R10, R22 to R11, R26 to R12, R27 to R13, R29 to R14, R31 to R15, R32 to R16, R33 to R17, R28 to R18, R34 to R19, R4 to R2, R30 to R20, R36 to R21, R35 to R22, R37 to R23, R38 to R24, R1 to R25, R2 to R26, R9 to R27, R11 to R28, R14 to R29, R7 to R3, R16 to R30, R18 to R31, R19 to R32, R20 to R33, R21 to R34, R23 to R35, R24 to R36, R25 to R37, R6 to R4, R8 to R5, R10 to R6, R12 to R7, R13 to R8, R15 to R9, SW4 to SW1, SW7 to SW2, SW1 to SW3, SW2 to SW4, U6 to U4, U7 to U5, U8 to U6, U4 to U7, U5 to U8
Connections:
- net +15V: now also J10.1 (Pin_1), J5.2 (Pin_2), J7.1 (Pin_1), J8.2 (Pin_2), J9.2 (Pin_2), R23.1, U6.2 (VIN), J15.1 (Pin_1), J15.3 (Pin_3)
- net GND: now also J10.2 (Pin_2), J5.1 (Pin_1), J7.2 (Pin_2), J8.1 (Pin_1), J9.1 (Pin_1), J14.2 (Pin_2), J14.4 (Pin_4), J15.2 (Pin_2), J15.4 (Pin_4)
- new net rp2040/GPIO12/16: J14.3 (Pin_3)
- new net rp2040/GPIO13/17: J14.1 (Pin_1)
Other:
- removed sheet Sheet61861092
- moved on the sheet: C1, C10, C4, C6, C7, C8, C9, D1, D10, D11, D12, D2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

Commit message: fix: main xbee
Parts:
- removed C2, C3: 10u, Capacitor_SMD:C_0603_1608Metric_Pad1.08x0.95mm_HandSolder, symbol Device:C
- removed D3: RSSI, LED_SMD:LED_0603_1608Metric_Pad1.05x0.95mm_HandSolder, symbol Device:LED
- removed D4: RX, LED_SMD:LED_0603_1608Metric_Pad1.05x0.95mm_HandSolder, symbol Device:LED
- removed D5: TX, LED_SMD:LED_0603_1608Metric_Pad1.05x0.95mm_HandSolder, symbol Device:LED
- removed R2, R6, R9: 470, Resistor_SMD:R_0603_1608Metric_Pad0.98x0.95mm_HandSolder, symbol Device:R
- removed R4, R5, R7, R8: 10k, Resistor_SMD:R_0603_1608Metric_Pad0.98x0.95mm_HandSolder, symbol Device:R
- removed SW1: Reset, 0.main.robot:THAU13-AB-R, symbol Switch:SW_Push
- removed U1: XBEE-S2C, 0.main.robot:XBEE-S2C, symbol 0.main.robot.library:XBEE-S2C
- removed U2: AZ1117CH-3.3, Package_TO_SOT_SMD:SOT-223-3_TabPin2, symbol Regulator_Linear:AZ1084-2.85
- added J4: XBee, 0.main.robot:JSTB4B-ZR, symbol Connector_Generic:Conn_01x04
- R18: renamed from R25; footprint Resistor_SMD:R_0603_1608Metric_Pad1.05x0.95mm_HandSolder -> Resistor_SMD:R_0603_1608Metric_Pad0.98x0.95mm_HandSolder
- R19: renamed from R26; footprint Resistor_SMD:R_0603_1608Metric_Pad1.05x0.95mm_HandSolder -> Resistor_SMD:R_0603_1608Metric_Pad0.98x0.95mm_HandSolder
- R20: renamed from R27; footprint Resistor_SMD:R_0603_1608Metric_Pad1.05x0.95mm_HandSolder -> Resistor_SMD:R_0603_1608Metric_Pad0.98x0.95mm_HandSolder
- R21: renamed from R28; footprint Resistor_SMD:R_0603_1608Metric_Pad1.05x0.95mm_HandSolder -> Resistor_SMD:R_0603_1608Metric_Pad0.98x0.95mm_HandSolder
- R22: renamed from R29; footprint Resistor_SMD:R_0603_1608Metric_Pad1.05x0.95mm_HandSolder -> Resistor_SMD:R_0603_1608Metric_Pad0.98x0.95mm_HandSolder
- R23: renamed from R30; footprint Resistor_SMD:R_0603_1608Metric_Pad1.05x0.95mm_HandSolder -> Resistor_SMD:R_0603_1608Metric_Pad0.98x0.95mm_HandSolder
- R24: renamed from R31; footprint Resistor_SMD:R_0603_1608Metric_Pad1.05x0.95mm_HandSolder -> Resistor_SMD:R_0603_1608Metric_Pad0.98x0.95mm_HandSolder
- R25: renamed from R32; footprint Resistor_SMD:R_0603_1608Metric_Pad1.05x0.95mm_HandSolder -> Resistor_SMD:R_0603_1608Metric_Pad0.98x0.95mm_HandSolder
- R26: renamed from R33; footprint Resistor_SMD:R_0603_1608Metric_Pad1.05x0.95mm_HandSolder -> Resistor_SMD:R_0603_1608Metric_Pad0.98x0.95mm_HandSolder
- R27: renamed from R34; footprint Resistor_SMD:R_0603_1608Metric_Pad1.05x0.95mm_HandSolder -> Resistor_SMD:R_0603_1608Metric_Pad0.98x0.95mm_HandSolder
- renumbered C4 to C2, C5 to C3, C6 to C4, C7 to C5, C8 to C6, C9 to C7, C10 to C8, D6 to D3, D7 to D4, D8 to D5, D9 to D6, D10 to D7, D11 to D8, D12 to D9, J9 to J10, J10 to J11, J11 to J12, J12 to J13, J13 to J14, J14 to J15, J15 to J16, J16 to J17, J17 to J18, J18 to J19, J19 to J20, J20 to J21, J4 to J5, J5 to J6, J6 to J7, J7 to J8, J8 to J9, R17 to R10, R18 to R11, R19 to R12, R20 to R13, R21 to R14, R22 to R15, R23 to R16, R24 to R17, R3 to R2, R35 to R28, R36 to R29, R10 to R3, R37 to R30, R11 to R4, R12 to R5, R13 to R6, R14 to R7, R15 to R8, R16 to R9, SW2 to SW1, SW3 to SW2, SW4 to SW3, SW5 to SW4, SW6 to SW5, U3 to U1, U4 to U2, U5 to U3, U6 to U4, U7 to U5, U8 to U6
Connections:
- net +5V: now also J4.2 (Pin_2)
- net GND: now also J4.4 (Pin_4)
- net rp2040/GPIO00/01: now also J4.1 (Pin_1)
- net rp2040/GPIO01/02: now also J4.3 (Pin_3)
- no-connect marks 23 -> 9

Commit message: ToF
Parts:
- removed J12: I2C_0, 0.main.robot:JSTB4B-ZR, symbol Connector_Generic:Conn_01x04
- removed J21: I2C/IMU, 0.main.robot:JSTB4B-ZR, symbol Connector_Generic:Conn_01x04
- renumbered J13 to J12, J14 to J13, J15 to J14, J16 to J15, J17 to J16, J18 to J17, J19 to J18, J20 to J19
Connections:
- net rp2040/GPIO04/06 is gone; now on net SDA_IMU: J13.3 (Pin_3), J16.3 (Pin_3), R6.2
- net rp2040/GPIO05/07 is gone; now on net SCL_IMU: J13.1 (Pin_1), J16.1 (Pin_1), R5.2
- net +3V3: now also C7.1, C8.1, R20.1, R21.1, R22.1, R23.1, R28.1, R29.1, R30.1, U5.5 (VCC), U6.1 (VIN)
- net SDA_IMU: now reaches R28.2, U5.4 (SDA), U6.3 (SDA)
- net SCL_IMU: now reaches R29.2, U5.2 (SCL), U6.4 (SCL)
Other:
- moved on the sheet: C1, C2, D1, D2, J1, R1, R2, U1

Commit message: no message
Parts:
- removed C7: 0.1u, Capacitor_SMD:C_0603_1608Metric_Pad1.08x0.95mm_HandSolder, symbol Device:C
- removed C8: 10u, Capacitor_SMD:C_0603_1608Metric_Pad1.08x0.95mm_HandSolder, symbol Device:C
- removed D5: LED1_R, 0.main.robot:LED_SMLE13WBC8W1, symbol Device:LED
- removed D6: LED2_G, 0.main.robot:LED_SMLE13WBC8W1, symbol Device:LED
- removed D7: LED3_Y, 0.main.robot:LED_SMLE13WBC8W1, symbol Device:LED
- removed D8: LED4_B, 0.main.robot:LED_SMLE13WBC8W1, symbol Device:LED
- removed D9: LED(OSWT1608), 0.main.robot:LED_SMLE13WBC8W1, symbol Device:LED
- removed J11: Drib, Connector_JST:JST_XH_B2B-XH-A_1x02_P2.50mm_Vertical, symbol Connector_Generic:Conn_01x02
- removed J12: SW1, 0.main.robot:JSTB6B-ZR, symbol Connector_Generic:Conn_01x06
- removed J19: SW1, 0.main.robot:JSTS6B-ZRLFSN, symbol Connector_Generic:Conn_01x06
- removed J7: LED, 0.main.robot:JSTB6B-ZR, symbol Connector_Generic:Conn_01x06
- removed J8: Kicker, Connector_JST:JST_XH_B2B-XH-A_1x02_P2.50mm_Vertical, symbol Connector_Generic:Conn_01x02
- removed JP1, JP2: SolderJumper_2_Open, Jumper:SolderJumper-2_P1.3mm_Open_RoundedPad1.0x1.5mm, symbol Jumper:SolderJumper_2_Open
- removed JP3: Jumper_2_Bridged, Connector_PinHeader_1.27mm:PinHeader_1x02_P1.27mm_Vertical, symbol Jumper:Jumper_2_Bridged
- removed R18, R19, R30: 470, Resistor_SMD:R_0603_1608Metric_Pad0.98x0.95mm_HandSolder, symbol Device:R
- removed R20, R21, R22, R23, R28, R29: 47k, Resistor_SMD:R_0603_1608Metric_Pad0.98x0.95mm_HandSolder, symbol Device:R
- removed R24, R25, R26, R27: 120, Resistor_SMD:R_0603_1608Metric_Pad0.98x0.95mm_HandSolder, symbol Device:R
- removed SW2: GOAL, 0.main.robot:MFS101D-14-Z, symbol Switch:SW_SPDT
- removed SW3: START, 0.main.robot:SW_NKK_B-12CCPRM, symbol 0.main.robot.library:SW_NKK_B-12CCPRM
- removed SW4: AUX1, Button_Switch_THT:SW_DIP_SPSTx02_Slide_9.78x7.26mm_W7.62mm_P2.54mm, symbol Switch:SW_DIP_x02
- removed SW5: IMU SET, 0.main.robot:TVAF06-A020B-R, symbol Switch:SW_Push
- removed U5: PCF8574PW, Package_SO:TSSOP-20_4.4x6.5mm_P0.65mm, symbol PCF8574:PCF8574PW
- removed U6: AE-BNO055, 0.main.robot:AE-BNO055, symbol 0.main.robot.library:AE-BNO055
- added R3: 10k, Resistor_SMD:R_0603_1608Metric_Pad0.98x0.95mm_HandSolder, symbol Device:R
- J12: renamed from J14; footprint 0.main.robot:JSTB4B-ZR -> Connector_PinHeader_2.54mm:PinHeader_1x04_P2.54mm_Vertical
- J13: renamed from J15; footprint 0.main.robot:JSTB4B-ZR -> Connector_PinHeader_2.54mm:PinHeader_1x04_P2.54mm_Vertical
- J4: footprint 0.main.robot:JSTB4B-ZR -> Connector_PinHeader_2.54mm:PinHeader_1x04_P2.54mm_Vertical
- R6: renamed from R5; value 10k -> 47k
- R7: renamed from R6; value 10k -> 47k
- renumbered J13 to J11, J16 to J14, J17 to J15, J18 to J16, J6 to J5, J5 to J6, J9 to J8, J10 to J9, R8 to R10, R13 to R11, R9 to R12, R10 to R13, R12 to R14, R14 to R16, R16 to R17, R17 to R18, R3 to R4, R4 to R5, R7 to R8, R11 to R9
Connections:
- net rp2040/RUN(RES)/30 is gone; now on net RESET: C3.2, D3.2 (A), R5.2, SW1.1
- net +5V: now also J15.1 (Pin_1), R15.1, U4.4 (VOUT), U4.5 (SENSE)
- net GND: now also C5.2, J15.2 (Pin_2)
- net rp2040/GPIO01/02: now also R3.1; no longer J4.3 (Pin_3)
- new net: J4.3 (Pin_3), R3.2
- no-connect marks 9 -> 5
Other:
- added sheet switch_section (switch_section.kicad_sch)
- note added: "IMU SET"
- note removed: "(Switch section)"
- note removed: "3V3"
- note removed: "SW-G"
- company: (none) -> A.Saeki
- title: (none) -> main board
- moved on the sheet: C4, C5, C6, D4, J15, J5, J8, J9, R11, R15, R17, R18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

Commit message: update: m1n-vison
Parts:
- added U?: RP2040_Stamp, symbol rp2040_stamp:RP2040_Stamp
Changed lines of the file:
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@@
     (pin "2")
+  )
+  (symbol (lib_id "rp2040_stamp:RP2040_Stamp") (at 3.81 129.54 0) (unit 1)
+    (in_bom yes) (on_board yes) (fields_autoplaced)
+    (property "Reference" "U?" (id 0) (at 3.81 84.0572 0))
+    (property "Value" "RP2040_Stamp" (id 1) (at 3.81 86.5941 0))
+    (property "Footprint" "" (id 2) (at 36.83 146.05 0)
+      (effects (font (size 1.27 1.27)) hide)
+    )
+    (property "Datasheet" "" (id 3) (at 36.83 146.05 0)
+      (effects (font (size 1.27 1.27)) hide)
+    )
+    (pin "1")
+    (pin "10")
+    (pin "11")
+    (pin "12")
+    (pin "13")
+    (pin "14")
+    (pin "15")
+    (pin "16")
+    (pin "17")
+    (pin "18")
+    (pin "19")
+    (pin "2")
+    (pin "20")
+    (pin "21")
+    (pin "22")
+    (pin "23")
+    (pin "24")
+    (pin "25")
+    (pin "26")
+    (pin "27")
+    (pin "28")
+    (pin "29")
+    (pin "3")
+    (pin "30")
+    (pin "31")
+    (pin "32")
+    (pin "33")
+    (pin "34")
+    (pin "35")
+    (pin "36")
+    (pin "37")
+    (pin "38")
+    (pin "39")
+    (pin "4")
+    (pin "40")
+    (pin "5")
+    (pin "6")
+    (pin "7")
+    (pin "8")
+    (pin "9")
   )
   (symbol (lib_id "rp2040-dev-board:USB2.0_C_v3") (at 31.75 46.99 0) (unit 1)
@@
       (reference "U11") (unit 1) (value "AE-BNO055") (footprint "0.main.robot:AE-BNO055")
     )
+    (path "/d4aa3900-20f8-4ef8-911c-365a69dad616"
+      (reference "U?") (unit 1) (value "RP2040_Stamp") (footprint "")
+    )
     (path "/17adc8c0-c792-4780-aab1-71d31733c779/5444318d-d53e-4fcf-93ea-ecb1f602de35"

Commit message: no message
Parts:
- added D? (x2): D_Schottky, Diode_SMD:D_0805_2012Metric_Pad1.15x1.40mm_HandSolder, symbol Device:D_Schottky
- added J?: USB_C_Receptacle_USB2.0, Connector_USB:USB_C_Receptacle_XKB_U262-16XN-4BVC11, symbol Connector:USB_C_Receptacle_USB2.0
- added R? (x2): 5.1K, Resistor_SMD:R_0603_1608Metric, symbol Device:R_Small
- added SW? (x2): BTN_UP, Button_Switch_SMD:Panasonic_EVQPUJ_EVQPUA, symbol Switch:SW_SPST
Connections:
- net rp2040/GPIO00/01 is gone; now on an unnamed net: J4.1 (Pin_1)
- net rp2040/GPIO01/02 is gone; now on an unnamed net: R3.1
- net rp2040/GPIO08/11 is gone; now on an unnamed net: J6.1 (Pin_1)
- net rp2040/GPIO09/12 is gone; now on an unnamed net: R4.1
- net rp2040/GPIO12/16 is gone; now on an unnamed net: J12.3 (Pin_3)
- net rp2040/GPIO13/17 is gone; now on an unnamed net: J12.1 (Pin_1)
- net rp2040/GPIO14/19 is gone; now on an unnamed net: J2.1 (Pin_1)
- net rp2040/GPIO15/20 is gone; now on an unnamed net: J2.3 (Pin_3)
- net rp2040/GPIO16/21 is gone; now on an unnamed net: U2.4, U3.2
- net rp2040/GPIO17/22 is gone; now on an unnamed net: U2.9, U3.4
- net rp2040/GPIO18/24 is gone; now on an unnamed net: U2.5, U3.6
- net rp2040/GPIO19/25 is gone; now on an unnamed net: U2.10, U3.8
- net rp2040/GPIO20/26 is gone; now on an unnamed net: U2.1, U3.10
- net rp2040/GPIO21/27 is gone; now on an unnamed net: Q1.1 (G)
- net rp2040/GPIO28/34 is gone; now on an unnamed net: U2.3
- net +3V3: now also U?.34 (3.3V)
- net +5V: now also D?.2 (A)
- net GND: now also U?.31 (GND), J?.A1 (GND), J?.A12 (GND), J?.B1 (GND), J?.B12 (GND), J?.S1 (SHIELD), R?.2, R?.2, SW?.1 (A), SW?.1 (A)
- net RESET: now also U?.39 (~{RESET}), SW?.2 (B)
- net SCL_IMU: now also U?.6 (GPIO5)
- net SDA_IMU: now also U?.5 (GPIO4)
- net SW1_1: now also U?.4 (GPIO3)
- net SW1_2: now also U?.7 (GPIO6)
- net SW1_4: now also U?.3 (GPIO2)
- net SW1_5: now also U?.8 (GPIO7)
- net Sheet63625160/SCL_1: now also U?.12 (GPIO11)
- net Sheet63625160/SDA_1: now also U?.11 (GPIO10)
- net Vbatt: now also U?.28 (GPIO27)
- net at U?.33 (5V): now also D?.1 (K), D?.1 (K)
- net USB_D-: now reaches U?.35 (USB_D-)
- net USB_D-: now also J?.A7 (D-), J?.B7 (D-)
- net USB_D+: now reaches U?.36 (USB_D+)
- net USB_D+: now also J?.A6 (D+), J?.B6 (D+)
- net BOOTSET: now reaches U?.40 (BOOTSEL)
- net BOOTSET: now also SW?.2 (B)
- new net: J?.A5 (CC1), R?.1
- new net: J?.B5 (CC2), R?.1
- new net VBUS: D?.2 (A), J?.A4 (VBUS), J?.A9 (VBUS), J?.B4 (VBUS), J?.B9 (VBUS)
- no-connect marks 5 -> 7
Other:
- removed sheet rp2040
- moved on the sheet: J2, J4, J6, R3, R4, U?

Commit message: no message
Parts:
- removed C1, C2: 10uF, Capacitor_SMD:C_0603_1608Metric_Pad1.08x0.95mm_HandSolder, symbol Device:C
- removed D1, D2: SX34F, Diode_SMD:D_SMA, symbol Device:D
- removed J1: USB2.0_C_v3, rp2040:USB-C-12-Pin-MidMount-ali-v4, symbol rp2040-dev-board:USB2.0_C_v3
- removed R1, R2: 5.1kR, Resistor_SMD:R_0603_1608Metric_Pad0.98x0.95mm_HandSolder, symbol Device:R
- removed U1: AZ1117CH-3.3, Package_TO_SOT_SMD:SOT-223-3_TabPin2, symbol Regulator_Linear:AZ1117-3.3
- added D?: LED, 0.main.robot:LED_SMLE13WBC8W1, symbol Device:LED
- added J?: to cam, 0.main.robot:JSTB6B-ZR, symbol Connector_Generic:Conn_01x06
- added R?: 470, Resistor_SMD:R_0603_1608Metric_Pad0.98x0.95mm_HandSolder, symbol Device:R
- J7: renamed from J4; value XBee -> Serial0/XBee
- J8: renamed from J6; value Serial3/OpenMV -> Serial1/IMU
- gave numbers to parts that had none: 8
- renumbered D3 to D5, D4 to D6, J11 to J10, J12 to J11, J13 to J12, J14 to J13, J15 to J14, J16 to J15, J3 to J2, J5 to J4, J8 to J5, J9 to J6, J2 to J9, R8 to R10, R9 to R11, R10 to R12, R11 to R13, R12 to R14, R13 to R15, R14 to R16, R15 to R17, R16 to R18, R17 to R19, R18 to R20, R3 to R5, R5 to R6, R4 to R7, R6 to R8, R7 to R9, SW1 to SW3, U2 to U3, U3 to U4, U4 to U5
Connections:
- net +5V: now also J?.2 (Pin_2), J?.4 (Pin_4)
- net GND: now also D?.1 (K), J?.5 (Pin_5), J?.6 (Pin_6)
- net at J7.3 (Pin_3): now also R5.1; no longer R5.2
- net at Q1.1 (G): now also U2.23 (GPIO22); no longer U2.22 (GPIO21)
- net at U2.2 (GPIO1): now also R5.2; no longer R5.1
- net at U2.25 (GPIO24): now also R?.2
- net SCL_IMU renamed SCL_I2C0
- net SCL_I2C0: now also J?.1 (Pin_1)
- net SDA_IMU renamed SDA_I2C0
- net SDA_I2C0: now also J?.3 (Pin_3)
- net MD/SCL_1 renamed SCL_I2C1
- net MD/SDA_1 renamed SDA_I2C1
- new net: D?.2 (A), R?.1
- no-connect marks 7 -> 9
Other:
- sheet Sheet63625160 renamed MD
- moved on the sheet: J3, J4, J5, J6, R3, R4
