File: kicad/main/main.kicad_sch (KiCad schematic)
At the start: 53 parts, among them J1 USB_C_Receptacle_USB2.0, J10 drib-kick, J11 drib-kick, J12 LINE, J2 I2C_2, J21 GND-Test, J3 Power IN, J4 MD1, J5 MD2, J6 Serial0/XBee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

Commit message: fix: 配線後
Parts:
- added R44: 10k, Resistor_SMD:R_0603_1608Metric_Pad0.98x0.95mm_HandSolder, symbol Device:R
Connections:
- net GND: now also J10.2 (Pin_2), J10.4 (Pin_4); no longer J11.2 (Pin_2), J11.4 (Pin_4)
- net at J7.4 (Pin_4): now also R44.2; no longer U1.8 (GPIO7)
- new net: J11.2 (Pin_2), J11.4 (Pin_4), JP1.2 (B)
- new net: R44.1, U1.8 (GPIO7)
Other:
- moved on the sheet: J11, JP1
Changed lines of the file:
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@@
   )
   (bus_alias "USB" (members "D+" "D-"))
-  (bus_alias "I2C_1" (members "SDA" "SCL"))
   (bus_alias "I2C_0" (members "SDA" "SCL"))
+  (bus_alias "I2C_1" (members "SDA" "SCL"))
   (junction (at 273.05 217.17) (diameter 0) (color 0 0 0 0)
   )
@@
   (junction (at 74.93 121.92) (diameter 0) (color 0 0 0 0)
   )
-  (junction (at 280.67 130.81) (diameter 0) (color 0 0 0 0)
+  (junction (at 288.29 130.81) (diameter 0) (color 0 0 0 0)
   )
   (junction (at 257.81 245.11) (diameter 0) (color 0 0 0 0)
@@
   (junction (at 83.82 139.7) (diameter 0) (color 0 0 0 0)
   )
-  (junction (at 283.21 138.43) (diameter 0) (color 0 0 0 0)
+  (junction (at 290.83 138.43) (diameter 0) (color 0 0 0 0)
   )
   (junction (at 246.38 35.56) (diameter 0) (color 0 0 0 0)
@@
     (stroke (width 0) (type default) (color 0 0 0 0))
   )
-  (wire (pts (xy 279.4 138.43) (xy 283.21 138.43))
+  (wire (pts (xy 273.05 138.43) (xy 276.86 138.43))
     (stroke (width 0) (type default) (color 0 0 0 0))
   )
@@
     (stroke (width 0) (type default) (color 0 0 0 0))
   )
-  (wire (pts (xy 284.48 135.89) (xy 280.67 135.89))
+  (wire (pts (xy 292.1 135.89) (xy 288.29 135.89))
     (stroke (width 0) (type default) (color 0 0 0 0))
   )
@@
     (stroke (width 0) (type default) (color 0 0 0 0))
   )
-  (wire (pts (xy 283.21 133.35) (xy 283.21 138.43))
+  (wire (pts (xy 290.83 133.35) (xy 290.83 138.43))
     (stroke (width 0) (type default) (color 0 0 0 0))
   )
@@
     (stroke (width 0) (type solid) (color 0 0 0 0))
   )
-  (wire (pts (xy 281.94 124.46) (xy 271.78 124.46))
+  (wire (pts (xy 257.81 124.46) (xy 281.94 124.46))
     (stroke (width 0) (type default) (color 0 0 0 0))
   )
@@
     (stroke (width 0) (type default) (color 0 0 0 0))
   )
+  (wire (pts (xy 227.33 148.59) (xy 229.87 148.59))
+    (stroke (width 0) (type default) (color 0 0 0 0))
+  )
   (wire (pts (xy 241.3 52.07) (xy 243.84 52.07))
     (stroke (width 0) (type default) (color 0 0 0 0))
@@
     (stroke (width 0) (type default) (color 0 0 0 0))
   )
-  (wire (pts (xy 280.67 130.81) (xy 284.48 130.81))
+  (wire (pts (xy 288.29 130.81) (xy 292.1 130.81))
     (stroke (width 0) (type default) (color 0 0 0 0))
   )
@@
     (stroke (width 0) (type default) (color 0 0 0 0))
   )
-  (wire (pts (xy 175.26 148.59) (xy 229.87 148.59))
+  (wire (pts (xy 175.26 148.59) (xy 219.71 148.59))
     (stroke (width 0) (type default) (color 0 0 0 0))
   )
@@
     (stroke (width 0) (type default) (color 0 0 0 0))
   )
-  (wire (pts (xy 284.48 133.35) (xy 283.21 133.35))
+  (wire (pts (xy 292.1 133.35) (xy 290.83 133.35))
     (stroke (width 0) (type default) (color 0 0 0 0))
   )
@@
     (stroke (width 0) (type default) (color 0 0 0 0))
   )
-  (wire (pts (xy 261.62 124.46) (xy 257.81 124.46))
-    (stroke (width 0) (type default) (color 0 0 0 0))
-  )
   (wire (pts (xy 210.82 63.5) (xy 210.82 90.17))
     (stroke (width 0) (type default) (color 0 0 0 0))
@@
     (stroke (width 0) (type default) (color 0 0 0 0))
   )
+  (wire (pts (xy 287.02 138.43) (xy 290.83 138.43))
+    (stroke (width 0) (type default) (color 0 0 0 0))
+  )
   (wire (pts (xy 276.86 73.66) (xy 276.86 82.55))
     (stroke (width 0) (type default) (color 0 0 0 0))
@@
     (stroke (width 0) (type default) (color 0 0 0 0))
   )
-  (wire (pts (xy 280.67 135.89) (xy 280.67 130.81))
+  (wire (pts (xy 288.29 135.89) (xy 288.29 130.81))
     (stroke (width 0) (type default) (color 0 0 0 0))
   )
@@
     (stroke (width 0) (type default) (color 0 0 0 0))
   )
-  (wire (pts (xy 279.4 130.81) (xy 280.67 130.81))
+  (wire (pts (xy 287.02 130.81) (xy 288.29 130.81))
     (stroke (width 0) (type default) (color 0 0 0 0))
   )
@@
     (stroke (width 0) (type default) (color 0 0 0 0))
   )
-  (wire (pts (xy 283.21 138.43) (xy 284.48 138.43))
+  (wire (pts (xy 290.83 138.43) (xy 292.1 138.43))
     (stroke (width 0) (type default) (color 0 0 0 0))
   )
@@
     (effects (font (size 1.27 1.27) (thickness 0.254) bold italic) (justify left bottom))
   )
-  (text "IMU SET" (at 220.98 148.59 0)
+  (text "IMU SET" (at 231.14 149.86 0)
     (effects (font (size 1.27 1.27) (thickness 0.254) bold italic) (justify left bottom))
   )
@@
     (pin "1")
   )
-  (symbol (lib_id "Connector_Generic:Conn_01x04") (at 289.56 133.35 0) (unit 1)
+  (symbol (lib_id "Connector_Generic:Conn_01x04") (at 297.18 133.35 0) (unit 1)
     (in_bom yes) (on_board yes)
-    (property "Reference" "J11" (id 0) (at 291.592 133.5532 0)
+    (property "Reference" "J11" (id 0) (at 299.212 133.5532 0)
       (effects (font (size 1.27 1.27)) (justify left))
     )
-    (property "Value" "drib-kick" (id 1) (at 291.592 135.8646 0)
+    (property "Value" "drib-kick" (id 1) (at 299.212 135.8646 0)
       (effects (font (size 1.27 1.27)) (justify left))
     )
-    (property "Footprint" "Connector_PinHeader_2.54mm:PinHeader_1x04_P2.54mm_Vertical" (id 2) (at 289.56 133.35 0)
+    (property "Footprint" "Connector_PinHeader_2.54mm:PinHeader_1x04_P2.54mm_Vertical" (id 2) (at 297.18 133.35 0)
       (effects (font (size 1.27 1.27)) hide)
     )
-    (property "Datasheet" "~" (id 3) (at 289.56 133.35 0)
+    (property "Datasheet" "~" (id 3) (at 297.18 133.35 0)
       (effects (font (size 1.27 1.27)) hide)
     )
@@
     (pin "S1")
   )
-  (symbol (lib_id "power:GND") (at 279.4 138.43 270) (unit 1)
+  (symbol (lib_id "power:GND") (at 273.05 138.43 270) (unit 1)
     (in_bom yes) (on_board yes)
-    (property "Reference" "#PWR027" (id 0) (at 273.05 138.43 0)
+    (property "Reference" "#PWR027" (id 0) (at 266.7 138.43 0)
       (effects (font (size 1.27 1.27)) hide)
     )
-    (property "Value" "GND" (id 1) (at 275.0058 138.557 0))
-    (property "Footprint" "" (id 2) (at 279.4 138.43 0)
+    (property "Value" "GND" (id 1) (at 268.6558 138.557 0))
+    (property "Footprint" "" (id 2) (at 273.05 138.43 0)
       (effects (font (size 1.27 1.27)) hide)
     )
-    (property "Datasheet" "" (id 3) (at 279.4 138.43 0)
+    (property "Datasheet" "" (id 3) (at 273.05 138.43 0)
       (effects (font (size 1.27 1.27)) hide)
     )
@@
     (pin "1")
   )
-  (symbol (lib_id "power:+15V") (at 279.4 130.81 90) (unit 1)
+  (symbol (lib_id "power:+15V") (at 287.02 130.81 90) (unit 1)
     (in_bom yes) (on_board yes)
-    (property "Reference" "#PWR026" (id 0) (at 283.21 130.81 0)
+    (property "Reference" "#PWR026" (id 0) (at 290.83 130.81 0)
       (effects (font (size 1.27 1.27)) hide)
     )
-    (property "Value" "+15V" (id 1) (at 275.0058 130.429 0))
-    (property "Footprint" "" (id 2) (at 279.4 130.81 0)
+    (property "Value" "+15V" (id 1) (at 282.6258 130.429 0))
+    (property "Footprint" "" (id 2) (at 287.02 130.81 0)
       (effects (font (size 1.27 1.27)) hide)
     )
-    (property "Datasheet" "" (id 3) (at 279.4 130.81 0)
+    (property "Datasheet" "" (id 3) (at 287.02 130.81 0)
       (effects (font (size 1.27 1.27)) hide)
     )
@@
     (pin "2")
   )
-  (symbol (lib_id "Jumper:Jumper_2_Bridged") (at 266.7 124.46 0) (unit 1)
+  (symbol (lib_id "Jumper:Jumper_2_Bridged") (at 281.94 138.43 0) (unit 1)
     (in_bom yes) (on_board yes) (fields_autoplaced)
-    (property "Reference" "JP1" (id 0) (at 266.7 120.1252 0))
-    (property "Value" "Jumper_2_Bridged" (id 1) (at 266.7 122.6621 0))
-    (property "Footprint" "Jumper:SolderJumper-2_P1.3mm_Bridged2Bar_RoundedPad1.0x1.5mm" (id 2) (at 266.7 124.46 0)
+    (property "Reference" "JP1" (id 0) (at 281.94 134.0952 0))
+    (property "Value" "Jumper_2_Bridged" (id 1) (at 281.94 136.6321 0))
+    (property "Footprint" "Jumper:SolderJumper-2_P1.3mm_Bridged2Bar_RoundedPad1.0x1.5mm" (id 2) (at 281.94 138.43 0)
       (effects (font (size 1.27 1.27)) hide)
     )
-    (property "Datasheet" "~" (id 3) (at 266.7 124.46 0)
+    (property "Datasheet" "~" (id 3) (at 281.94 138.43 0)
       (effects (font (size 1.27 1.27)) hide)
     )
@@
     (pin "1")
   )
+  (symbol (lib_id "Device:R") (at 223.52 148.59 90) (mirror x) (unit 1)
+    (in_bom yes) (on_board yes)
+    (property "Reference" "R44" (id 0) (at 222.3516 150.368 0)
+      (effects (font (size 1.27 1.27)) (justify left))
+    )
+    (property "Value" "10k" (id 1) (at 224.663 150.368 0)
+      (effects (font (size 1.27 1.27)) (justify left))
+    )
+    (property "Footprint" "Resistor_SMD:R_0603_1608Metric_Pad0.98x0.95mm_HandSolder" (id 2) (at 223.52 146.812 90)
+      (effects (font (size 1.27 1.27)) hide)
+    )
+    (property "Datasheet" "~" (id 3) (at 223.52 148.59 0)
+      (effects (font (size 1.27 1.27)) hide)
+    )
+    (pin "1")
+    (pin "2")
+  )
   (symbol (lib_id "74xx:74LS32") (at 359.41 109.22 270) (unit 5)
     (in_bom yes) (on_board yes)
@@
       (reference "R43") (unit 1) (value "470") (footprint "Resistor_SMD:R_0603_1608Metric_Pad0.98x0.95mm_HandSolder")
     )
+    (path "/a6ce0a30-a891-4a57-8055-c4618ffd5ce6"
+      (reference "R44") (unit 1) (value "10k") (footprint "Resistor_SMD:R_0603_1608Metric_Pad0.98x0.95mm_HandSolder")
+    )
     (path "/54dc5971-37b9-46a7-8049-349fe99f9b14/e15ab46d-42eb-474f-881c-556db992e495"

Commit message: fix: rx tx
Other:
- note added: "RX"
- note added: "TX"
Changed lines of the file:
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@@
+    (effects (font (size 1.27 1.27) (thickness 0.254) bold italic) (justify left bottom))
+  )
+  (text "RX" (at 190.5 55.88 0)
     (effects (font (size 1.27 1.27) (thickness 0.254) bold italic) (justify left bottom))
   )
@@
     (effects (font (size 1.27 1.27) (thickness 0.254) bold italic) (justify left bottom))
   )
+  (text "TX" (at 190.5 60.96 0)
+    (effects (font (size 1.27 1.27) (thickness 0.254) bold italic) (justify left bottom))
+  )
   (text "Center" (at 364.49 203.2 0)
+    (effects (font (size 1.27 1.27) (thickness 0.254) bold italic) (justify left bottom))
+  )
+  (text "RX" (at 228.6 137.16 0)
     (effects (font (size 1.27 1.27) (thickness 0.254) bold italic) (justify left bottom))
   )
@@
     (effects (font (size 1.27 1.27) (thickness 0.254) bold italic) (justify left bottom))
   )
+  (text "TX" (at 228.6 132.08 0)
+    (effects (font (size 1.27 1.27) (thickness 0.254) bold italic) (justify left bottom))
+  )
