File: kicad/main/_autosave-main.kicad_sch (KiCad schematic)
At the start: 52 parts, among them J1 to cam, J10 I2C_1, J11 drib-kick, J12 drib-kick, J14 5V OUT, J15 LINE, J3 USB_C_Receptacle_USB2.0, J4 Power IN, J5 MD1, J6 MD2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

Commit message: bus
Connections:
- net USB_D+ renamed USB.D+
- net USB_D- renamed USB.D-
Changed lines of the file:
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@@
     (company "A.Saeki")
   )
+  (bus_alias "USB" (members "D+" "D-"))
   (junction (at 273.05 217.17) (diameter 0) (color 0 0 0 0)
   )
@@
   (no_connect (at 52.07 55.88))
   (no_connect (at 203.2 194.31))
+  (bus_entry (at 60.96 43.18) (size 2.54 2.54)
+    (stroke (width 0) (type default) (color 0 0 0 0))
+  )
+  (bus_entry (at 139.7 148.59) (size 2.54 2.54)
+    (stroke (width 0) (type default) (color 0 0 0 0))
+  )
+  (bus_entry (at 60.96 40.64) (size 2.54 2.54)
+    (stroke (width 0) (type default) (color 0 0 0 0))
+  )
+  (bus_entry (at 139.7 151.13) (size 2.54 2.54)
+    (stroke (width 0) (type default) (color 0 0 0 0))
+  )
   (wire (pts (xy 218.44 83.82) (xy 219.71 83.82))
     (stroke (width 0) (type default) (color 0 0 0 0))
@@
     (stroke (width 0) (type default) (color 0 0 0 0))
   )
+  (bus (pts (xy 63.5 43.18) (xy 63.5 45.72))
+    (stroke (width 0) (type default) (color 0 0 0 0))
+  )
   (wire (pts (xy 222.25 217.17) (xy 222.25 176.53))
     (stroke (width 0) (type default) (color 0 0 0 0))
@@
     (stroke (width 0) (type default) (color 0 0 0 0))
   )
+  (bus (pts (xy 139.7 148.59) (xy 137.16 148.59))
+    (stroke (width 0) (type default) (color 0 0 0 0))
+  )
   (wire (pts (xy 273.05 217.17) (xy 279.4 217.17))
     (stroke (width 0) (type default) (color 0 0 0 0))
@@
     (stroke (width 0) (type default) (color 0 0 0 0))
   )
-  (wire (pts (xy 53.34 43.18) (xy 54.61 43.18))
+  (wire (pts (xy 53.34 43.18) (xy 60.96 43.18))
     (stroke (width 0) (type solid) (color 0 0 0 0))
   )
@@
     (stroke (width 0) (type default) (color 0 0 0 0))
   )
+  (wire (pts (xy 142.24 153.67) (xy 149.86 153.67))
+    (stroke (width 0) (type default) (color 0 0 0 0))
+  )
   (wire (pts (xy 191.77 135.89) (xy 191.77 101.6))
     (stroke (width 0) (type default) (color 0 0 0 0))
@@
     (stroke (width 0) (type default) (color 0 0 0 0))
   )
+  (bus (pts (xy 63.5 48.26) (xy 67.31 48.26))
+    (stroke (width 0) (type default) (color 0 0 0 0))
+  )
   (wire (pts (xy 349.25 41.91) (xy 353.06 41.91))
     (stroke (width 0) (type default) (color 0 0 0 0))
@@
     (stroke (width 0) (type default) (color 0 0 0 0))
   )
-  (wire (pts (xy 53.34 40.64) (xy 54.61 40.64))
+  (wire (pts (xy 53.34 40.64) (xy 60.96 40.64))
     (stroke (width 0) (type solid) (color 0 0 0 0))
   )
@@
     (stroke (width 0) (type default) (color 0 0 0 0))
   )
+  (bus (pts (xy 63.5 45.72) (xy 63.5 48.26))
+    (stroke (width 0) (type default) (color 0 0 0 0))
+  )
   (wire (pts (xy 364.49 41.91) (xy 364.49 43.18))
     (stroke (width 0) (type default) (color 0 0 0 0))
@@
     (stroke (width 0) (type default) (color 0 0 0 0))
   )
-  (wire (pts (xy 148.59 153.67) (xy 149.86 153.67))
-    (stroke (width 0) (type default) (color 0 0 0 0))
-  )
   (wire (pts (xy 383.54 29.21) (xy 383.54 31.75))
     (stroke (width 0) (type default) (color 0 0 0 0))
@@
     (stroke (width 0) (type default) (color 0 0 0 0))
   )
+  (bus (pts (xy 139.7 151.13) (xy 139.7 148.59))
+    (stroke (width 0) (type default) (color 0 0 0 0))
+  )
   (wire (pts (xy 232.41 83.82) (xy 240.03 83.82))
     (stroke (width 0) (type default) (color 0 0 0 0))
@@
     (stroke (width 0) (type default) (color 0 0 0 0))
   )
+  (wire (pts (xy 142.24 151.13) (xy 149.86 151.13))
+    (stroke (width 0) (type default) (color 0 0 0 0))
+  )
   (wire (pts (xy 278.13 160.02) (xy 278.13 245.11))
     (stroke (width 0) (type default) (color 0 0 0 0))
@@
   )
   (wire (pts (xy 227.33 171.45) (xy 227.33 193.04))
-    (stroke (width 0) (type default) (color 0 0 0 0))
-  )
-  (wire (pts (xy 148.59 151.13) (xy 149.86 151.13))
     (stroke (width 0) (type default) (color 0 0 0 0))
   )
@@
     (effects (font (size 1.27 1.27) (thickness 0.254) bold italic) (justify left bottom))
   )
+  (label "USB.D+" (at 54.61 43.18 0)
+    (effects (font (size 1.27 1.27)) (justify left bottom))
+  )
   (label "RESET" (at 204.47 218.44 0)
     (effects (font (size 1.27 1.27)) (justify left bottom))
   )
-  (label "USB_D-" (at 148.59 151.13 180)
+  (label "USB.D-" (at 149.86 151.13 180)
     (effects (font (size 1.27 1.27)) (justify right bottom))
-  )
-  (label "USB_D-" (at 54.61 40.64 0)
-    (effects (font (size 1.27 1.27)) (justify left bottom))
   )
   (label "RESET" (at 148.59 146.05 180)
     (effects (font (size 1.27 1.27)) (justify right bottom))
   )
+  (label "USB.D-" (at 54.61 40.64 0)
+    (effects (font (size 1.27 1.27)) (justify left bottom))
+  )
   (label "RESET" (at 213.36 109.22 180)
     (effects (font (size 1.27 1.27)) (justify right bottom))
@@
     (effects (font (size 1.27 1.27)) (justify right bottom))
   )
-  (label "USB_D+" (at 148.59 153.67 180)
+  (label "USB.D+" (at 149.86 153.67 180)
     (effects (font (size 1.27 1.27)) (justify right bottom))
-  )
-  (label "USB_D+" (at 54.61 43.18 0)
-    (effects (font (size 1.27 1.27)) (justify left bottom))
   )
   (global_label "SCL_I2C0" (shape input) (at 260.35 71.12 0) (fields_autoplaced)
@@
     )
   )
+  (global_label "USB{USB}" (shape input) (at 67.31 48.26 0) (fields_autoplaced)
+    (effects (font (size 1.27 1.27)) (justify left))
+    (property "Intersheet References" "${INTERSHEET_REFS}" (id 0) (at 79.0364 48.1806 0)
+      (effects (font (size 1.27 1.27)) (justify left) hide)
+    )
+  )
   (global_label "SDA_I2C1" (shape input) (at 86.36 144.78 0) (fields_autoplaced)
     (effects (font (size 1.27 1.27)) (justify left))
@@
     )
   )
+  (global_label "USB{USB}" (shape input) (at 137.16 148.59 180) (fields_autoplaced)
+    (effects (font (size 1.27 1.27)) (justify right))
+    (property "Intersheet References" "${INTERSHEET_REFS}" (id 0) (at 125.4336 148.6694 0)
+      (effects (font (size 1.27 1.27)) (justify right) hide)
+    )
+  )
