File: kicad/main/4ch_mcb.kicad_sch (KiCad schematic)
At the start: 19 parts, among them J26 ICSP, J27 MD1, J28 MD2, J29 MD3, J30 MD4, U12 ATmega328P-AU, Y1 8Mhz

Commit message: fix: main
Parts:
- renumbered C14 to C11, C15 to C12, D16 to D13, D17 to D14, D18 to D15, D19 to D16, J26 to J21, J27 to J22, J28 to J23, J29 to J24, J30 to J25, R44 to R38, R45 to R39, R46 to R40, R47 to R41, R48 to R42, R49 to R43, U12 to U9
Changed lines of the file:
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@@
   (symbol (lib_id "MCU_Microchip_ATmega:ATmega328P-A") (at 78.74 68.58 0) (unit 1)
     (in_bom yes) (on_board yes)
-    (property "Reference" "U12" (id 0) (at 78.74 108.9406 0))
+    (property "Reference" "U9" (id 0) (at 78.74 108.9406 0))
     (property "Value" "ATmega328P-AU" (id 1) (at 78.74 111.252 0))
     (property "Footprint" "Package_QFP:TQFP-32_7x7mm_P0.8mm" (id 2) (at 78.74 68.58 0)
@@
   (symbol (lib_id "Device:C") (at 127 80.01 0) (unit 1)
     (in_bom yes) (on_board yes) (fields_autoplaced)
-    (property "Reference" "C15" (id 0) (at 129.921 79.1753 0)
+    (property "Reference" "C12" (id 0) (at 129.921 79.1753 0)
       (effects (font (size 1.27 1.27)) (justify left))
     )
@@
   (symbol (lib_id "Connector_Generic:Conn_01x06") (at 147.32 30.48 90) (unit 1)
     (in_bom yes) (on_board yes)
-    (property "Reference" "J26" (id 0) (at 157.1752 31.3944 90)
+    (property "Reference" "J21" (id 0) (at 157.1752 31.3944 90)
       (effects (font (size 1.27 1.27)) (justify right))
     )
@@
   (symbol (lib_id "power:GND") (at 138.43 59.69 0) (unit 1)
     (in_bom yes) (on_board yes)
-    (property "Reference" "#PWR046" (id 0) (at 138.43 66.04 0)
+    (property "Reference" "#PWR050" (id 0) (at 138.43 66.04 0)
       (effects (font (size 1.27 1.27)) hide)
     )
@@
   (symbol (lib_id "Connector_Generic:Conn_01x04") (at 195.58 114.3 0) (unit 1)
     (in_bom yes) (on_board yes)
-    (property "Reference" "J29" (id 0) (at 193.4972 106.2482 0))
+    (property "Reference" "J24" (id 0) (at 193.4972 106.2482 0))
     (property "Value" "MD3" (id 1) (at 193.4972 108.5596 0))
     (property "Footprint" "0.main.robot:JSTB4B-ZR" (id 2) (at 195.58 114.3 0)
@@
   (symbol (lib_id "Diode:1N4001") (at 41.91 29.21 180) (unit 1)
     (in_bom yes) (on_board yes)
-    (property "Reference" "D16" (id 0) (at 41.91 23.6982 0))
+    (property "Reference" "D13" (id 0) (at 41.91 23.6982 0))
     (property "Value" "RSX101VAM-30TR" (id 1) (at 41.91 26.0096 0))
     (property "Footprint" "Diode_SMD:D_0805_2012Metric_Pad1.15x1.40mm_HandSolder" (id 2) (at 41.91 24.765 0)
@@
   (symbol (lib_id "Device:R") (at 78.74 130.81 0) (unit 1)
     (in_bom yes) (on_board yes)
-    (property "Reference" "R46" (id 0) (at 80.772 130.81 90))
+    (property "Reference" "R40" (id 0) (at 80.772 130.81 90))
     (property "Value" "47k" (id 1) (at 78.74 130.81 90))
     (property "Footprint" "Resistor_SMD:R_0603_1608Metric_Pad0.98x0.95mm_HandSolder" (id 2) (at 76.962 130.81 90)
@@
   (symbol (lib_id "power:GND") (at 153.67 106.68 0) (unit 1)
     (in_bom yes) (on_board yes)
-    (property "Reference" "#PWR047" (id 0) (at 153.67 113.03 0)
+    (property "Reference" "#PWR051" (id 0) (at 153.67 113.03 0)
       (effects (font (size 1.27 1.27)) hide)
     )
@@
   (symbol (lib_id "power:+3.3VA") (at 68.58 123.19 0) (unit 1)
     (in_bom yes) (on_board yes)
-    (property "Reference" "#PWR041" (id 0) (at 68.58 127 0)
+    (property "Reference" "#PWR045" (id 0) (at 68.58 127 0)
       (effects (font (size 1.27 1.27)) hide)
     )
@@
   (symbol (lib_id "Device:LED") (at 81.28 165.1 90) (unit 1)
     (in_bom yes) (on_board yes)
-    (property "Reference" "D17" (id 0) (at 78.74 165.1 0))
+    (property "Reference" "D14" (id 0) (at 78.74 165.1 0))
     (property "Value" "LED(OSWT1608)" (id 1) (at 83.82 165.1 0))
     (property "Footprint" "LED_SMD:LED_0603_1608Metric_Pad1.05x0.95mm_HandSolder" (id 2) (at 81.28 165.1 0)
@@
   (symbol (lib_id "power:GND") (at 68.58 171.45 0) (unit 1)
     (in_bom yes) (on_board yes)
-    (property "Reference" "#PWR042" (id 0) (at 68.58 177.8 0)
+    (property "Reference" "#PWR046" (id 0) (at 68.58 177.8 0)
       (effects (font (size 1.27 1.27)) hide)
     )
@@
   (symbol (lib_id "Connector_Generic:Conn_01x04") (at 195.58 88.9 0) (unit 1)
     (in_bom yes) (on_board yes)
-    (property "Reference" "J28" (id 0) (at 193.4972 80.8482 0))
+    (property "Reference" "J23" (id 0) (at 193.4972 80.8482 0))
     (property "Value" "MD2" (id 1) (at 193.4972 83.1596 0))
     (property "Footprint" "0.main.robot:JSTB4B-ZR" (id 2) (at 195.58 88.9 0)
@@
   (symbol (lib_id "Device:R") (at 55.88 43.18 270) (unit 1)
     (in_bom yes) (on_board yes)
-    (property "Reference" "R44" (id 0) (at 55.88 37.9222 90))
+    (property "Reference" "R38" (id 0) (at 55.88 37.9222 90))
     (property "Value" "47k" (id 1) (at 55.88 40.2336 90))
     (property "Footprint" "Resistor_SMD:R_0603_1608Metric_Pad0.98x0.95mm_HandSolder" (id 2) (at 55.88 41.402 90)
@@
   (symbol (lib_id "Device:R") (at 85.09 130.81 0) (unit 1)
     (in_bom yes) (on_board yes)
-    (property "Reference" "R47" (id 0) (at 87.122 130.81 90))
+    (property "Reference" "R41" (id 0) (at 87.122 130.81 90))
     (property "Value" "47k" (id 1) (at 85.09 130.81 90))
     (property "Footprint" "Resistor_SMD:R_0603_1608Metric_Pad0.98x0.95mm_HandSolder" (id 2) (at 83.312 130.81 90)
@@
   (symbol (lib_id "Device:R") (at 138.43 102.87 90) (unit 1)
     (in_bom yes) (on_board yes)
-    (property "Reference" "R48" (id 0) (at 138.43 100.838 90))
+    (property "Reference" "R42" (id 0) (at 138.43 100.838 90))
     (property "Value" "470" (id 1) (at 138.43 102.87 90))
     (property "Footprint" "Resistor_SMD:R_0603_1608Metric_Pad0.98x0.95mm_HandSolder" (id 2) (at 138.43 104.648 90)
@@
   (symbol (lib_id "Connector_Generic:Conn_01x04") (at 195.58 48.26 0) (unit 1)
     (in_bom yes) (on_board yes)
-    (property "Reference" "J27" (id 0) (at 193.4972 40.2082 0))
+    (property "Reference" "J22" (id 0) (at 193.4972 40.2082 0))
     (property "Value" "MD1" (id 1) (at 193.4972 42.5196 0))
     (property "Footprint" "0.main.robot:JSTB4B-ZR" (id 2) (at 195.58 48.26 0)
@@
   (symbol (lib_id "power:+3.3VA") (at 93.98 29.21 0) (unit 1)
     (in_bom yes) (on_board yes) (fields_autoplaced)
-    (property "Reference" "#PWR043" (id 0) (at 93.98 33.02 0)
+    (property "Reference" "#PWR047" (id 0) (at 93.98 33.02 0)
       (effects (font (size 1.27 1.27)) hide)
     )
@@
   (symbol (lib_id "Device:LED") (at 149.86 102.87 180) (unit 1)
     (in_bom yes) (on_board yes)
-    (property "Reference" "D18" (id 0) (at 149.86 105.41 0))
+    (property "Reference" "D15" (id 0) (at 149.86 105.41 0))
     (property "Value" "LED(OSWT1608)" (id 1) (at 149.86 100.33 0))
     (property "Footprint" "LED_SMD:LED_0603_1608Metric_Pad1.05x0.95mm_HandSolder" (id 2) (at 149.86 102.87 0)
@@
   (symbol (lib_id "Device:R") (at 74.93 160.02 90) (unit 1)
     (in_bom yes) (on_board yes)
-    (property "Reference" "R45" (id 0) (at 74.93 157.988 90))
+    (property "Reference" "R39" (id 0) (at 74.93 157.988 90))
     (property "Value" "470" (id 1) (at 74.93 160.02 90))
     (property "Footprint" "Resistor_SMD:R_0603_1608Metric_Pad0.98x0.95mm_HandSolder" (id 2) (at 74.93 161.798 90)
@@
   (symbol (lib_id "power:+3.3VA") (at 158.75 74.93 0) (unit 1)
     (in_bom yes) (on_board yes) (fields_autoplaced)
-    (property "Reference" "#PWR049" (id 0) (at 158.75 78.74 0)
+    (property "Reference" "#PWR053" (id 0) (at 158.75 78.74 0)
       (effects (font (size 1.27 1.27)) hide)
     )
@@
   (symbol (lib_id "Device:R") (at 151.13 76.2 90) (unit 1)
     (in_bom yes) (on_board yes)
-    (property "Reference" "R49" (id 0) (at 151.13 74.168 90))
+    (property "Reference" "R43" (id 0) (at 151.13 74.168 90))
     (property "Value" "10k" (id 1) (at 151.13 76.2 90))
     (property "Footprint" "Resistor_SMD:R_0603_1608Metric_Pad0.98x0.95mm_HandSolder" (id 2) (at 151.13 77.978 90)
@@
   (symbol (lib_id "Device:C") (at 49.53 85.09 0) (unit 1)
     (in_bom yes) (on_board yes)
-    (property "Reference" "C14" (id 0) (at 50.165 82.55 0)
+    (property "Reference" "C11" (id 0) (at 50.165 82.55 0)
       (effects (font (size 1.27 1.27)) (justify left))
     )
@@
   (symbol (lib_id "power:+3.3VA") (at 137.16 39.37 0) (unit 1)
     (in_bom yes) (on_board yes) (fields_autoplaced)
-    (property "Reference" "#PWR045" (id 0) (at 137.16 43.18 0)
+    (property "Reference" "#PWR049" (id 0) (at 137.16 43.18 0)
       (effects (font (size 1.27 1.27)) hide)
     )
@@
   (symbol (lib_id "Connector_Generic:Conn_01x04") (at 195.58 130.81 0) (unit 1)
     (in_bom yes) (on_board yes)
-    (property "Reference" "J30" (id 0) (at 193.4972 122.7582 0))
+    (property "Reference" "J25" (id 0) (at 193.4972 122.7582 0))
     (property "Value" "MD4" (id 1) (at 193.4972 125.0696 0))
     (property "Footprint" "0.main.robot:JSTB4B-ZR" (id 2) (at 195.58 130.81 0)
@@
   (symbol (lib_id "power:GND") (at 49.53 120.65 0) (unit 1)
     (in_bom yes) (on_board yes)
-    (property "Reference" "#PWR040" (id 0) (at 49.53 127 0)
+    (property "Reference" "#PWR044" (id 0) (at 49.53 127 0)
       (effects (font (size 1.27 1.27)) hide)
     )
@@
   (symbol (lib_id "power:GND") (at 154.94 38.1 0) (unit 1)
     (in_bom yes) (on_board yes)
-    (property "Reference" "#PWR048" (id 0) (at 154.94 44.45 0)
+    (property "Reference" "#PWR052" (id 0) (at 154.94 44.45 0)
       (effects (font (size 1.27 1.27)) hide)
     )
@@
   (symbol (lib_id "Device:D") (at 151.13 81.28 0) (mirror y) (unit 1)
     (in_bom yes) (on_board yes)
-    (property "Reference" "D19" (id 0) (at 151.13 78.74 0))
+    (property "Reference" "D16" (id 0) (at 151.13 78.74 0))
     (property "Value" "RSX101VAM-30TR" (id 1) (at 151.13 83.82 0))
     (property "Footprint" "Diode_SMD:D_0805_2012Metric_Pad1.15x1.40mm_HandSolder" (id 2) (at 151.13 81.28 0)
@@
   (symbol (lib_id "power:GND") (at 127 96.52 0) (unit 1)
     (in_bom yes) (on_board yes)
-    (property "Reference" "#PWR044" (id 0) (at 127 102.87 0)
-      (effects (font (size 1.27 1.27)) hide)
-    )
+    (property "Reference" "#PWR048" (id 0) (at 127 102.87 0)
+      (effects (font (size 1.27 1.27)) hide)
+    )

Commit message: fix: main xbee
Parts:
- renumbered C12 to C10, C11 to C9, D13 to D10, D14 to D11, D15 to D12, D16 to D13, J21 to J22, J22 to J23, J23 to J24, J24 to J25, J25 to J26, R38 to R31, R39 to R32, R40 to R33, R41 to R34, R42 to R35, R43 to R36, U9 to U7
Changed lines of the file:
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@@
   (symbol (lib_id "MCU_Microchip_ATmega:ATmega328P-A") (at 78.74 68.58 0) (unit 1)
     (in_bom yes) (on_board yes)
-    (property "Reference" "U9" (id 0) (at 78.74 108.9406 0))
+    (property "Reference" "U7" (id 0) (at 78.74 108.9406 0))
     (property "Value" "ATmega328P-AU" (id 1) (at 78.74 111.252 0))
     (property "Footprint" "Package_QFP:TQFP-32_7x7mm_P0.8mm" (id 2) (at 78.74 68.58 0)
@@
   (symbol (lib_id "Device:C") (at 127 80.01 0) (unit 1)
     (in_bom yes) (on_board yes) (fields_autoplaced)
-    (property "Reference" "C12" (id 0) (at 129.921 79.1753 0)
+    (property "Reference" "C10" (id 0) (at 129.921 79.1753 0)
       (effects (font (size 1.27 1.27)) (justify left))
     )
@@
   (symbol (lib_id "Connector_Generic:Conn_01x06") (at 147.32 30.48 90) (unit 1)
     (in_bom yes) (on_board yes)
-    (property "Reference" "J21" (id 0) (at 157.1752 31.3944 90)
+    (property "Reference" "J22" (id 0) (at 157.1752 31.3944 90)
       (effects (font (size 1.27 1.27)) (justify right))
     )
@@
   (symbol (lib_id "power:GND") (at 138.43 59.69 0) (unit 1)
     (in_bom yes) (on_board yes)
-    (property "Reference" "#PWR050" (id 0) (at 138.43 66.04 0)
+    (property "Reference" "#PWR049" (id 0) (at 138.43 66.04 0)
       (effects (font (size 1.27 1.27)) hide)
     )
@@
   (symbol (lib_id "Connector_Generic:Conn_01x04") (at 195.58 114.3 0) (unit 1)
     (in_bom yes) (on_board yes)
-    (property "Reference" "J24" (id 0) (at 193.4972 106.2482 0))
+    (property "Reference" "J25" (id 0) (at 193.4972 106.2482 0))
     (property "Value" "MD3" (id 1) (at 193.4972 108.5596 0))
     (property "Footprint" "0.main.robot:JSTB4B-ZR" (id 2) (at 195.58 114.3 0)
@@
   (symbol (lib_id "Diode:1N4001") (at 41.91 29.21 180) (unit 1)
     (in_bom yes) (on_board yes)
-    (property "Reference" "D13" (id 0) (at 41.91 23.6982 0))
+    (property "Reference" "D10" (id 0) (at 41.91 23.6982 0))
     (property "Value" "RSX101VAM-30TR" (id 1) (at 41.91 26.0096 0))
     (property "Footprint" "Diode_SMD:D_0805_2012Metric_Pad1.15x1.40mm_HandSolder" (id 2) (at 41.91 24.765 0)
@@
   (symbol (lib_id "Device:R") (at 78.74 130.81 0) (unit 1)
     (in_bom yes) (on_board yes)
-    (property "Reference" "R40" (id 0) (at 80.772 130.81 90))
+    (property "Reference" "R33" (id 0) (at 80.772 130.81 90))
     (property "Value" "47k" (id 1) (at 78.74 130.81 90))
     (property "Footprint" "Resistor_SMD:R_0603_1608Metric_Pad0.98x0.95mm_HandSolder" (id 2) (at 76.962 130.81 90)
@@
   (symbol (lib_id "power:GND") (at 153.67 106.68 0) (unit 1)
     (in_bom yes) (on_board yes)
-    (property "Reference" "#PWR051" (id 0) (at 153.67 113.03 0)
+    (property "Reference" "#PWR050" (id 0) (at 153.67 113.03 0)
       (effects (font (size 1.27 1.27)) hide)
     )
@@
   (symbol (lib_id "power:+3.3VA") (at 68.58 123.19 0) (unit 1)
     (in_bom yes) (on_board yes)
-    (property "Reference" "#PWR045" (id 0) (at 68.58 127 0)
+    (property "Reference" "#PWR044" (id 0) (at 68.58 127 0)
       (effects (font (size 1.27 1.27)) hide)
     )
@@
   (symbol (lib_id "Device:LED") (at 81.28 165.1 90) (unit 1)
     (in_bom yes) (on_board yes)
-    (property "Reference" "D14" (id 0) (at 78.74 165.1 0))
+    (property "Reference" "D11" (id 0) (at 78.74 165.1 0))
     (property "Value" "LED(OSWT1608)" (id 1) (at 83.82 165.1 0))
     (property "Footprint" "LED_SMD:LED_0603_1608Metric_Pad1.05x0.95mm_HandSolder" (id 2) (at 81.28 165.1 0)
@@
   (symbol (lib_id "power:GND") (at 68.58 171.45 0) (unit 1)
     (in_bom yes) (on_board yes)
-    (property "Reference" "#PWR046" (id 0) (at 68.58 177.8 0)
+    (property "Reference" "#PWR045" (id 0) (at 68.58 177.8 0)
       (effects (font (size 1.27 1.27)) hide)
     )
@@
   (symbol (lib_id "Connector_Generic:Conn_01x04") (at 195.58 88.9 0) (unit 1)
     (in_bom yes) (on_board yes)
-    (property "Reference" "J23" (id 0) (at 193.4972 80.8482 0))
+    (property "Reference" "J24" (id 0) (at 193.4972 80.8482 0))
     (property "Value" "MD2" (id 1) (at 193.4972 83.1596 0))
     (property "Footprint" "0.main.robot:JSTB4B-ZR" (id 2) (at 195.58 88.9 0)
@@
   (symbol (lib_id "Device:R") (at 55.88 43.18 270) (unit 1)
     (in_bom yes) (on_board yes)
-    (property "Reference" "R38" (id 0) (at 55.88 37.9222 90))
+    (property "Reference" "R31" (id 0) (at 55.88 37.9222 90))
     (property "Value" "47k" (id 1) (at 55.88 40.2336 90))
     (property "Footprint" "Resistor_SMD:R_0603_1608Metric_Pad0.98x0.95mm_HandSolder" (id 2) (at 55.88 41.402 90)
@@
   (symbol (lib_id "Device:R") (at 85.09 130.81 0) (unit 1)
     (in_bom yes) (on_board yes)
-    (property "Reference" "R41" (id 0) (at 87.122 130.81 90))
+    (property "Reference" "R34" (id 0) (at 87.122 130.81 90))
     (property "Value" "47k" (id 1) (at 85.09 130.81 90))
     (property "Footprint" "Resistor_SMD:R_0603_1608Metric_Pad0.98x0.95mm_HandSolder" (id 2) (at 83.312 130.81 90)
@@
   (symbol (lib_id "Device:R") (at 138.43 102.87 90) (unit 1)
     (in_bom yes) (on_board yes)
-    (property "Reference" "R42" (id 0) (at 138.43 100.838 90))
+    (property "Reference" "R35" (id 0) (at 138.43 100.838 90))
     (property "Value" "470" (id 1) (at 138.43 102.87 90))
     (property "Footprint" "Resistor_SMD:R_0603_1608Metric_Pad0.98x0.95mm_HandSolder" (id 2) (at 138.43 104.648 90)
@@
   (symbol (lib_id "Connector_Generic:Conn_01x04") (at 195.58 48.26 0) (unit 1)
     (in_bom yes) (on_board yes)
-    (property "Reference" "J22" (id 0) (at 193.4972 40.2082 0))
+    (property "Reference" "J23" (id 0) (at 193.4972 40.2082 0))
     (property "Value" "MD1" (id 1) (at 193.4972 42.5196 0))
     (property "Footprint" "0.main.robot:JSTB4B-ZR" (id 2) (at 195.58 48.26 0)
@@
   (symbol (lib_id "power:+3.3VA") (at 93.98 29.21 0) (unit 1)
     (in_bom yes) (on_board yes) (fields_autoplaced)
-    (property "Reference" "#PWR047" (id 0) (at 93.98 33.02 0)
+    (property "Reference" "#PWR046" (id 0) (at 93.98 33.02 0)
       (effects (font (size 1.27 1.27)) hide)
     )
@@
   (symbol (lib_id "Device:LED") (at 149.86 102.87 180) (unit 1)
     (in_bom yes) (on_board yes)
-    (property "Reference" "D15" (id 0) (at 149.86 105.41 0))
+    (property "Reference" "D12" (id 0) (at 149.86 105.41 0))
     (property "Value" "LED(OSWT1608)" (id 1) (at 149.86 100.33 0))
     (property "Footprint" "LED_SMD:LED_0603_1608Metric_Pad1.05x0.95mm_HandSolder" (id 2) (at 149.86 102.87 0)
@@
   (symbol (lib_id "Device:R") (at 74.93 160.02 90) (unit 1)
     (in_bom yes) (on_board yes)
-    (property "Reference" "R39" (id 0) (at 74.93 157.988 90))
+    (property "Reference" "R32" (id 0) (at 74.93 157.988 90))
     (property "Value" "470" (id 1) (at 74.93 160.02 90))
     (property "Footprint" "Resistor_SMD:R_0603_1608Metric_Pad0.98x0.95mm_HandSolder" (id 2) (at 74.93 161.798 90)
@@
   (symbol (lib_id "power:+3.3VA") (at 158.75 74.93 0) (unit 1)
     (in_bom yes) (on_board yes) (fields_autoplaced)
-    (property "Reference" "#PWR053" (id 0) (at 158.75 78.74 0)
+    (property "Reference" "#PWR052" (id 0) (at 158.75 78.74 0)
       (effects (font (size 1.27 1.27)) hide)
     )
@@
   (symbol (lib_id "Device:R") (at 151.13 76.2 90) (unit 1)
     (in_bom yes) (on_board yes)
-    (property "Reference" "R43" (id 0) (at 151.13 74.168 90))
+    (property "Reference" "R36" (id 0) (at 151.13 74.168 90))
     (property "Value" "10k" (id 1) (at 151.13 76.2 90))
     (property "Footprint" "Resistor_SMD:R_0603_1608Metric_Pad0.98x0.95mm_HandSolder" (id 2) (at 151.13 77.978 90)
@@
   (symbol (lib_id "Device:C") (at 49.53 85.09 0) (unit 1)
     (in_bom yes) (on_board yes)
-    (property "Reference" "C11" (id 0) (at 50.165 82.55 0)
+    (property "Reference" "C9" (id 0) (at 50.165 82.55 0)
       (effects (font (size 1.27 1.27)) (justify left))
     )
@@
   (symbol (lib_id "power:+3.3VA") (at 137.16 39.37 0) (unit 1)
     (in_bom yes) (on_board yes) (fields_autoplaced)
-    (property "Reference" "#PWR049" (id 0) (at 137.16 43.18 0)
+    (property "Reference" "#PWR048" (id 0) (at 137.16 43.18 0)
       (effects (font (size 1.27 1.27)) hide)
     )
@@
   (symbol (lib_id "Connector_Generic:Conn_01x04") (at 195.58 130.81 0) (unit 1)
     (in_bom yes) (on_board yes)
-    (property "Reference" "J25" (id 0) (at 193.4972 122.7582 0))
+    (property "Reference" "J26" (id 0) (at 193.4972 122.7582 0))
     (property "Value" "MD4" (id 1) (at 193.4972 125.0696 0))
     (property "Footprint" "0.main.robot:JSTB4B-ZR" (id 2) (at 195.58 130.81 0)
@@
   (symbol (lib_id "power:GND") (at 49.53 120.65 0) (unit 1)
     (in_bom yes) (on_board yes)
-    (property "Reference" "#PWR044" (id 0) (at 49.53 127 0)
+    (property "Reference" "#PWR043" (id 0) (at 49.53 127 0)
       (effects (font (size 1.27 1.27)) hide)
     )
@@
   (symbol (lib_id "power:GND") (at 154.94 38.1 0) (unit 1)
     (in_bom yes) (on_board yes)
-    (property "Reference" "#PWR052" (id 0) (at 154.94 44.45 0)
+    (property "Reference" "#PWR051" (id 0) (at 154.94 44.45 0)
       (effects (font (size 1.27 1.27)) hide)
     )
@@
   (symbol (lib_id "Device:D") (at 151.13 81.28 0) (mirror y) (unit 1)
     (in_bom yes) (on_board yes)
-    (property "Reference" "D16" (id 0) (at 151.13 78.74 0))
+    (property "Reference" "D13" (id 0) (at 151.13 78.74 0))
     (property "Value" "RSX101VAM-30TR" (id 1) (at 151.13 83.82 0))
     (property "Footprint" "Diode_SMD:D_0805_2012Metric_Pad1.15x1.40mm_HandSolder" (id 2) (at 151.13 81.28 0)
@@
   (symbol (lib_id "power:GND") (at 127 96.52 0) (unit 1)
     (in_bom yes) (on_board yes)
-    (property "Reference" "#PWR048" (id 0) (at 127 102.87 0)
-      (effects (font (size 1.27 1.27)) hide)
-    )
+    (property "Reference" "#PWR047" (id 0) (at 127 102.87 0)
+      (effects (font (size 1.27 1.27)) hide)
+    )
