File: kicad/main/4ch_mcb.kicad_sch (KiCad schematic)
At the start: 19 parts, among them J16 ICSP, J17 MD1, J18 MD2, J19 MD3, J20 MD4, U6 ATmega328P-AU, Y1 8Mhz

Commit message: update
Parts:
- renumbered C7 to C5, C8 to C6, D7 to D6, D8 to D7, D9 to D8, D10 to D9, J16 to J15, J17 to J16, J18 to J17, J19 to J18, J20 to J19, R21 to R20, R22 to R21, R23 to R22, R24 to R23, R25 to R24, R26 to R25, U6 to U5
Changed lines of the file:
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@@
   (symbol (lib_id "MCU_Microchip_ATmega:ATmega328P-A") (at 78.74 68.58 0) (unit 1)
     (in_bom yes) (on_board yes)
-    (property "Reference" "U6" (id 0) (at 78.74 108.9406 0))
+    (property "Reference" "U5" (id 0) (at 78.74 108.9406 0))
     (property "Value" "ATmega328P-AU" (id 1) (at 78.74 111.252 0))
     (property "Footprint" "Package_QFP:TQFP-32_7x7mm_P0.8mm" (id 2) (at 78.74 68.58 0)
@@
   (symbol (lib_id "Device:C") (at 127 80.01 0) (unit 1)
     (in_bom yes) (on_board yes) (fields_autoplaced)
-    (property "Reference" "C8" (id 0) (at 129.921 79.1753 0)
+    (property "Reference" "C6" (id 0) (at 129.921 79.1753 0)
       (effects (font (size 1.27 1.27)) (justify left))
     )
@@
   (symbol (lib_id "power:GND") (at 138.43 59.69 0) (unit 1)
     (in_bom yes) (on_board yes)
-    (property "Reference" "#PWR055" (id 0) (at 138.43 66.04 0)
+    (property "Reference" "#PWR051" (id 0) (at 138.43 66.04 0)
       (effects (font (size 1.27 1.27)) hide)
     )
@@
   (symbol (lib_id "Connector_Generic:Conn_01x04") (at 195.58 114.3 0) (unit 1)
     (in_bom yes) (on_board yes)
-    (property "Reference" "J19" (id 0) (at 193.4972 106.2482 0))
+    (property "Reference" "J18" (id 0) (at 193.4972 106.2482 0))
     (property "Value" "MD3" (id 1) (at 193.4972 108.5596 0))
     (property "Footprint" "0.main.robot:JSTB4B-ZR" (id 2) (at 195.58 114.3 0)
@@
   (symbol (lib_id "Diode:1N4001") (at 41.91 29.21 180) (unit 1)
     (in_bom yes) (on_board yes)
-    (property "Reference" "D7" (id 0) (at 41.91 23.6982 0))
+    (property "Reference" "D6" (id 0) (at 41.91 23.6982 0))
     (property "Value" "RSX101VAM-30TR" (id 1) (at 41.91 26.0096 0))
     (property "Footprint" "Diode_SMD:D_0805_2012Metric_Pad1.15x1.40mm_HandSolder" (id 2) (at 41.91 24.765 0)
@@
   (symbol (lib_id "Device:R") (at 78.74 130.81 0) (unit 1)
     (in_bom yes) (on_board yes)
-    (property "Reference" "R23" (id 0) (at 80.772 130.81 90))
+    (property "Reference" "R22" (id 0) (at 80.772 130.81 90))
     (property "Value" "47k" (id 1) (at 78.74 130.81 90))
     (property "Footprint" "Resistor_SMD:R_0603_1608Metric_Pad0.98x0.95mm_HandSolder" (id 2) (at 76.962 130.81 90)
@@
   (symbol (lib_id "power:GND") (at 154.94 38.1 0) (unit 1)
     (in_bom yes) (on_board yes)
-    (property "Reference" "#PWR057" (id 0) (at 154.94 44.45 0)
+    (property "Reference" "#PWR053" (id 0) (at 154.94 44.45 0)
       (effects (font (size 1.27 1.27)) hide)
     )
@@
   (symbol (lib_id "power:GND") (at 153.67 106.68 0) (unit 1)
     (in_bom yes) (on_board yes)
-    (property "Reference" "#PWR056" (id 0) (at 153.67 113.03 0)
+    (property "Reference" "#PWR052" (id 0) (at 153.67 113.03 0)
       (effects (font (size 1.27 1.27)) hide)
     )
@@
   (symbol (lib_id "power:+3.3VA") (at 68.58 123.19 0) (unit 1)
     (in_bom yes) (on_board yes)
-    (property "Reference" "#PWR050" (id 0) (at 68.58 127 0)
+    (property "Reference" "#PWR046" (id 0) (at 68.58 127 0)
       (effects (font (size 1.27 1.27)) hide)
     )
@@
   (symbol (lib_id "power:+3.3VA") (at 137.16 39.37 0) (unit 1)
     (in_bom yes) (on_board yes) (fields_autoplaced)
-    (property "Reference" "#PWR054" (id 0) (at 137.16 43.18 0)
+    (property "Reference" "#PWR050" (id 0) (at 137.16 43.18 0)
       (effects (font (size 1.27 1.27)) hide)
     )
@@
   (symbol (lib_id "Device:LED") (at 81.28 165.1 90) (unit 1)
     (in_bom yes) (on_board yes)
-    (property "Reference" "D8" (id 0) (at 78.74 165.1 0))
+    (property "Reference" "D7" (id 0) (at 78.74 165.1 0))
     (property "Value" "LED(OSWT1608)" (id 1) (at 83.82 165.1 0))
     (property "Footprint" "LED_SMD:LED_0603_1608Metric_Pad1.05x0.95mm_HandSolder" (id 2) (at 81.28 165.1 0)
@@
   (symbol (lib_id "power:GND") (at 68.58 171.45 0) (unit 1)
     (in_bom yes) (on_board yes)
-    (property "Reference" "#PWR051" (id 0) (at 68.58 177.8 0)
+    (property "Reference" "#PWR047" (id 0) (at 68.58 177.8 0)
       (effects (font (size 1.27 1.27)) hide)
     )
@@
   (symbol (lib_id "Connector_Generic:Conn_01x04") (at 195.58 88.9 0) (unit 1)
     (in_bom yes) (on_board yes)
-    (property "Reference" "J18" (id 0) (at 193.4972 80.8482 0))
+    (property "Reference" "J17" (id 0) (at 193.4972 80.8482 0))
     (property "Value" "MD2" (id 1) (at 193.4972 83.1596 0))
     (property "Footprint" "0.main.robot:JSTB4B-ZR" (id 2) (at 195.58 88.9 0)
@@
   (symbol (lib_id "Device:R") (at 55.88 43.18 270) (unit 1)
     (in_bom yes) (on_board yes)
-    (property "Reference" "R21" (id 0) (at 55.88 37.9222 90))
+    (property "Reference" "R20" (id 0) (at 55.88 37.9222 90))
     (property "Value" "47k" (id 1) (at 55.88 40.2336 90))
     (property "Footprint" "Resistor_SMD:R_0603_1608Metric_Pad0.98x0.95mm_HandSolder" (id 2) (at 55.88 41.402 90)
@@
   (symbol (lib_id "Device:R") (at 85.09 130.81 0) (unit 1)
     (in_bom yes) (on_board yes)
-    (property "Reference" "R24" (id 0) (at 87.122 130.81 90))
+    (property "Reference" "R23" (id 0) (at 87.122 130.81 90))
     (property "Value" "47k" (id 1) (at 85.09 130.81 90))
     (property "Footprint" "Resistor_SMD:R_0603_1608Metric_Pad0.98x0.95mm_HandSolder" (id 2) (at 83.312 130.81 90)
@@
   (symbol (lib_id "Device:R") (at 138.43 102.87 90) (unit 1)
     (in_bom yes) (on_board yes)
-    (property "Reference" "R25" (id 0) (at 138.43 100.838 90))
+    (property "Reference" "R24" (id 0) (at 138.43 100.838 90))
     (property "Value" "470" (id 1) (at 138.43 102.87 90))
     (property "Footprint" "Resistor_SMD:R_0603_1608Metric_Pad0.98x0.95mm_HandSolder" (id 2) (at 138.43 104.648 90)
@@
   (symbol (lib_id "Connector_Generic:Conn_01x04") (at 195.58 48.26 0) (unit 1)
     (in_bom yes) (on_board yes)
-    (property "Reference" "J17" (id 0) (at 193.4972 40.2082 0))
+    (property "Reference" "J16" (id 0) (at 193.4972 40.2082 0))
     (property "Value" "MD1" (id 1) (at 193.4972 42.5196 0))
     (property "Footprint" "0.main.robot:JSTB4B-ZR" (id 2) (at 195.58 48.26 0)
@@
   (symbol (lib_id "power:+3.3VA") (at 93.98 29.21 0) (unit 1)
     (in_bom yes) (on_board yes) (fields_autoplaced)
-    (property "Reference" "#PWR052" (id 0) (at 93.98 33.02 0)
+    (property "Reference" "#PWR048" (id 0) (at 93.98 33.02 0)
       (effects (font (size 1.27 1.27)) hide)
     )
@@
   (symbol (lib_id "Device:LED") (at 149.86 102.87 180) (unit 1)
     (in_bom yes) (on_board yes)
-    (property "Reference" "D9" (id 0) (at 149.86 105.41 0))
+    (property "Reference" "D8" (id 0) (at 149.86 105.41 0))
     (property "Value" "LED(OSWT1608)" (id 1) (at 149.86 100.33 0))
     (property "Footprint" "LED_SMD:LED_0603_1608Metric_Pad1.05x0.95mm_HandSolder" (id 2) (at 149.86 102.87 0)
@@
   (symbol (lib_id "Device:R") (at 74.93 160.02 90) (unit 1)
     (in_bom yes) (on_board yes)
-    (property "Reference" "R22" (id 0) (at 74.93 157.988 90))
+    (property "Reference" "R21" (id 0) (at 74.93 157.988 90))
     (property "Value" "470" (id 1) (at 74.93 160.02 90))
     (property "Footprint" "Resistor_SMD:R_0603_1608Metric_Pad0.98x0.95mm_HandSolder" (id 2) (at 74.93 161.798 90)
@@
   (symbol (lib_id "power:+3.3VA") (at 158.75 74.93 0) (unit 1)
     (in_bom yes) (on_board yes) (fields_autoplaced)
-    (property "Reference" "#PWR058" (id 0) (at 158.75 78.74 0)
+    (property "Reference" "#PWR054" (id 0) (at 158.75 78.74 0)
       (effects (font (size 1.27 1.27)) hide)
     )
@@
   (symbol (lib_id "Device:R") (at 151.13 76.2 90) (unit 1)
     (in_bom yes) (on_board yes)
-    (property "Reference" "R26" (id 0) (at 151.13 74.168 90))
+    (property "Reference" "R25" (id 0) (at 151.13 74.168 90))
     (property "Value" "10k" (id 1) (at 151.13 76.2 90))
     (property "Footprint" "Resistor_SMD:R_0603_1608Metric_Pad0.98x0.95mm_HandSolder" (id 2) (at 151.13 77.978 90)
@@
   (symbol (lib_id "Device:C") (at 49.53 85.09 0) (unit 1)
     (in_bom yes) (on_board yes)
-    (property "Reference" "C7" (id 0) (at 50.165 82.55 0)
+    (property "Reference" "C5" (id 0) (at 50.165 82.55 0)
       (effects (font (size 1.27 1.27)) (justify left))
     )
@@
   (symbol (lib_id "Connector_Generic:Conn_01x04") (at 195.58 130.81 0) (unit 1)
     (in_bom yes) (on_board yes)
-    (property "Reference" "J20" (id 0) (at 193.4972 122.7582 0))
+    (property "Reference" "J19" (id 0) (at 193.4972 122.7582 0))
     (property "Value" "MD4" (id 1) (at 193.4972 125.0696 0))
     (property "Footprint" "0.main.robot:JSTB4B-ZR" (id 2) (at 195.58 130.81 0)
@@
   (symbol (lib_id "Connector_Generic:Conn_01x06") (at 147.32 30.48 90) (unit 1)
     (in_bom yes) (on_board yes)
-    (property "Reference" "J16" (id 0) (at 157.1752 31.3944 90)
+    (property "Reference" "J15" (id 0) (at 157.1752 31.3944 90)
       (effects (font (size 1.27 1.27)) (justify right))
     )
@@
   (symbol (lib_id "power:GND") (at 49.53 120.65 0) (unit 1)
     (in_bom yes) (on_board yes)
-    (property "Reference" "#PWR049" (id 0) (at 49.53 127 0)
+    (property "Reference" "#PWR045" (id 0) (at 49.53 127 0)
       (effects (font (size 1.27 1.27)) hide)
     )
@@
   (symbol (lib_id "Device:D") (at 151.13 81.28 0) (mirror y) (unit 1)
     (in_bom yes) (on_board yes)
-    (property "Reference" "D10" (id 0) (at 151.13 78.74 0))
+    (property "Reference" "D9" (id 0) (at 151.13 78.74 0))
     (property "Value" "RSX101VAM-30TR" (id 1) (at 151.13 83.82 0))
     (property "Footprint" "Diode_SMD:D_0805_2012Metric_Pad1.15x1.40mm_HandSolder" (id 2) (at 151.13 81.28 0)
@@
   (symbol (lib_id "power:GND") (at 127 96.52 0) (unit 1)
     (in_bom yes) (on_board yes)
-    (property "Reference" "#PWR053" (id 0) (at 127 102.87 0)
-      (effects (font (size 1.27 1.27)) hide)
-    )
+    (property "Reference" "#PWR049" (id 0) (at 127 102.87 0)
+      (effects (font (size 1.27 1.27)) hide)
+    )

Commit message: update: main
Parts:
- R22, R23: value 47k -> 10k
Changed lines of the file:
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@@
     (in_bom yes) (on_board yes)
     (property "Reference" "R22" (id 0) (at 80.772 130.81 90))
-    (property "Value" "47k" (id 1) (at 78.74 130.81 90))
+    (property "Value" "10k" (id 1) (at 78.74 130.81 90))
     (property "Footprint" "Resistor_SMD:R_0603_1608Metric_Pad0.98x0.95mm_HandSolder" (id 2) (at 76.962 130.81 90)
       (effects (font (size 1.27 1.27)) hide)
@@
     (in_bom yes) (on_board yes)
     (property "Reference" "R23" (id 0) (at 87.122 130.81 90))
-    (property "Value" "47k" (id 1) (at 85.09 130.81 90))
+    (property "Value" "10k" (id 1) (at 85.09 130.81 90))
     (property "Footprint" "Resistor_SMD:R_0603_1608Metric_Pad0.98x0.95mm_HandSolder" (id 2) (at 83.312 130.81 90)
       (effects (font (size 1.27 1.27)) hide)
