File: kicad/main/LineTrimmer.kicad_sch (KiCad schematic)
At the start: 22 parts, among them J31 I2C/OLED, J32 ICSP, J33 Trimmer, SW8 RESET, U13 ATmega328P-AU, Y2 8Mhz

Commit message: fix: main
Parts:
- renumbered C16 to C13, C17 to C14, C18 to C15, D20 to D17, D21 to D18, D22 to D19, J31 to J26, J32 to J27, J33 to J28, R50 to R44, R51 to R45, R52 to R46, R53 to R47, R54 to R48, RV2 to RV1, RV3 to RV2, RV4 to RV3, RV5 to RV4, RV6 to RV5, SW8 to SW7, U13 to U10
Changed lines of the file:
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@@
   (symbol (lib_id "power:GND") (at 133.35 82.55 0) (unit 1)
     (in_bom yes) (on_board yes)
-    (property "Reference" "#PWR053" (id 0) (at 133.35 88.9 0)
+    (property "Reference" "#PWR057" (id 0) (at 133.35 88.9 0)
       (effects (font (size 1.27 1.27)) hide)
     )
@@
   (symbol (lib_id "Device:R") (at 50.8 68.58 270) (unit 1)
     (in_bom yes) (on_board yes)
-    (property "Reference" "R50" (id 0) (at 50.8 63.3222 90))
+    (property "Reference" "R44" (id 0) (at 50.8 63.3222 90))
     (property "Value" "47k" (id 1) (at 50.8 65.6336 90))
     (property "Footprint" "Resistor_SMD:R_0603_1608Metric_Pad0.98x0.95mm_HandSolder" (id 2) (at 50.8 66.802 90)
@@
   (symbol (lib_id "MCU_Microchip_ATmega:ATmega328P-A") (at 73.66 91.44 0) (unit 1)
     (in_bom yes) (on_board yes)
-    (property "Reference" "U13" (id 0) (at 73.66 131.8006 0))
+    (property "Reference" "U10" (id 0) (at 73.66 131.8006 0))
     (property "Value" "ATmega328P-AU" (id 1) (at 73.66 134.112 0))
     (property "Footprint" "Package_QFP:TQFP-32_7x7mm_P0.8mm" (id 2) (at 73.66 91.44 0)
@@
   (symbol (lib_id "control20220206-rescue:R_POT-Device") (at 182.88 53.34 0) (unit 1)
     (in_bom yes) (on_board yes)
-    (property "Reference" "RV3" (id 0) (at 181.102 52.1716 0)
+    (property "Reference" "RV2" (id 0) (at 181.102 52.1716 0)
       (effects (font (size 1.27 1.27)) (justify right))
     )
@@
   (symbol (lib_id "Connector_Generic:Conn_01x06") (at 142.24 43.18 90) (unit 1)
     (in_bom yes) (on_board yes)
-    (property "Reference" "J32" (id 0) (at 152.0952 44.0944 90)
+    (property "Reference" "J27" (id 0) (at 152.0952 44.0944 90)
       (effects (font (size 1.27 1.27)) (justify right))
     )
@@
   (symbol (lib_id "Device:C") (at 44.45 107.95 0) (unit 1)
     (in_bom yes) (on_board yes)
-    (property "Reference" "C17" (id 0) (at 45.085 105.41 0)
+    (property "Reference" "C14" (id 0) (at 45.085 105.41 0)
       (effects (font (size 1.27 1.27)) (justify left))
     )
@@
   (symbol (lib_id "Device:R") (at 80.01 153.67 0) (unit 1)
     (in_bom yes) (on_board yes)
-    (property "Reference" "R52" (id 0) (at 82.042 153.67 90))
+    (property "Reference" "R46" (id 0) (at 82.042 153.67 90))
     (property "Value" "47k" (id 1) (at 80.01 153.67 90))
     (property "Footprint" "Resistor_SMD:R_0603_1608Metric_Pad0.98x0.95mm_HandSolder" (id 2) (at 78.232 153.67 90)
@@
   (symbol (lib_id "Switch:SW_Push") (at 153.67 123.19 0) (unit 1)
     (in_bom yes) (on_board yes) (fields_autoplaced)
-    (property "Reference" "SW8" (id 0) (at 153.67 116.5692 0))
+    (property "Reference" "SW7" (id 0) (at 153.67 116.5692 0))
     (property "Value" "RESET" (id 1) (at 153.67 119.1061 0))
     (property "Footprint" "0.main.robot:TVAF06-A020B-R" (id 2) (at 153.67 118.11 0)
@@
   (symbol (lib_id "Device:R") (at 107.95 139.7 0) (unit 1)
     (in_bom yes) (on_board yes)
-    (property "Reference" "R53" (id 0) (at 109.982 139.7 90))
+    (property "Reference" "R47" (id 0) (at 109.982 139.7 90))
     (property "Value" "470" (id 1) (at 107.95 139.7 90))
     (property "Footprint" "Resistor_SMD:R_0603_1608Metric_Pad0.98x0.95mm_HandSolder" (id 2) (at 106.172 139.7 90)
@@
   (symbol (lib_id "control20220206-rescue:R_POT-Device") (at 217.17 53.34 0) (unit 1)
     (in_bom yes) (on_board yes)
-    (property "Reference" "RV5" (id 0) (at 215.392 52.1716 0)
+    (property "Reference" "RV4" (id 0) (at 215.392 52.1716 0)
       (effects (font (size 1.27 1.27)) (justify right))
     )
@@
   (symbol (lib_id "Device:LED") (at 107.95 151.13 90) (unit 1)
     (in_bom yes) (on_board yes)
-    (property "Reference" "D20" (id 0) (at 105.41 151.13 0))
+    (property "Reference" "D17" (id 0) (at 105.41 151.13 0))
     (property "Value" "LED(OSWT1608)" (id 1) (at 110.49 151.13 0))
     (property "Footprint" "0.main.robot:LED_SMLE13WBC8W1" (id 2) (at 107.95 151.13 0)
@@
   (symbol (lib_id "power:GND") (at 44.45 143.51 0) (unit 1)
     (in_bom yes) (on_board yes)
-    (property "Reference" "#PWR050" (id 0) (at 44.45 149.86 0)
+    (property "Reference" "#PWR054" (id 0) (at 44.45 149.86 0)
       (effects (font (size 1.27 1.27)) hide)
     )
@@
   (symbol (lib_id "Connector_Generic:Conn_01x04") (at 43.18 162.56 0) (mirror y) (unit 1)
     (in_bom yes) (on_board yes)
-    (property "Reference" "J31" (id 0) (at 43.18 157.48 0))
+    (property "Reference" "J26" (id 0) (at 43.18 157.48 0))
     (property "Value" "I2C/OLED" (id 1) (at 43.18 170.18 0))
     (property "Footprint" "0.main.robot:JSTB4B-ZR" (id 2) (at 43.18 162.56 0)
@@
   (symbol (lib_id "Device:D") (at 165.1 110.49 0) (mirror y) (unit 1)
     (in_bom yes) (on_board yes)
-    (property "Reference" "D21" (id 0) (at 165.1 107.95 0))
+    (property "Reference" "D18" (id 0) (at 165.1 107.95 0))
     (property "Value" "RSX101VAM-30" (id 1) (at 165.1 113.03 0))
     (property "Footprint" "Diode_SMD:D_0805_2012Metric_Pad1.15x1.40mm_HandSolder" (id 2) (at 165.1 110.49 0)
@@
   (symbol (lib_id "Device:C") (at 35.56 107.95 0) (unit 1)
     (in_bom yes) (on_board yes)
-    (property "Reference" "C16" (id 0) (at 36.195 105.41 0)
+    (property "Reference" "C13" (id 0) (at 36.195 105.41 0)
       (effects (font (size 1.27 1.27)) (justify left))
     )
@@
   (symbol (lib_id "control20220206-rescue:R_POT-Device") (at 199.39 53.34 0) (unit 1)
     (in_bom yes) (on_board yes)
-    (property "Reference" "RV4" (id 0) (at 197.612 52.1716 0)
+    (property "Reference" "RV3" (id 0) (at 197.612 52.1716 0)
       (effects (font (size 1.27 1.27)) (justify right))
     )
@@
   (symbol (lib_id "power:GND") (at 149.86 50.8 0) (unit 1)
     (in_bom yes) (on_board yes)
-    (property "Reference" "#PWR055" (id 0) (at 149.86 57.15 0)
+    (property "Reference" "#PWR059" (id 0) (at 149.86 57.15 0)
       (effects (font (size 1.27 1.27)) hide)
     )
@@
   (symbol (lib_id "Device:D") (at 190.5 40.64 0) (unit 1)
     (in_bom yes) (on_board yes) (fields_autoplaced)
-    (property "Reference" "D22" (id 0) (at 190.5 35.6702 0))
+    (property "Reference" "D19" (id 0) (at 190.5 35.6702 0))
     (property "Value" "RSX101VAM-30" (id 1) (at 190.5 38.2071 0))
     (property "Footprint" "Diode_SMD:D_0805_2012Metric_Pad1.15x1.40mm_HandSolder" (id 2) (at 190.5 40.64 0)
@@
   (symbol (lib_id "Device:R") (at 165.1 105.41 90) (unit 1)
     (in_bom yes) (on_board yes)
-    (property "Reference" "R54" (id 0) (at 165.1 103.378 90))
+    (property "Reference" "R48" (id 0) (at 165.1 103.378 90))
     (property "Value" "10k" (id 1) (at 165.1 105.41 90))
     (property "Footprint" "Resistor_SMD:R_0603_1608Metric_Pad0.98x0.95mm_HandSolder" (id 2) (at 165.1 107.188 90)
@@
   (symbol (lib_id "power:GND") (at 147.32 125.73 0) (unit 1)
     (in_bom yes) (on_board yes)
-    (property "Reference" "#PWR054" (id 0) (at 147.32 132.08 0)
+    (property "Reference" "#PWR058" (id 0) (at 147.32 132.08 0)
       (effects (font (size 1.27 1.27)) hide)
     )
@@
   (symbol (lib_id "Device:C") (at 147.32 109.22 0) (unit 1)
     (in_bom yes) (on_board yes)
-    (property "Reference" "C18" (id 0) (at 147.955 106.68 0)
+    (property "Reference" "C15" (id 0) (at 147.955 106.68 0)
       (effects (font (size 1.27 1.27)) (justify left))
     )
@@
   (symbol (lib_id "control20220206-rescue:R_POT-Device") (at 233.68 53.34 0) (unit 1)
     (in_bom yes) (on_board yes)
-    (property "Reference" "RV6" (id 0) (at 231.902 52.1716 0)
+    (property "Reference" "RV5" (id 0) (at 231.902 52.1716 0)
       (effects (font (size 1.27 1.27)) (justify right))
     )
@@
   (symbol (lib_id "Device:R") (at 73.66 153.67 0) (unit 1)
     (in_bom yes) (on_board yes)
-    (property "Reference" "R51" (id 0) (at 75.692 153.67 90))
+    (property "Reference" "R45" (id 0) (at 75.692 153.67 90))
     (property "Value" "47k" (id 1) (at 73.66 153.67 90))
     (property "Footprint" "Resistor_SMD:R_0603_1608Metric_Pad0.98x0.95mm_HandSolder" (id 2) (at 71.882 153.67 90)
@@
   (symbol (lib_id "control20220206-rescue:R_POT-Device") (at 166.37 53.34 0) (unit 1)
     (in_bom yes) (on_board yes)
-    (property "Reference" "RV2" (id 0) (at 164.592 52.1716 0)
+    (property "Reference" "RV1" (id 0) (at 164.592 52.1716 0)
       (effects (font (size 1.27 1.27)) (justify right))
     )
@@
   (symbol (lib_id "power:GND") (at 107.95 158.75 0) (unit 1)
     (in_bom yes) (on_board yes)
-    (property "Reference" "#PWR052" (id 0) (at 107.95 165.1 0)
+    (property "Reference" "#PWR056" (id 0) (at 107.95 165.1 0)
       (effects (font (size 1.27 1.27)) hide)
     )
@@
   (symbol (lib_id "power:GND") (at 53.34 167.64 0) (unit 1)
     (in_bom yes) (on_board yes)
-    (property "Reference" "#PWR051" (id 0) (at 53.34 173.99 0)
+    (property "Reference" "#PWR055" (id 0) (at 53.34 173.99 0)
       (effects (font (size 1.27 1.27)) hide)
     )
@@
   (symbol (lib_id "Connector_Generic:Conn_01x06") (at 271.78 55.88 0) (mirror x) (unit 1)
     (in_bom yes) (on_board yes)
-    (property "Reference" "J33" (id 0) (at 269.6972 66.4718 0))
+    (property "Reference" "J28" (id 0) (at 269.6972 66.4718 0))
     (property "Value" "Trimmer" (id 1) (at 269.6972 64.1604 0))
     (property "Footprint" "0.main.robot:JSTS6B-ZRLFSN" (id 2) (at 271.78 55.88 0)

Commit message: fix: main xbee
Parts:
- renumbered C13 to C11, C14 to C12, C15 to C13, D17 to D14, D18 to D15, D19 to D16, J26 to J27, J27 to J28, J28 to J29, R44 to R37, R45 to R38, R46 to R39, R47 to R40, R48 to R41, SW7 to SW6, U10 to U8
Changed lines of the file:
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@@
   (symbol (lib_id "power:GND") (at 133.35 82.55 0) (unit 1)
     (in_bom yes) (on_board yes)
-    (property "Reference" "#PWR057" (id 0) (at 133.35 88.9 0)
+    (property "Reference" "#PWR056" (id 0) (at 133.35 88.9 0)
       (effects (font (size 1.27 1.27)) hide)
     )
@@
   (symbol (lib_id "Device:R") (at 50.8 68.58 270) (unit 1)
     (in_bom yes) (on_board yes)
-    (property "Reference" "R44" (id 0) (at 50.8 63.3222 90))
+    (property "Reference" "R37" (id 0) (at 50.8 63.3222 90))
     (property "Value" "47k" (id 1) (at 50.8 65.6336 90))
     (property "Footprint" "Resistor_SMD:R_0603_1608Metric_Pad0.98x0.95mm_HandSolder" (id 2) (at 50.8 66.802 90)
@@
   (symbol (lib_id "MCU_Microchip_ATmega:ATmega328P-A") (at 73.66 91.44 0) (unit 1)
     (in_bom yes) (on_board yes)
-    (property "Reference" "U10" (id 0) (at 73.66 131.8006 0))
+    (property "Reference" "U8" (id 0) (at 73.66 131.8006 0))
     (property "Value" "ATmega328P-AU" (id 1) (at 73.66 134.112 0))
     (property "Footprint" "Package_QFP:TQFP-32_7x7mm_P0.8mm" (id 2) (at 73.66 91.44 0)
@@
   (symbol (lib_id "Connector_Generic:Conn_01x06") (at 142.24 43.18 90) (unit 1)
     (in_bom yes) (on_board yes)
-    (property "Reference" "J27" (id 0) (at 152.0952 44.0944 90)
+    (property "Reference" "J28" (id 0) (at 152.0952 44.0944 90)
       (effects (font (size 1.27 1.27)) (justify right))
     )
@@
   (symbol (lib_id "Device:C") (at 44.45 107.95 0) (unit 1)
     (in_bom yes) (on_board yes)
-    (property "Reference" "C14" (id 0) (at 45.085 105.41 0)
+    (property "Reference" "C12" (id 0) (at 45.085 105.41 0)
       (effects (font (size 1.27 1.27)) (justify left))
     )
@@
   (symbol (lib_id "Device:R") (at 80.01 153.67 0) (unit 1)
     (in_bom yes) (on_board yes)
-    (property "Reference" "R46" (id 0) (at 82.042 153.67 90))
+    (property "Reference" "R39" (id 0) (at 82.042 153.67 90))
     (property "Value" "47k" (id 1) (at 80.01 153.67 90))
     (property "Footprint" "Resistor_SMD:R_0603_1608Metric_Pad0.98x0.95mm_HandSolder" (id 2) (at 78.232 153.67 90)
@@
   (symbol (lib_id "Switch:SW_Push") (at 153.67 123.19 0) (unit 1)
     (in_bom yes) (on_board yes) (fields_autoplaced)
-    (property "Reference" "SW7" (id 0) (at 153.67 116.5692 0))
+    (property "Reference" "SW6" (id 0) (at 153.67 116.5692 0))
     (property "Value" "RESET" (id 1) (at 153.67 119.1061 0))
     (property "Footprint" "0.main.robot:TVAF06-A020B-R" (id 2) (at 153.67 118.11 0)
@@
   (symbol (lib_id "Device:R") (at 107.95 139.7 0) (unit 1)
     (in_bom yes) (on_board yes)
-    (property "Reference" "R47" (id 0) (at 109.982 139.7 90))
+    (property "Reference" "R40" (id 0) (at 109.982 139.7 90))
     (property "Value" "470" (id 1) (at 107.95 139.7 90))
     (property "Footprint" "Resistor_SMD:R_0603_1608Metric_Pad0.98x0.95mm_HandSolder" (id 2) (at 106.172 139.7 90)
@@
   (symbol (lib_id "Device:LED") (at 107.95 151.13 90) (unit 1)
     (in_bom yes) (on_board yes)
-    (property "Reference" "D17" (id 0) (at 105.41 151.13 0))
+    (property "Reference" "D14" (id 0) (at 105.41 151.13 0))
     (property "Value" "LED(OSWT1608)" (id 1) (at 110.49 151.13 0))
     (property "Footprint" "0.main.robot:LED_SMLE13WBC8W1" (id 2) (at 107.95 151.13 0)
@@
   (symbol (lib_id "power:GND") (at 44.45 143.51 0) (unit 1)
     (in_bom yes) (on_board yes)
-    (property "Reference" "#PWR054" (id 0) (at 44.45 149.86 0)
+    (property "Reference" "#PWR053" (id 0) (at 44.45 149.86 0)
       (effects (font (size 1.27 1.27)) hide)
     )
@@
   (symbol (lib_id "Connector_Generic:Conn_01x04") (at 43.18 162.56 0) (mirror y) (unit 1)
     (in_bom yes) (on_board yes)
-    (property "Reference" "J26" (id 0) (at 43.18 157.48 0))
+    (property "Reference" "J27" (id 0) (at 43.18 157.48 0))
     (property "Value" "I2C/OLED" (id 1) (at 43.18 170.18 0))
     (property "Footprint" "0.main.robot:JSTB4B-ZR" (id 2) (at 43.18 162.56 0)
@@
   (symbol (lib_id "Device:D") (at 165.1 110.49 0) (mirror y) (unit 1)
     (in_bom yes) (on_board yes)
-    (property "Reference" "D18" (id 0) (at 165.1 107.95 0))
+    (property "Reference" "D15" (id 0) (at 165.1 107.95 0))
     (property "Value" "RSX101VAM-30" (id 1) (at 165.1 113.03 0))
     (property "Footprint" "Diode_SMD:D_0805_2012Metric_Pad1.15x1.40mm_HandSolder" (id 2) (at 165.1 110.49 0)
@@
   (symbol (lib_id "Device:C") (at 35.56 107.95 0) (unit 1)
     (in_bom yes) (on_board yes)
-    (property "Reference" "C13" (id 0) (at 36.195 105.41 0)
+    (property "Reference" "C11" (id 0) (at 36.195 105.41 0)
       (effects (font (size 1.27 1.27)) (justify left))
     )
@@
   (symbol (lib_id "power:GND") (at 149.86 50.8 0) (unit 1)
     (in_bom yes) (on_board yes)
-    (property "Reference" "#PWR059" (id 0) (at 149.86 57.15 0)
+    (property "Reference" "#PWR058" (id 0) (at 149.86 57.15 0)
       (effects (font (size 1.27 1.27)) hide)
     )
@@
   (symbol (lib_id "Device:D") (at 190.5 40.64 0) (unit 1)
     (in_bom yes) (on_board yes) (fields_autoplaced)
-    (property "Reference" "D19" (id 0) (at 190.5 35.6702 0))
+    (property "Reference" "D16" (id 0) (at 190.5 35.6702 0))
     (property "Value" "RSX101VAM-30" (id 1) (at 190.5 38.2071 0))
     (property "Footprint" "Diode_SMD:D_0805_2012Metric_Pad1.15x1.40mm_HandSolder" (id 2) (at 190.5 40.64 0)
@@
   (symbol (lib_id "Device:R") (at 165.1 105.41 90) (unit 1)
     (in_bom yes) (on_board yes)
-    (property "Reference" "R48" (id 0) (at 165.1 103.378 90))
+    (property "Reference" "R41" (id 0) (at 165.1 103.378 90))
     (property "Value" "10k" (id 1) (at 165.1 105.41 90))
     (property "Footprint" "Resistor_SMD:R_0603_1608Metric_Pad0.98x0.95mm_HandSolder" (id 2) (at 165.1 107.188 90)
@@
   (symbol (lib_id "power:GND") (at 147.32 125.73 0) (unit 1)
     (in_bom yes) (on_board yes)
-    (property "Reference" "#PWR058" (id 0) (at 147.32 132.08 0)
+    (property "Reference" "#PWR057" (id 0) (at 147.32 132.08 0)
       (effects (font (size 1.27 1.27)) hide)
     )
@@
   (symbol (lib_id "Device:C") (at 147.32 109.22 0) (unit 1)
     (in_bom yes) (on_board yes)
-    (property "Reference" "C15" (id 0) (at 147.955 106.68 0)
+    (property "Reference" "C13" (id 0) (at 147.955 106.68 0)
       (effects (font (size 1.27 1.27)) (justify left))
     )
@@
   (symbol (lib_id "Device:R") (at 73.66 153.67 0) (unit 1)
     (in_bom yes) (on_board yes)
-    (property "Reference" "R45" (id 0) (at 75.692 153.67 90))
+    (property "Reference" "R38" (id 0) (at 75.692 153.67 90))
     (property "Value" "47k" (id 1) (at 73.66 153.67 90))
     (property "Footprint" "Resistor_SMD:R_0603_1608Metric_Pad0.98x0.95mm_HandSolder" (id 2) (at 71.882 153.67 90)
@@
   (symbol (lib_id "power:GND") (at 107.95 158.75 0) (unit 1)
     (in_bom yes) (on_board yes)
-    (property "Reference" "#PWR056" (id 0) (at 107.95 165.1 0)
+    (property "Reference" "#PWR055" (id 0) (at 107.95 165.1 0)
       (effects (font (size 1.27 1.27)) hide)
     )
@@
   (symbol (lib_id "power:GND") (at 53.34 167.64 0) (unit 1)
     (in_bom yes) (on_board yes)
-    (property "Reference" "#PWR055" (id 0) (at 53.34 173.99 0)
+    (property "Reference" "#PWR054" (id 0) (at 53.34 173.99 0)
       (effects (font (size 1.27 1.27)) hide)
     )
@@
   (symbol (lib_id "Connector_Generic:Conn_01x06") (at 271.78 55.88 0) (mirror x) (unit 1)
     (in_bom yes) (on_board yes)
-    (property "Reference" "J28" (id 0) (at 269.6972 66.4718 0))
+    (property "Reference" "J29" (id 0) (at 269.6972 66.4718 0))
     (property "Value" "Trimmer" (id 1) (at 269.6972 64.1604 0))
     (property "Footprint" "0.main.robot:JSTS6B-ZRLFSN" (id 2) (at 271.78 55.88 0)

Commit message: ToF
Parts:
- renumbered J27 to J25, J28 to J26, J29 to J27
Changed lines of the file:
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@@
   (symbol (lib_id "power:GND") (at 133.35 82.55 0) (unit 1)
     (in_bom yes) (on_board yes)
-    (property "Reference" "#PWR056" (id 0) (at 133.35 88.9 0)
+    (property "Reference" "#PWR058" (id 0) (at 133.35 88.9 0)
       (effects (font (size 1.27 1.27)) hide)
     )
@@
   (symbol (lib_id "Connector_Generic:Conn_01x06") (at 142.24 43.18 90) (unit 1)
     (in_bom yes) (on_board yes)
-    (property "Reference" "J28" (id 0) (at 152.0952 44.0944 90)
+    (property "Reference" "J26" (id 0) (at 152.0952 44.0944 90)
       (effects (font (size 1.27 1.27)) (justify right))
     )
@@
   (symbol (lib_id "power:GND") (at 44.45 143.51 0) (unit 1)
     (in_bom yes) (on_board yes)
-    (property "Reference" "#PWR053" (id 0) (at 44.45 149.86 0)
+    (property "Reference" "#PWR055" (id 0) (at 44.45 149.86 0)
       (effects (font (size 1.27 1.27)) hide)
     )
@@
   (symbol (lib_id "Connector_Generic:Conn_01x04") (at 43.18 162.56 0) (mirror y) (unit 1)
     (in_bom yes) (on_board yes)
-    (property "Reference" "J27" (id 0) (at 43.18 157.48 0))
+    (property "Reference" "J25" (id 0) (at 43.18 157.48 0))
     (property "Value" "I2C/OLED" (id 1) (at 43.18 170.18 0))
     (property "Footprint" "0.main.robot:JSTB4B-ZR" (id 2) (at 43.18 162.56 0)
@@
   (symbol (lib_id "power:GND") (at 149.86 50.8 0) (unit 1)
     (in_bom yes) (on_board yes)
-    (property "Reference" "#PWR058" (id 0) (at 149.86 57.15 0)
+    (property "Reference" "#PWR060" (id 0) (at 149.86 57.15 0)
       (effects (font (size 1.27 1.27)) hide)
     )
@@
   (symbol (lib_id "power:GND") (at 147.32 125.73 0) (unit 1)
     (in_bom yes) (on_board yes)
-    (property "Reference" "#PWR057" (id 0) (at 147.32 132.08 0)
+    (property "Reference" "#PWR059" (id 0) (at 147.32 132.08 0)
       (effects (font (size 1.27 1.27)) hide)
     )
@@
   (symbol (lib_id "power:GND") (at 107.95 158.75 0) (unit 1)
     (in_bom yes) (on_board yes)
-    (property "Reference" "#PWR055" (id 0) (at 107.95 165.1 0)
+    (property "Reference" "#PWR057" (id 0) (at 107.95 165.1 0)
       (effects (font (size 1.27 1.27)) hide)
     )
@@
   (symbol (lib_id "power:GND") (at 53.34 167.64 0) (unit 1)
     (in_bom yes) (on_board yes)
-    (property "Reference" "#PWR054" (id 0) (at 53.34 173.99 0)
+    (property "Reference" "#PWR056" (id 0) (at 53.34 173.99 0)
       (effects (font (size 1.27 1.27)) hide)
     )
@@
   (symbol (lib_id "Connector_Generic:Conn_01x06") (at 271.78 55.88 0) (mirror x) (unit 1)
     (in_bom yes) (on_board yes)
-    (property "Reference" "J29" (id 0) (at 269.6972 66.4718 0))
+    (property "Reference" "J27" (id 0) (at 269.6972 66.4718 0))
     (property "Value" "Trimmer" (id 1) (at 269.6972 64.1604 0))
     (property "Footprint" "0.main.robot:JSTS6B-ZRLFSN" (id 2) (at 271.78 55.88 0)

Commit message: no message
Parts:
- removed J26: ICSP, 0.main.robot:JSTB6B-ZR, symbol Connector_Generic:Conn_01x06
- added D10: RSX101VAM-30, Diode_SMD:D_0805_2012Metric_Pad1.15x1.40mm_HandSolder, symbol Device:D
- added J23: ICSP, 0.main.robot:JSTB6B-ZR, symbol Connector_Generic:Conn_01x06
- J24: renamed from J27; footprint 0.main.robot:JSTS6B-ZRLFSN -> 0.main.robot:JSTB6B-ZR
- renumbered C12 to C10, C13 to C11, C11 to C9, D15 to D11, D16 to D12, D14 to D9, J25 to J22, R37 to R25, R38 to R26, R39 to R27, R40 to R28, R41 to R29, SW6 to SW2, U8 to U6
Connections:
- net GND: now also J23.6 (Pin_6)
- net RESET: now also D10.1 (K); no longer C11.1, D11.2 (A), R29.1, SW2.2, U6.29 (~{RESET}/PC6)
- net Vcc1: now also J23.2 (Pin_2)
- net at U6.15 (PB3): now also J23.4 (Pin_4)
- net at U6.16 (PB4): now also J23.1 (Pin_1)
- net at U6.17 (PB5): now also J23.3 (Pin_3)
- new net: C11.1, D10.2 (A), D11.2 (A), J23.5 (Pin_5), R29.1, SW2.2, U6.29 (~{RESET}/PC6)
