File: kicad/main/LineTrimmer.kicad_sch (KiCad schematic)
At the start: 23 parts, among them J22 I2C/OLED, J23 ICSP, J24 Trimmer, SW2 RESET, U6 ATmega328P-AU, Y2 8Mhz

Commit message: no message
Parts:
- renumbered D9 to D11, D10 to D12, D11 to D13, D12 to D14, J22 to J21, J23 to J22, J24 to J23, R25 to R27, R26 to R28, R27 to R29, R28 to R30, R29 to R31, SW2 to SW4, U6 to U7
Changed lines of the file:
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@@
   (symbol (lib_id "power:GND") (at 133.35 82.55 0) (unit 1)
     (in_bom yes) (on_board yes)
-    (property "Reference" "#PWR050" (id 0) (at 133.35 88.9 0)
+    (property "Reference" "#PWR062" (id 0) (at 133.35 88.9 0)
       (effects (font (size 1.27 1.27)) hide)
     )
@@
   (symbol (lib_id "power:GND") (at 149.86 50.8 0) (unit 1)
     (in_bom yes) (on_board yes)
-    (property "Reference" "#PWR052" (id 0) (at 149.86 57.15 0)
+    (property "Reference" "#PWR064" (id 0) (at 149.86 57.15 0)
       (effects (font (size 1.27 1.27)) hide)
     )
@@
   (symbol (lib_id "Device:R") (at 50.8 68.58 270) (unit 1)
     (in_bom yes) (on_board yes)
-    (property "Reference" "R25" (id 0) (at 50.8 63.3222 90))
+    (property "Reference" "R27" (id 0) (at 50.8 63.3222 90))
     (property "Value" "47k" (id 1) (at 50.8 65.6336 90))
     (property "Footprint" "Resistor_SMD:R_0603_1608Metric_Pad0.98x0.95mm_HandSolder" (id 2) (at 50.8 66.802 90)
@@
   (symbol (lib_id "MCU_Microchip_ATmega:ATmega328P-A") (at 73.66 91.44 0) (unit 1)
     (in_bom yes) (on_board yes)
-    (property "Reference" "U6" (id 0) (at 73.66 131.8006 0))
+    (property "Reference" "U7" (id 0) (at 73.66 131.8006 0))
     (property "Value" "ATmega328P-AU" (id 1) (at 73.66 134.112 0))
     (property "Footprint" "Package_QFP:TQFP-32_7x7mm_P0.8mm" (id 2) (at 73.66 91.44 0)
@@
   (symbol (lib_id "Device:R") (at 80.01 153.67 0) (unit 1)
     (in_bom yes) (on_board yes)
-    (property "Reference" "R27" (id 0) (at 82.042 153.67 90))
+    (property "Reference" "R29" (id 0) (at 82.042 153.67 90))
     (property "Value" "47k" (id 1) (at 80.01 153.67 90))
     (property "Footprint" "Resistor_SMD:R_0603_1608Metric_Pad0.98x0.95mm_HandSolder" (id 2) (at 78.232 153.67 90)
@@
   (symbol (lib_id "Switch:SW_Push") (at 153.67 123.19 0) (unit 1)
     (in_bom yes) (on_board yes) (fields_autoplaced)
-    (property "Reference" "SW2" (id 0) (at 153.67 116.5692 0))
+    (property "Reference" "SW4" (id 0) (at 153.67 116.5692 0))
     (property "Value" "RESET" (id 1) (at 153.67 119.1061 0))
     (property "Footprint" "0.main.robot:TVAF06-A020B-R" (id 2) (at 153.67 118.11 0)
@@
   (symbol (lib_id "Device:R") (at 107.95 139.7 0) (unit 1)
     (in_bom yes) (on_board yes)
-    (property "Reference" "R28" (id 0) (at 109.982 139.7 90))
+    (property "Reference" "R30" (id 0) (at 109.982 139.7 90))
     (property "Value" "470" (id 1) (at 107.95 139.7 90))
     (property "Footprint" "Resistor_SMD:R_0603_1608Metric_Pad0.98x0.95mm_HandSolder" (id 2) (at 106.172 139.7 90)
@@
   (symbol (lib_id "Device:LED") (at 107.95 151.13 90) (unit 1)
     (in_bom yes) (on_board yes)
-    (property "Reference" "D9" (id 0) (at 105.41 151.13 0))
+    (property "Reference" "D11" (id 0) (at 105.41 151.13 0))
     (property "Value" "LED(OSWT1608)" (id 1) (at 110.49 151.13 0))
     (property "Footprint" "0.main.robot:LED_SMLE13WBC8W1" (id 2) (at 107.95 151.13 0)
@@
   (symbol (lib_id "Device:D") (at 140.97 105.41 0) (unit 1)
     (in_bom yes) (on_board yes) (fields_autoplaced)
-    (property "Reference" "D10" (id 0) (at 140.97 100.4402 0))
+    (property "Reference" "D12" (id 0) (at 140.97 100.4402 0))
     (property "Value" "RSX101VAM-30" (id 1) (at 140.97 102.9771 0))
     (property "Footprint" "Diode_SMD:D_0805_2012Metric_Pad1.15x1.40mm_HandSolder" (id 2) (at 140.97 105.41 0)
@@
   (symbol (lib_id "power:GND") (at 44.45 143.51 0) (unit 1)
     (in_bom yes) (on_board yes)
-    (property "Reference" "#PWR047" (id 0) (at 44.45 149.86 0)
+    (property "Reference" "#PWR059" (id 0) (at 44.45 149.86 0)
       (effects (font (size 1.27 1.27)) hide)
     )
@@
   (symbol (lib_id "Connector_Generic:Conn_01x04") (at 43.18 162.56 0) (mirror y) (unit 1)
     (in_bom yes) (on_board yes)
-    (property "Reference" "J22" (id 0) (at 43.18 157.48 0))
+    (property "Reference" "J21" (id 0) (at 43.18 157.48 0))
     (property "Value" "I2C/OLED" (id 1) (at 43.18 170.18 0))
     (property "Footprint" "0.main.robot:JSTB4B-ZR" (id 2) (at 43.18 162.56 0)
@@
   (symbol (lib_id "Device:D") (at 165.1 110.49 0) (mirror y) (unit 1)
     (in_bom yes) (on_board yes)
-    (property "Reference" "D11" (id 0) (at 165.1 107.95 0))
+    (property "Reference" "D13" (id 0) (at 165.1 107.95 0))
     (property "Value" "RSX101VAM-30" (id 1) (at 165.1 113.03 0))
     (property "Footprint" "Diode_SMD:D_0805_2012Metric_Pad1.15x1.40mm_HandSolder" (id 2) (at 165.1 110.49 0)
@@
   (symbol (lib_id "power:GND") (at 149.86 50.8 0) (unit 1)
     (in_bom yes) (on_board yes)
-    (property "Reference" "#PWR053" (id 0) (at 149.86 57.15 0)
+    (property "Reference" "#PWR065" (id 0) (at 149.86 57.15 0)
       (effects (font (size 1.27 1.27)) hide)
     )
@@
   (symbol (lib_id "Device:D") (at 190.5 40.64 0) (unit 1)
     (in_bom yes) (on_board yes) (fields_autoplaced)
-    (property "Reference" "D12" (id 0) (at 190.5 35.6702 0))
+    (property "Reference" "D14" (id 0) (at 190.5 35.6702 0))
     (property "Value" "RSX101VAM-30" (id 1) (at 190.5 38.2071 0))
     (property "Footprint" "Diode_SMD:D_0805_2012Metric_Pad1.15x1.40mm_HandSolder" (id 2) (at 190.5 40.64 0)
@@
   (symbol (lib_id "Device:R") (at 165.1 105.41 90) (unit 1)
     (in_bom yes) (on_board yes)
-    (property "Reference" "R29" (id 0) (at 165.1 103.378 90))
+    (property "Reference" "R31" (id 0) (at 165.1 103.378 90))
     (property "Value" "10k" (id 1) (at 165.1 105.41 90))
     (property "Footprint" "Resistor_SMD:R_0603_1608Metric_Pad0.98x0.95mm_HandSolder" (id 2) (at 165.1 107.188 90)
@@
   (symbol (lib_id "power:GND") (at 147.32 125.73 0) (unit 1)
     (in_bom yes) (on_board yes)
-    (property "Reference" "#PWR051" (id 0) (at 147.32 132.08 0)
+    (property "Reference" "#PWR063" (id 0) (at 147.32 132.08 0)
       (effects (font (size 1.27 1.27)) hide)
     )
@@
   (symbol (lib_id "Connector_Generic:Conn_01x06") (at 142.24 43.18 90) (unit 1)
     (in_bom yes) (on_board yes)
-    (property "Reference" "J23" (id 0) (at 152.0952 44.0944 90)
+    (property "Reference" "J22" (id 0) (at 152.0952 44.0944 90)
       (effects (font (size 1.27 1.27)) (justify right))
     )
@@
   (symbol (lib_id "Device:R") (at 73.66 153.67 0) (unit 1)
     (in_bom yes) (on_board yes)
-    (property "Reference" "R26" (id 0) (at 75.692 153.67 90))
+    (property "Reference" "R28" (id 0) (at 75.692 153.67 90))
     (property "Value" "47k" (id 1) (at 73.66 153.67 90))
     (property "Footprint" "Resistor_SMD:R_0603_1608Metric_Pad0.98x0.95mm_HandSolder" (id 2) (at 71.882 153.67 90)
@@
   (symbol (lib_id "power:GND") (at 107.95 158.75 0) (unit 1)
     (in_bom yes) (on_board yes)
-    (property "Reference" "#PWR049" (id 0) (at 107.95 165.1 0)
+    (property "Reference" "#PWR061" (id 0) (at 107.95 165.1 0)
       (effects (font (size 1.27 1.27)) hide)
     )
@@
   (symbol (lib_id "power:GND") (at 53.34 167.64 0) (unit 1)
     (in_bom yes) (on_board yes)
-    (property "Reference" "#PWR048" (id 0) (at 53.34 173.99 0)
+    (property "Reference" "#PWR060" (id 0) (at 53.34 173.99 0)
       (effects (font (size 1.27 1.27)) hide)
     )
@@
   (symbol (lib_id "Connector_Generic:Conn_01x06") (at 271.78 55.88 0) (mirror x) (unit 1)
     (in_bom yes) (on_board yes)
-    (property "Reference" "J24" (id 0) (at 269.6972 66.4718 0))
+    (property "Reference" "J23" (id 0) (at 269.6972 66.4718 0))
     (property "Value" "Trimmer" (id 1) (at 269.6972 64.1604 0))
     (property "Footprint" "0.main.robot:JSTB6B-ZR" (id 2) (at 271.78 55.88 0)

Commit message: bus
Parts:
- removed D12: RSX101VAM-30, Diode_SMD:D_0805_2012Metric_Pad1.15x1.40mm_HandSolder, symbol Device:D
Changed lines of the file:
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@@
-    (stroke (width 0) (type default) (color 0 0 0 0))
-  )
-  (wire (pts (xy 129.54 105.41) (xy 137.16 105.41))
     (stroke (width 0) (type default) (color 0 0 0 0))
   )
@@
   )
   (wire (pts (xy 35.56 52.07) (xy 44.45 52.07))
-    (stroke (width 0) (type default) (color 0 0 0 0))
-  )
-  (wire (pts (xy 144.78 105.41) (xy 147.32 105.41))
     (stroke (width 0) (type default) (color 0 0 0 0))
   )
@@
   (label "SDA" (at 85.09 165.1 0)
     (effects (font (size 1.524 1.524)) (justify left bottom))
-  )
-  (global_label "RESET" (shape input) (at 129.54 105.41 180) (fields_autoplaced)
-    (effects (font (size 1.27 1.27)) (justify right))
-    (property "Intersheet References" "${INTERSHEET_REFS}" (id 0) (at 121.4706 105.3306 0)
-      (effects (font (size 1.27 1.27)) (justify right) hide)
-    )
   )
   (global_label "Vcc1" (shape input) (at 76.2 46.99 90) (fields_autoplaced)
@@
       (effects (font (size 1.27 1.27)) hide)
     )
-    (pin "1")
-    (pin "2")
-  )
-  (symbol (lib_id "Device:D") (at 140.97 105.41 0) (unit 1)
-    (in_bom yes) (on_board yes) (fields_autoplaced)
-    (property "Reference" "D12" (id 0) (at 140.97 100.4402 0))
-    (property "Value" "RSX101VAM-30" (id 1) (at 140.97 102.9771 0))
-    (property "Footprint" "Diode_SMD:D_0805_2012Metric_Pad1.15x1.40mm_HandSolder" (id 2) (at 140.97 105.41 0)
-      (effects (font (size 1.27 1.27)) hide)
-    )
-    (property "Datasheet" "~" (id 3) (at 140.97 105.41 0)
-      (effects (font (size 1.27 1.27)) hide)
-    )

Commit message: update
Parts:
- renumbered C9 to C7, C10 to C8, C11 to C9, D11 to D10, D13 to D11, D14 to D12, J21 to J20, J22 to J21, J23 to J22, R27 to R26, R28 to R27, R29 to R28, R30 to R29, R31 to R30, SW4 to SW5, U7 to U6
Changed lines of the file:
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@@
   (symbol (lib_id "power:GND") (at 133.35 82.55 0) (unit 1)
     (in_bom yes) (on_board yes)
-    (property "Reference" "#PWR062" (id 0) (at 133.35 88.9 0)
+    (property "Reference" "#PWR058" (id 0) (at 133.35 88.9 0)
       (effects (font (size 1.27 1.27)) hide)
     )
@@
   (symbol (lib_id "power:GND") (at 149.86 50.8 0) (unit 1)
     (in_bom yes) (on_board yes)
-    (property "Reference" "#PWR064" (id 0) (at 149.86 57.15 0)
+    (property "Reference" "#PWR060" (id 0) (at 149.86 57.15 0)
       (effects (font (size 1.27 1.27)) hide)
     )
@@
   (symbol (lib_id "Device:R") (at 50.8 68.58 270) (unit 1)
     (in_bom yes) (on_board yes)
-    (property "Reference" "R27" (id 0) (at 50.8 63.3222 90))
+    (property "Reference" "R26" (id 0) (at 50.8 63.3222 90))
     (property "Value" "47k" (id 1) (at 50.8 65.6336 90))
     (property "Footprint" "Resistor_SMD:R_0603_1608Metric_Pad0.98x0.95mm_HandSolder" (id 2) (at 50.8 66.802 90)
@@
   (symbol (lib_id "MCU_Microchip_ATmega:ATmega328P-A") (at 73.66 91.44 0) (unit 1)
     (in_bom yes) (on_board yes)
-    (property "Reference" "U7" (id 0) (at 73.66 131.8006 0))
+    (property "Reference" "U6" (id 0) (at 73.66 131.8006 0))
     (property "Value" "ATmega328P-AU" (id 1) (at 73.66 134.112 0))
     (property "Footprint" "Package_QFP:TQFP-32_7x7mm_P0.8mm" (id 2) (at 73.66 91.44 0)
@@
   (symbol (lib_id "Device:C") (at 44.45 107.95 0) (unit 1)
     (in_bom yes) (on_board yes)
-    (property "Reference" "C10" (id 0) (at 45.085 105.41 0)
+    (property "Reference" "C8" (id 0) (at 45.085 105.41 0)
       (effects (font (size 1.27 1.27)) (justify left))
     )
@@
   (symbol (lib_id "Device:R") (at 80.01 153.67 0) (unit 1)
     (in_bom yes) (on_board yes)
-    (property "Reference" "R29" (id 0) (at 82.042 153.67 90))
+    (property "Reference" "R28" (id 0) (at 82.042 153.67 90))
     (property "Value" "47k" (id 1) (at 80.01 153.67 90))
     (property "Footprint" "Resistor_SMD:R_0603_1608Metric_Pad0.98x0.95mm_HandSolder" (id 2) (at 78.232 153.67 90)
@@
   (symbol (lib_id "Switch:SW_Push") (at 153.67 123.19 0) (unit 1)
     (in_bom yes) (on_board yes) (fields_autoplaced)
-    (property "Reference" "SW4" (id 0) (at 153.67 116.5692 0))
+    (property "Reference" "SW5" (id 0) (at 153.67 116.5692 0))
     (property "Value" "RESET" (id 1) (at 153.67 119.1061 0))
     (property "Footprint" "0.main.robot:TVAF06-A020B-R" (id 2) (at 153.67 118.11 0)
@@
   (symbol (lib_id "Device:R") (at 107.95 139.7 0) (unit 1)
     (in_bom yes) (on_board yes)
-    (property "Reference" "R30" (id 0) (at 109.982 139.7 90))
+    (property "Reference" "R29" (id 0) (at 109.982 139.7 90))
     (property "Value" "470" (id 1) (at 107.95 139.7 90))
     (property "Footprint" "Resistor_SMD:R_0603_1608Metric_Pad0.98x0.95mm_HandSolder" (id 2) (at 106.172 139.7 90)
@@
   (symbol (lib_id "Device:LED") (at 107.95 151.13 90) (unit 1)
     (in_bom yes) (on_board yes)
-    (property "Reference" "D11" (id 0) (at 105.41 151.13 0))
+    (property "Reference" "D10" (id 0) (at 105.41 151.13 0))
     (property "Value" "LED(OSWT1608)" (id 1) (at 110.49 151.13 0))
     (property "Footprint" "0.main.robot:LED_SMLE13WBC8W1" (id 2) (at 107.95 151.13 0)
@@
   (symbol (lib_id "power:GND") (at 44.45 143.51 0) (unit 1)
     (in_bom yes) (on_board yes)
-    (property "Reference" "#PWR059" (id 0) (at 44.45 149.86 0)
+    (property "Reference" "#PWR055" (id 0) (at 44.45 149.86 0)
       (effects (font (size 1.27 1.27)) hide)
     )
@@
   (symbol (lib_id "Connector_Generic:Conn_01x04") (at 43.18 162.56 0) (mirror y) (unit 1)
     (in_bom yes) (on_board yes)
-    (property "Reference" "J21" (id 0) (at 43.18 157.48 0))
+    (property "Reference" "J20" (id 0) (at 43.18 157.48 0))
     (property "Value" "I2C/OLED" (id 1) (at 43.18 170.18 0))
     (property "Footprint" "0.main.robot:JSTB4B-ZR" (id 2) (at 43.18 162.56 0)
@@
   (symbol (lib_id "Device:D") (at 165.1 110.49 0) (mirror y) (unit 1)
     (in_bom yes) (on_board yes)
-    (property "Reference" "D13" (id 0) (at 165.1 107.95 0))
+    (property "Reference" "D11" (id 0) (at 165.1 107.95 0))
     (property "Value" "RSX101VAM-30" (id 1) (at 165.1 113.03 0))
     (property "Footprint" "Diode_SMD:D_0805_2012Metric_Pad1.15x1.40mm_HandSolder" (id 2) (at 165.1 110.49 0)
@@
   (symbol (lib_id "Device:C") (at 35.56 107.95 0) (unit 1)
     (in_bom yes) (on_board yes)
-    (property "Reference" "C9" (id 0) (at 36.195 105.41 0)
+    (property "Reference" "C7" (id 0) (at 36.195 105.41 0)
       (effects (font (size 1.27 1.27)) (justify left))
     )
@@
   (symbol (lib_id "power:GND") (at 149.86 50.8 0) (unit 1)
     (in_bom yes) (on_board yes)
-    (property "Reference" "#PWR065" (id 0) (at 149.86 57.15 0)
+    (property "Reference" "#PWR061" (id 0) (at 149.86 57.15 0)
       (effects (font (size 1.27 1.27)) hide)
     )
@@
   (symbol (lib_id "Device:D") (at 190.5 40.64 0) (unit 1)
     (in_bom yes) (on_board yes) (fields_autoplaced)
-    (property "Reference" "D14" (id 0) (at 190.5 35.6702 0))
+    (property "Reference" "D12" (id 0) (at 190.5 35.6702 0))
     (property "Value" "RSX101VAM-30" (id 1) (at 190.5 38.2071 0))
     (property "Footprint" "Diode_SMD:D_0805_2012Metric_Pad1.15x1.40mm_HandSolder" (id 2) (at 190.5 40.64 0)
@@
   (symbol (lib_id "Device:R") (at 165.1 105.41 90) (unit 1)
     (in_bom yes) (on_board yes)
-    (property "Reference" "R31" (id 0) (at 165.1 103.378 90))
+    (property "Reference" "R30" (id 0) (at 165.1 103.378 90))
     (property "Value" "10k" (id 1) (at 165.1 105.41 90))
     (property "Footprint" "Resistor_SMD:R_0603_1608Metric_Pad0.98x0.95mm_HandSolder" (id 2) (at 165.1 107.188 90)
@@
   (symbol (lib_id "power:GND") (at 147.32 125.73 0) (unit 1)
     (in_bom yes) (on_board yes)
-    (property "Reference" "#PWR063" (id 0) (at 147.32 132.08 0)
+    (property "Reference" "#PWR059" (id 0) (at 147.32 132.08 0)
       (effects (font (size 1.27 1.27)) hide)
     )
@@
   (symbol (lib_id "Connector_Generic:Conn_01x06") (at 142.24 43.18 90) (unit 1)
     (in_bom yes) (on_board yes)
-    (property "Reference" "J22" (id 0) (at 152.0952 44.0944 90)
+    (property "Reference" "J21" (id 0) (at 152.0952 44.0944 90)
       (effects (font (size 1.27 1.27)) (justify right))
     )
@@
   (symbol (lib_id "Device:C") (at 147.32 109.22 0) (unit 1)
     (in_bom yes) (on_board yes)
-    (property "Reference" "C11" (id 0) (at 147.955 106.68 0)
+    (property "Reference" "C9" (id 0) (at 147.955 106.68 0)
       (effects (font (size 1.27 1.27)) (justify left))
     )
@@
   (symbol (lib_id "Device:R") (at 73.66 153.67 0) (unit 1)
     (in_bom yes) (on_board yes)
-    (property "Reference" "R28" (id 0) (at 75.692 153.67 90))
+    (property "Reference" "R27" (id 0) (at 75.692 153.67 90))
     (property "Value" "47k" (id 1) (at 73.66 153.67 90))
     (property "Footprint" "Resistor_SMD:R_0603_1608Metric_Pad0.98x0.95mm_HandSolder" (id 2) (at 71.882 153.67 90)
@@
   (symbol (lib_id "power:GND") (at 107.95 158.75 0) (unit 1)
     (in_bom yes) (on_board yes)
-    (property "Reference" "#PWR061" (id 0) (at 107.95 165.1 0)
+    (property "Reference" "#PWR057" (id 0) (at 107.95 165.1 0)
       (effects (font (size 1.27 1.27)) hide)
     )
@@
   (symbol (lib_id "power:GND") (at 53.34 167.64 0) (unit 1)
     (in_bom yes) (on_board yes)
-    (property "Reference" "#PWR060" (id 0) (at 53.34 173.99 0)
+    (property "Reference" "#PWR056" (id 0) (at 53.34 173.99 0)
       (effects (font (size 1.27 1.27)) hide)
     )
@@
   (symbol (lib_id "Connector_Generic:Conn_01x06") (at 271.78 55.88 0) (mirror x) (unit 1)
     (in_bom yes) (on_board yes)
-    (property "Reference" "J23" (id 0) (at 269.6972 66.4718 0))
+    (property "Reference" "J22" (id 0) (at 269.6972 66.4718 0))
     (property "Value" "Trimmer" (id 1) (at 269.6972 64.1604 0))
     (property "Footprint" "0.main.robot:JSTB6B-ZR" (id 2) (at 271.78 55.88 0)

Commit message: update: main
Parts:
- R27, R28: value 47k -> 10k
Changed lines of the file:
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@@
     (in_bom yes) (on_board yes)
     (property "Reference" "R28" (id 0) (at 82.042 153.67 90))
-    (property "Value" "47k" (id 1) (at 80.01 153.67 90))
+    (property "Value" "10k" (id 1) (at 80.01 153.67 90))
     (property "Footprint" "Resistor_SMD:R_0603_1608Metric_Pad0.98x0.95mm_HandSolder" (id 2) (at 78.232 153.67 90)
       (effects (font (size 1.27 1.27)) hide)
@@
     (in_bom yes) (on_board yes)
     (property "Reference" "R27" (id 0) (at 75.692 153.67 90))
-    (property "Value" "47k" (id 1) (at 73.66 153.67 90))
+    (property "Value" "10k" (id 1) (at 73.66 153.67 90))
     (property "Footprint" "Resistor_SMD:R_0603_1608Metric_Pad0.98x0.95mm_HandSolder" (id 2) (at 71.882 153.67 90)
       (effects (font (size 1.27 1.27)) hide)
