File: kicad/main/LineTrimmer.kicad_sch (KiCad schematic)
At the start: 22 parts, among them J20 I2C/OLED, J21 ICSP, J22 Trimmer, SW5 RESET, U6 ATmega328P-AU, Y2 8Mhz

Commit message: fix:
Parts:
- renumbered J20 to J19, J21 to J20, J22 to J21
Changed lines of the file:
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@@
   (symbol (lib_id "power:GND") (at 133.35 82.55 0) (unit 1)
     (in_bom yes) (on_board yes)
-    (property "Reference" "#PWR058" (id 0) (at 133.35 88.9 0)
+    (property "Reference" "#PWR056" (id 0) (at 133.35 88.9 0)
       (effects (font (size 1.27 1.27)) hide)
     )
@@
   (symbol (lib_id "power:GND") (at 149.86 50.8 0) (unit 1)
     (in_bom yes) (on_board yes)
-    (property "Reference" "#PWR060" (id 0) (at 149.86 57.15 0)
+    (property "Reference" "#PWR058" (id 0) (at 149.86 57.15 0)
       (effects (font (size 1.27 1.27)) hide)
     )
@@
   (symbol (lib_id "power:GND") (at 44.45 143.51 0) (unit 1)
     (in_bom yes) (on_board yes)
-    (property "Reference" "#PWR055" (id 0) (at 44.45 149.86 0)
+    (property "Reference" "#PWR053" (id 0) (at 44.45 149.86 0)
       (effects (font (size 1.27 1.27)) hide)
     )
@@
   (symbol (lib_id "Connector_Generic:Conn_01x04") (at 43.18 162.56 0) (mirror y) (unit 1)
     (in_bom yes) (on_board yes)
-    (property "Reference" "J20" (id 0) (at 43.18 157.48 0))
+    (property "Reference" "J19" (id 0) (at 43.18 157.48 0))
     (property "Value" "I2C/OLED" (id 1) (at 43.18 170.18 0))
     (property "Footprint" "0.main.robot:JSTB4B-ZR" (id 2) (at 43.18 162.56 0)
@@
   (symbol (lib_id "power:GND") (at 149.86 50.8 0) (unit 1)
     (in_bom yes) (on_board yes)
-    (property "Reference" "#PWR061" (id 0) (at 149.86 57.15 0)
+    (property "Reference" "#PWR059" (id 0) (at 149.86 57.15 0)
       (effects (font (size 1.27 1.27)) hide)
     )
@@
   (symbol (lib_id "power:GND") (at 147.32 125.73 0) (unit 1)
     (in_bom yes) (on_board yes)
-    (property "Reference" "#PWR059" (id 0) (at 147.32 132.08 0)
+    (property "Reference" "#PWR057" (id 0) (at 147.32 132.08 0)
       (effects (font (size 1.27 1.27)) hide)
     )
@@
   (symbol (lib_id "Connector_Generic:Conn_01x06") (at 142.24 43.18 90) (unit 1)
     (in_bom yes) (on_board yes)
-    (property "Reference" "J21" (id 0) (at 152.0952 44.0944 90)
+    (property "Reference" "J20" (id 0) (at 152.0952 44.0944 90)
       (effects (font (size 1.27 1.27)) (justify right))
     )
@@
   (symbol (lib_id "power:GND") (at 107.95 158.75 0) (unit 1)
     (in_bom yes) (on_board yes)
-    (property "Reference" "#PWR057" (id 0) (at 107.95 165.1 0)
+    (property "Reference" "#PWR055" (id 0) (at 107.95 165.1 0)
       (effects (font (size 1.27 1.27)) hide)
     )
@@
   (symbol (lib_id "power:GND") (at 53.34 167.64 0) (unit 1)
     (in_bom yes) (on_board yes)
-    (property "Reference" "#PWR056" (id 0) (at 53.34 173.99 0)
+    (property "Reference" "#PWR054" (id 0) (at 53.34 173.99 0)
       (effects (font (size 1.27 1.27)) hide)
     )
@@
   (symbol (lib_id "Connector_Generic:Conn_01x06") (at 271.78 55.88 0) (mirror x) (unit 1)
     (in_bom yes) (on_board yes)
-    (property "Reference" "J22" (id 0) (at 269.6972 66.4718 0))
+    (property "Reference" "J21" (id 0) (at 269.6972 66.4718 0))
     (property "Value" "Trimmer" (id 1) (at 269.6972 64.1604 0))
     (property "Footprint" "0.main.robot:JSTB6B-ZR" (id 2) (at 271.78 55.88 0)

Commit message: fix: vison-board GND
Parts:
- renumbered J19 to J18, J20 to J19, J21 to J20, SW5 to SW4
Changed lines of the file:
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@@
   (symbol (lib_id "power:GND") (at 133.35 82.55 0) (unit 1)
     (in_bom yes) (on_board yes)
-    (property "Reference" "#PWR056" (id 0) (at 133.35 88.9 0)
+    (property "Reference" "#PWR055" (id 0) (at 133.35 88.9 0)
       (effects (font (size 1.27 1.27)) hide)
     )
@@
   (symbol (lib_id "power:GND") (at 149.86 50.8 0) (unit 1)
     (in_bom yes) (on_board yes)
-    (property "Reference" "#PWR058" (id 0) (at 149.86 57.15 0)
+    (property "Reference" "#PWR057" (id 0) (at 149.86 57.15 0)
       (effects (font (size 1.27 1.27)) hide)
     )
@@
   (symbol (lib_id "Switch:SW_Push") (at 153.67 123.19 0) (unit 1)
     (in_bom yes) (on_board yes) (fields_autoplaced)
-    (property "Reference" "SW5" (id 0) (at 153.67 116.5692 0))
+    (property "Reference" "SW4" (id 0) (at 153.67 116.5692 0))
     (property "Value" "RESET" (id 1) (at 153.67 119.1061 0))
     (property "Footprint" "0.main.robot:TVAF06-A020B-R" (id 2) (at 153.67 118.11 0)
@@
   (symbol (lib_id "power:GND") (at 44.45 143.51 0) (unit 1)
     (in_bom yes) (on_board yes)
-    (property "Reference" "#PWR053" (id 0) (at 44.45 149.86 0)
+    (property "Reference" "#PWR052" (id 0) (at 44.45 149.86 0)
       (effects (font (size 1.27 1.27)) hide)
     )
@@
   (symbol (lib_id "Connector_Generic:Conn_01x04") (at 43.18 162.56 0) (mirror y) (unit 1)
     (in_bom yes) (on_board yes)
-    (property "Reference" "J19" (id 0) (at 43.18 157.48 0))
+    (property "Reference" "J18" (id 0) (at 43.18 157.48 0))
     (property "Value" "I2C/OLED" (id 1) (at 43.18 170.18 0))
     (property "Footprint" "0.main.robot:JSTB4B-ZR" (id 2) (at 43.18 162.56 0)
@@
   (symbol (lib_id "power:GND") (at 149.86 50.8 0) (unit 1)
     (in_bom yes) (on_board yes)
-    (property "Reference" "#PWR059" (id 0) (at 149.86 57.15 0)
+    (property "Reference" "#PWR058" (id 0) (at 149.86 57.15 0)
       (effects (font (size 1.27 1.27)) hide)
     )
@@
   (symbol (lib_id "power:GND") (at 147.32 125.73 0) (unit 1)
     (in_bom yes) (on_board yes)
-    (property "Reference" "#PWR057" (id 0) (at 147.32 132.08 0)
+    (property "Reference" "#PWR056" (id 0) (at 147.32 132.08 0)
       (effects (font (size 1.27 1.27)) hide)
     )
@@
   (symbol (lib_id "Connector_Generic:Conn_01x06") (at 142.24 43.18 90) (unit 1)
     (in_bom yes) (on_board yes)
-    (property "Reference" "J20" (id 0) (at 152.0952 44.0944 90)
+    (property "Reference" "J19" (id 0) (at 152.0952 44.0944 90)
       (effects (font (size 1.27 1.27)) (justify right))
     )
@@
   (symbol (lib_id "power:GND") (at 107.95 158.75 0) (unit 1)
     (in_bom yes) (on_board yes)
-    (property "Reference" "#PWR055" (id 0) (at 107.95 165.1 0)
+    (property "Reference" "#PWR054" (id 0) (at 107.95 165.1 0)
       (effects (font (size 1.27 1.27)) hide)
     )
@@
   (symbol (lib_id "power:GND") (at 53.34 167.64 0) (unit 1)
     (in_bom yes) (on_board yes)
-    (property "Reference" "#PWR054" (id 0) (at 53.34 173.99 0)
+    (property "Reference" "#PWR053" (id 0) (at 53.34 173.99 0)
       (effects (font (size 1.27 1.27)) hide)
     )
@@
   (symbol (lib_id "Connector_Generic:Conn_01x06") (at 271.78 55.88 0) (mirror x) (unit 1)
     (in_bom yes) (on_board yes)
-    (property "Reference" "J21" (id 0) (at 269.6972 66.4718 0))
+    (property "Reference" "J20" (id 0) (at 269.6972 66.4718 0))
     (property "Value" "Trimmer" (id 1) (at 269.6972 64.1604 0))
     (property "Footprint" "0.main.robot:JSTB6B-ZR" (id 2) (at 271.78 55.88 0)

Commit message: fix: main
Parts:
- SW4: footprint 0.main.robot:TVAF06-A020B-R -> 0.main.robot:THAU13-AB-R
Changed lines of the file:
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@@
     (property "Reference" "SW4" (id 0) (at 153.67 116.5692 0))
     (property "Value" "RESET" (id 1) (at 153.67 119.1061 0))
-    (property "Footprint" "0.main.robot:TVAF06-A020B-R" (id 2) (at 153.67 118.11 0)
+    (property "Footprint" "0.main.robot:THAU13-AB-R" (id 2) (at 153.67 118.11 0)
       (effects (font (size 1.27 1.27)) hide)
     )
