File: kicad/main/main.kicad_pcb (KiCad board)
At the start: 2 copper layers, 170 x 110 mm, 120 parts, among them J1 USB_C_Receptacle_USB2.0, J10 drib-kick, J11 drib-kick, J12 LINE, J13 ICSP, J14 MD1, J15 MD2, J16 MD3, J17 MD4, J18 I2C/OLED, J19 ICSP, J2 I2C_2, J20 Trimmer, J3 Power IN, J4 MD1, J5 MD2, J6 Serial0/XBee, J7 Serial1/IMU, J8 to cam, J9 I2C_1, Q1 AO3400A, Q2 AO3401A, SW1 BOOTSET, SW2 IMU SET, SW3 Reset, SW4 RESET, SW5 GOAL, SW6 START, SW7 AUX1, U1 RP2040_Stamp, U2 74HC32, U3 74HC04, U4 OKL-T_3-W12N-C, U5 ATmega328P-AU, U6 ATmega328P-AU, U7 AZ1117CH-3.3, U8 PCF8574PW, Y1 8Mhz, Y2 8Mhz

Commit message: 配線　標準
Routing:
- net SW1_6: track 0.00 -> 791.8 mm, vias 0 -> 7
- net SW1_3: track 0.00 -> 286.3 mm, vias 0 -> 3
- net +5V: track 0.00 -> 252.4 mm, vias 0 -> 4
- net +15V: track 0.00 -> 200.0 mm, vias 0 -> 1
- net Vcc1: track 0.00 -> 189.2 mm, vias 0 -> 4
- net LINE_D_1: track 0.00 -> 164.8 mm, vias 0 -> 3
- net LINE_D_6: track 0.00 -> 159.3 mm, vias 0 -> 3
- net LINE_D_2: track 0.00 -> 151.4 mm, vias 0 -> 4
- net Net-(J10-Pad1): track 0.00 -> 150.2 mm, vias 0 -> 1
- net LINE_D_5: track 0.00 -> 148.7 mm, vias 0 -> 3
- net LINE_D_3: track 0.00 -> 142.4 mm, vias 0 -> 2
- net LINE_D_4: track 0.00 -> 140.0 mm, vias 0 -> 3
- net Net-(C11-Pad1): track 0.00 -> 133.8 mm, vias 0 -> 2
- net I2C_1.SDA: track 0.00 -> 125.8 mm, vias 0 -> 2
- net I2C_1.SCL: track 0.00 -> 124.9 mm, vias 0 -> 1
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