File: kicad/main/main.kicad_pcb (KiCad board)
At the start: 2 copper layers, 178 parts, among them J1 Power IN1, J10 Drib, J11 Serial3/OpenMV, J12 LED, J13 I2C/IMU, J14 I2C_0, J15 SW1, J16 I2C_1, J17 I2C_2, J18 5V OUT, J19 Power IN, J2 AUX1, J20 LINE, J21 Conn_01x03, J22 DribblerMotor, J23 DribblerPower, J24 CAP, J25 Kicker1, J26 ICSP, J27 MD1, J28 MD2, J29 MD3, J3 USB2.0_C_v3, J30 MD4, J31 I2C/OLED, J32 ICSP, J33 Trimmer, J4 SW1, J5 MAIN, J6 I2C_3, J7 Kicker, J8 MD1, J9 MD2, K1 G5V-1/12V, Q1 AO3400A, Q2 AO3401A, Q3 NP52N06SLG, SW1 GOAL, SW2 START, SW3 SW_SPST, SW4 Reset, SW5 AUX1, SW6 IMU SET, SW7 Reset, SW8 RESET, SW9 BOOTSEL, U1 XBEE-S2C, U10 TLP152, U11 XL6009/HW-432, U12 ATmega328P-AU, U13 ATmega328P-AU, U14 RP2040, U15 W25Q128JVS, U2 AZ1117CH-3.3, U3 AZ1117CH-3.3, U4 PCF8574PW, U6 74HC32, U7 74HC04, U8 OKL-T_3-W12N-C, U9 TLP152, Y1 8Mhz, Y2 8Mhz, Y3 12Mhz

Commit message: fix: main
Parts:
- removed C28, C29, C30: 0.1u, Capacitor_SMD:C_0603_1608Metric_Pad1.08x0.95mm_HandSolder
- removed D20: LED(OSWT1608), 0.main.robot:LED_SMLE13WBC8W1
- removed D21, D22: RSX101VAM-30, Diode_SMD:D_0805_2012Metric_Pad1.15x1.40mm_HandSolder
- removed F1: Fuse 15A, 0.main.robot:FUSE_20mm
- removed J29: MD3, 0.main.robot:JSTB4B-ZR
- removed J30: MD4, 0.main.robot:JSTB4B-ZR
- removed J31: I2C/OLED, 0.main.robot:JSTB4B-ZR
- removed J32: ICSP, 0.main.robot:JSTB6B-ZR
- removed J33: Trimmer, 0.main.robot:JSTS6B-ZRLFSN
- removed K1: G5V-1/12V, Relay_THT:Relay_SPDT_Omron_G5V-1
- removed Q3: NP52N06SLG, Package_TO_SOT_SMD:TO-252-2
- removed R25: 470, Resistor_SMD:R_0603_1608Metric_Pad0.98x0.95mm_HandSolder
- removed R26, R27, R29, R31, R32, R33, R34: 10k, Resistor_SMD:R_0603_1608Metric_Pad0.98x0.95mm_HandSolder
- removed R28: 1k, Resistor_THT:R_Axial_DIN0204_L3.6mm_D1.6mm_P5.08mm_Horizontal
- removed R30: 330, Resistor_THT:R_Axial_DIN0204_L3.6mm_D1.6mm_P5.08mm_Horizontal
- removed R57: 200R, Resistor_SMD:R_0603_1608Metric_Pad0.98x0.95mm_HandSolder
- removed R58: 1R, Resistor_SMD:R_0603_1608Metric_Pad0.98x0.95mm_HandSolder
- removed R59, R60: 27.4R, Resistor_SMD:R_0603_1608Metric_Pad0.98x0.95mm_HandSolder
- removed R61: 10kR, Resistor_SMD:R_0603_1608Metric_Pad0.98x0.95mm_HandSolder
- removed R62: 1kR, Resistor_SMD:R_0603_1608Metric_Pad0.98x0.95mm_HandSolder
- removed RV6: 20K, 0.main.robot:Trim-GF063P
- removed SW9: BOOTSEL, 0.main.robot:TVAF06-A020B-R
- removed TP1: GND, TestPoint:TestPoint_Loop_D2.60mm_Drill0.9mm_Beaded
- removed TP2: V+, TestPoint:TestPoint_Loop_D2.60mm_Drill0.9mm_Beaded
- removed U13: ATmega328P-AU, Package_QFP:TQFP-32_7x7mm_P0.8mm
- removed U14: RP2040, rp2040:RP2040_hand
- removed U15: W25Q128JVS, rp2040:W25Q16-128JV-SOIC
- added R1: 5.1kR, Resistor_SMD:R_0603_1608Metric_Pad0.98x0.95mm_HandSolder, F.Cu at (85.1, 79.6)
- added R11: 47k, Resistor_SMD:R_0603_1608Metric_Pad0.98x0.95mm_HandSolder, F.Cu at (86.0, 77.1)
- added R14: 10k, Resistor_SMD:R_0603_1608Metric_Pad0.98x0.95mm_HandSolder, F.Cu at (119.7, 41.0)
- added R16: 10k, Resistor_SMD:R_0603_1608Metric_Pad0.98x0.95mm_HandSolder, F.Cu at (117.6, 46.5)
- added R18: 1k, Resistor_THT:R_Axial_DIN0204_L3.6mm_D1.6mm_P5.08mm_Horizontal, F.Cu at (103.5, 44.8)
- added R19: 10k, Resistor_SMD:R_0603_1608Metric_Pad0.98x0.95mm_HandSolder, F.Cu at (128.7, 32.5)
- added R2: 470, Resistor_SMD:R_0603_1608Metric_Pad0.98x0.95mm_HandSolder, F.Cu at (122.0, 47.0)
- added R20: 330, Resistor_THT:R_Axial_DIN0204_L3.6mm_D1.6mm_P5.08mm_Horizontal, F.Cu at (128.7, 24.6)
- added R21: 10k, Resistor_SMD:R_0603_1608Metric_Pad0.98x0.95mm_HandSolder, F.Cu at (138.2, 26.8)
- added R3: 5.1kR, Resistor_SMD:R_0603_1608Metric_Pad0.98x0.95mm_HandSolder, F.Cu at (80.7, 79.1)
- added R9: 470, Resistor_SMD:R_0603_1608Metric_Pad0.98x0.95mm_HandSolder, F.Cu at (110.4, 55.4)
- added U5: 74HC04, 0.main.robot:SOP14W, F.Cu at (85.1, 50.7)
- C1, C4: value 10u -> 10uF
- C11, C21, C26: value 1uF -> 0.1u
- C12: value 1uF -> 10u
- C13: value 2200uF/63V -> 10u; footprint Capacitor_THT:CP_Radial_D16.0mm_P7.50mm -> Capacitor_SMD:C_0603_1608Metric_Pad1.08x0.95mm_HandSolder
- C16, C9: value 10u -> 0.1u
- C18: value 10u -> 1uF
- C2, C5: value 10uF -> 10u
- C20: value 0.1u -> 1uF
- C3: value 0.1u -> 10u
- D1: value LED -> SX34F; footprint 0.main.robot:LED_SMLE13WBC8W1 -> Diode_SMD:D_SMA
- D10: value LED4_B -> LED3_Y
- D11: value RSX101VAM-30TR -> LED4_B; footprint Diode_SMD:D_SMA -> 0.main.robot:LED_SMLE13WBC8W1
- D13: value LED -> RSX101VAM-30TR; footprint 0.main.robot:LED_SMLE13WBC8W1 -> Diode_SMD:D_0805_2012Metric_Pad1.15x1.40mm_HandSolder
- D14: value SX34F -> LED(OSWT1608); footprint Diode_SMD:D_SMA -> LED_SMD:LED_0603_1608Metric_Pad1.05x0.95mm_HandSolder
- D15: value LED -> LED(OSWT1608)
- D17: footprint LED_SMD:LED_0603_1608Metric_Pad1.05x0.95mm_HandSolder -> 0.main.robot:LED_SMLE13WBC8W1
- D18: value LED(OSWT1608) -> RSX101VAM-30; footprint LED_SMD:LED_0603_1608Metric_Pad1.05x0.95mm_HandSolder -> Diode_SMD:D_0805_2012Metric_Pad1.15x1.40mm_HandSolder
- D19: value RSX101VAM-30TR -> RSX101VAM-30
- D4: value SX34F -> RX; footprint Diode_SMD:D_SMA -> LED_SMD:LED_0603_1608Metric_Pad1.05x0.95mm_HandSolder
- D5: value RX -> TX
- D6: value TX -> RSX101VAM-30TR; footprint LED_SMD:LED_0603_1608Metric_Pad1.05x0.95mm_HandSolder -> Diode_SMD:D_SMA
- D7: value LED1_R -> LED
- D8: value LED2_G -> LED1_R
- D9: value LED3_Y -> LED2_G
- J1: value Power IN1 -> USB2.0_C_v3; footprint 0.main.robot:AMASS_XT60-M_1x02_P7.20mm_Vertical -> rp2040:USB-C-12-Pin-MidMount-ali-v4
- J11: value Serial3/OpenMV -> I2C_0
- J12: value LED -> SW1
- J13: value I2C/IMU -> I2C_1
- J14: value I2C_0 -> drib-kick
- J15: value SW1 -> drib-kick; footprint 0.main.robot:JSTB6B-ZR -> 0.main.robot:JSTB4B-ZR
- J16: value I2C_1 -> I2C_2
- J17: value I2C_2 -> 5V OUT; footprint 0.main.robot:JSTB4B-ZR -> Connector_JST:JST_XH_B2B-XH-A_1x02_P2.50mm_Vertical
- J18: value 5V OUT -> LINE; footprint Connector_JST:JST_XH_B2B-XH-A_1x02_P2.50mm_Vertical -> 0.main.robot:JSTB8B-ZR
- J19: value Power IN -> SW1; footprint Connector_JST:JST_XH_B2B-XH-A_1x02_P2.50mm_Vertical -> 0.main.robot:JSTS6B-ZRLFSN
- J20: value LINE -> I2C/IMU; footprint 0.main.robot:JSTB8B-ZR -> 0.main.robot:JSTB4B-ZR
- J21: value Conn_01x03 -> ICSP; footprint Connector_PinHeader_2.54mm:PinHeader_1x03_P2.54mm_Vertical -> 0.main.robot:JSTB6B-ZR
- J22: value DribblerMotor -> MD1; footprint Connector_JST:JST_XH_B2B-XH-A_1x02_P2.50mm_Vertical -> 0.main.robot:JSTB4B-ZR
- J23: value DribblerPower -> MD2; footprint Connector_JST:JST_XH_B2B-XH-A_1x02_P2.50mm_Vertical -> 0.main.robot:JSTB4B-ZR
- J24: value CAP -> MD3; footprint Connector_JST:JST_XH_B2B-XH-A_1x02_P2.50mm_Vertical -> 0.main.robot:JSTB4B-ZR
- J25: value Kicker1 -> MD4; footprint Connector_JST:JST_XH_B2B-XH-A_1x02_P2.50mm_Vertical -> 0.main.robot:JSTB4B-ZR
- J26: value ICSP -> I2C/OLED; footprint 0.main.robot:JSTB6B-ZR -> 0.main.robot:JSTB4B-ZR
- J27: value MD1 -> ICSP; footprint 0.main.robot:JSTB4B-ZR -> 0.main.robot:JSTB6B-ZR
- J28: value MD2 -> Trimmer; footprint 0.main.robot:JSTB4B-ZR -> 0.main.robot:JSTS6B-ZRLFSN
- J3: value USB2.0_C_v3 -> I2C_3; footprint rp2040:USB-C-12-Pin-MidMount-ali-v4 -> 0.main.robot:JSTB4B-ZR
- J4: value SW1 -> Serial3/OpenMV; footprint 0.main.robot:JSTS6B-ZRLFSN -> 0.main.robot:JSTB4B-ZR
- J5: value MAIN -> Power IN; footprint Connector_JST:JST_XH_B2B-XH-A_1x02_P2.50mm_Vertical -> Connector_JST:JST_VH_B2P-VH-B_1x02_P3.96mm_Vertical
- J6: value I2C_3 -> LED; footprint 0.main.robot:JSTB4B-ZR -> 0.main.robot:JSTB6B-ZR
- R10, R15, R4, R48: value 470 -> 10k
- R22, R37, R47: value 47k -> 470
- R24: value 47k -> 10k
- R35, R45: value 470 -> 47k
- R36, R38: value 10k -> 47k
- R39: value 120 -> 470
- R40: value 120 -> 47k
- R41: value 200 -> 47k; footprint Resistor_THT:R_Axial_DIN0204_L3.6mm_D1.6mm_P5.08mm_Horizontal -> Resistor_SMD:R_0603_1608Metric_Pad0.98x0.95mm_HandSolder
- R42: value 100 -> 470; footprint Resistor_THT:R_Axial_DIN0411_L9.9mm_D3.6mm_P20.32mm_Horizontal -> Resistor_SMD:R_0603_1608Metric_Pad0.98x0.95mm_HandSolder
- R43: value 30k -> 10k; footprint Resistor_THT:R_Axial_DIN0204_L3.6mm_D1.6mm_P5.08mm_Horizontal -> Resistor_SMD:R_0603_1608Metric_Pad0.98x0.95mm_HandSolder
- R49: value 10k -> 1k
- R5, R7: value 5.1kR -> 10k
- R50: value 47k -> 1k
- R51: value 47k -> 200R
- R52: value 47k -> 1R
- R53: value 470 -> 27.4R
- R54: value 10k -> 27.4R
- R55: value 1k -> 10kR
- R56: value 1k -> 1kR
- R6: value 10k -> 470
- RV1: value 20k -> 20K; footprint 0.main.robot:Trim-GF063X -> 0.main.robot:Trim-GF063P
- SW1: value GOAL -> Reset; footprint 0.main.robot:MFS101D-14-Z -> 0.main.robot:THAU13-AB-R
- SW2: value START -> Reset; footprint 0.main.robot:SW_NKK_B-12CCPRM -> 0.main.robot:THAU13-AB-R
- SW3: value SW_SPST -> GOAL; footprint 0.main.robot:SW_SPST_POWER -> 0.main.robot:MFS101D-14-Z
- SW4: value Reset -> START; footprint 0.main.robot:THAU13-AB-R -> 0.main.robot:SW_NKK_B-12CCPRM
- SW7: value Reset -> RESET; footprint 0.main.robot:THAU13-AB-R -> 0.main.robot:TVAF06-A020B-R
- SW8: value RESET -> BOOTSEL
- U10, U9: value TLP152 -> ATmega328P-AU; footprint 0.main.robot:TLP152 -> Package_QFP:TQFP-32_7x7mm_P0.8mm
- U11: value XL6009/HW-432 -> RP2040; footprint 0.main.robot:XL6009_HW432 -> rp2040:RP2040_hand
- U12: value ATmega328P-AU -> W25Q128JVS; footprint Package_QFP:TQFP-32_7x7mm_P0.8mm -> rp2040:W25Q16-128JV-SOIC
- U4: value PCF8574PW -> 74HC32; footprint Package_SO:TSSOP-20_4.4x6.5mm_P0.65mm -> 0.main.robot:SOP14W
- U6: value 74HC32 -> OKL-T_3-W12N-C; footprint 0.main.robot:SOP14W -> 0.main.robot:OKL-T3-W12N-C
- U7: value 74HC04 -> PCF8574PW; footprint 0.main.robot:SOP14W -> Package_SO:TSSOP-20_4.4x6.5mm_P0.65mm
- U8: value OKL-T_3-W12N-C -> AE-BNO055; footprint 0.main.robot:OKL-T3-W12N-C -> 0.main.robot:AE-BNO055
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Connections:
- C1 pad 2: Net-(C1-Pad2) -> GND
- C10 pad 1: Vbatt -> Net-(C10-Pad1)
- C11 pad 1: Net-(C11-Pad1) -> +3.3VA
- C11 pad 2: Net-(C11-Pad2) -> GND
- C12 pad 1: +15V -> Net-(C12-Pad1)
- C13 pad 1: Net-(C13-Pad1) -> Vcc1
- C14 pad 1: +3.3VA -> Vcc1
- C15 pad 1: Net-(C15-Pad1) -> RESET
- C16 pad 1: Vcc1 -> +1V1
- C17 pad 1: Vcc1 -> +1V1
- C18 pad 1: RESET -> +1V1
- C19 pad 1: +1V1 -> +3V3
- C2 pad 2: GND -> Net-(C2-Pad2)
- C20 pad 1: +1V1 -> +3V3
- C21 pad 1: +1V1 -> +3V3
- C23 pad 1: +3V3 -> Net-(C23-Pad1)
- C26 pad 1: Net-(C26-Pad1) -> +3V3
- C3 pad 1: Net-(C3-Pad1) -> +5V
- C3 pad 2: GND -> Net-(C2-Pad2)
- C4 pad 1: +5V -> +3V3
- C4 pad 2: Net-(C1-Pad2) -> GND
- C5 pad 1: +3V3 -> GND
- C5 pad 2: GND -> /rp2040/RUN(RES)/30
- C6 pad 1: GND -> +15V
- C6 pad 2: /rp2040/RUN(RES)/30 -> GND
- C7 pad 1: Net-(C3-Pad1) -> +5V
- C7 pad 2: GND -> Net-(C7-Pad2)
- C8 pad 1: +15V -> Vbatt
- C9 pad 1: +5V -> Net-(C10-Pad1)
- C9 pad 2: Net-(C9-Pad2) -> GND
- D1 pad 1: Net-(D1-Pad1) -> Net-(C1-Pad1)
- D11 pad 1: +3V3 -> Net-(D10-Pad1)
- D11 pad 2: /rp2040/RUN(RES)/30 -> Net-(D11-Pad2)
- D13 pad 1: GND -> +3.3VA
- D13 pad 2: Net-(D13-Pad2) -> +3V3
- D14 pad 1: Net-(C11-Pad1) -> GND
- D16 pad 2: +3V3 -> Net-(C12-Pad1)
- D18 pad 1: GND -> Vcc1
- D18 pad 2: Net-(D18-Pad2) -> RESET
- D19 pad 1: +3.3VA -> Vcc1
- D19 pad 2: Net-(C15-Pad1) -> Net-(D19-Pad2)
- D2 pad 1: Net-(C2-Pad1) -> Net-(C1-Pad1)
- D2 pad 2: Net-(D2-Pad2) -> +5V
- D4 pad 1: Net-(C2-Pad1) -> GND
- D4 pad 2: +5V -> Net-(D4-Pad2)
- D6 pad 1: GND -> +3V3
- D6 pad 2: Net-(D6-Pad2) -> /rp2040/RUN(RES)/30
- D7 pad 1: Net-(D10-Pad1) -> GND
- J1 pad 1: Net-(D1-Pad1) -> Net-(D1-Pad2)
- J1 pad 2: Net-(J1-Pad2) -> USB_DM
- J10 pad 1: Net-(F1-Pad1) -> +15V
- J10 pad 2: Net-(D1-Pad1) -> GND
- J11 pad 1: /rp2040/GPIO08/11 -> /rp2040/GPIO05/07
- J11 pad 2: +5V -> +3V3
- J11 pad 3: Net-(J11-Pad3) -> /rp2040/GPIO04/06
- J12 pad 1: /rp2040/GPIO26/31 -> /rp2040/GPIO03/05
- J12 pad 2: unconnected-(J12-Pad2) -> /rp2040/GPIO06/09
- J12 pad 3: unconnected-(J12-Pad3) -> +3V3
- J12 pad 4: unconnected-(J12-Pad4) -> /rp2040/GPIO02/04
- J12 pad 5: /rp2040/GPIO22/29 -> /rp2040/GPIO07/10
- J13 pad 1: Net-(J13-Pad1) -> /rp2040/GPIO05/07
- J13 pad 2: Net-(C3-Pad1) -> +3V3
- J13 pad 3: Net-(J13-Pad3) -> /rp2040/GPIO04/06
- J14 pad 1: /rp2040/GPIO05/07 -> /rp2040/GPIO13/17
- J14 pad 2: +3V3 -> GND
- J14 pad 3: /rp2040/GPIO04/06 -> /rp2040/GPIO12/16
- J15 pad 1: /rp2040/GPIO03/05 -> +15V
- J15 pad 2: /rp2040/GPIO06/09 -> GND
- J15 pad 3: +3V3 -> +15V
- J15 pad 4: /rp2040/GPIO02/04 -> GND
- J17 pad 1: /rp2040/GPIO05/07 -> Net-(J17-Pad1)
- J17 pad 2: +3V3 -> Net-(C7-Pad2)
- J18 pad 2: Net-(C9-Pad2) -> Net-(J18-Pad2)
- J19 pad 2: GND -> Net-(J19-Pad2)
- J20 pad 2: Net-(J20-Pad2) -> Net-(C10-Pad1)
- J20 pad 4: Net-(J20-Pad4) -> GND
- J21 pad 2: Net-(J21-Pad2) -> +3.3VA
- J22 pad 1: Net-(C11-Pad1) -> Net-(J21-Pad4)
- J22 pad 2: Net-(D14-Pad2) -> Net-(J21-Pad1)
- J23 pad 1: Net-(C11-Pad1) -> Net-(J23-Pad1)
- J23 pad 2: Net-(C11-Pad2) -> Net-(J23-Pad2)
- J24 pad 1: Net-(C13-Pad1) -> Net-(J24-Pad1)
- J24 pad 2: GND -> Net-(J24-Pad2)
- J25 pad 2: GND -> Net-(J25-Pad2)
- J26 pad 1: Net-(J26-Pad1) -> /LineTrimmer/SCL
- J26 pad 2: +3.3VA -> Vcc1
- J26 pad 3: Net-(J26-Pad3) -> /LineTrimmer/SDA
- J26 pad 4: Net-(J26-Pad4) -> GND
- J27 pad 1: Net-(J26-Pad4) -> Net-(J27-Pad1)
- J27 pad 2: Net-(J26-Pad1) -> Vcc1
- J27 pad 3: Net-(J26-Pad4) -> Net-(J27-Pad3)
- J27 pad 4: Net-(J26-Pad3) -> Net-(J27-Pad4)
- J28 pad 3: Net-(J28-Pad1) -> Net-(J28-Pad3)
- J3 pad 1: Net-(D2-Pad2) -> /Sheet63625160/SCL_1
- J3 pad 2: USB_DM -> +3V3
- J3 pad 3: USB_DP -> /Sheet63625160/SDA_1
- J4 pad 1: Net-(J4-Pad1) -> /rp2040/GPIO08/11
- J4 pad 2: Net-(J4-Pad2) -> +5V
- J4 pad 4: Net-(J4-Pad4) -> GND
- J5 pad 1: Net-(F1-Pad1) -> GND
- J5 pad 2: Net-(D1-Pad1) -> +15V
- J6 pad 1: /Sheet63625160/SCL_1 -> /rp2040/GPIO26/31
- J6 pad 2: +3V3 -> unconnected-(J6-Pad2)
- J6 pad 3: /Sheet63625160/SDA_1 -> unconnected-(J6-Pad3)
- J6 pad 4: GND -> unconnected-(J6-Pad4)
- J7 pad 1: Net-(F1-Pad1) -> +15V
- J7 pad 2: Net-(D1-Pad1) -> GND
- J8 pad 1: Net-(D1-Pad1) -> GND
- J8 pad 2: Net-(F1-Pad1) -> +15V
- J9 pad 1: Net-(D1-Pad1) -> GND
- J9 pad 2: Net-(F1-Pad1) -> +15V
- JP1 pad 2: Net-(J4-Pad5) -> Net-(J19-Pad5)
- Q2 pad 3: Net-(J20-Pad4) -> Net-(J18-Pad4)
- R10 pad 1: Net-(R10-Pad1) -> /rp2040/GPIO09/12
- R10 pad 2: Net-(D5-Pad2) -> Net-(J4-Pad3)
- R12 pad 1: Net-(R12-Pad1) -> +3V3
- R12 pad 2: /rp2040/GPIO00/01 -> /rp2040/GPIO05/07
- R13 pad 1: Net-(R10-Pad1) -> +3V3
- R13 pad 2: /rp2040/GPIO01/02 -> /rp2040/GPIO04/06
- R15 pad 1: /rp2040/GPIO00/01 -> Net-(R15-Pad1)
- R15 pad 2: Net-(D6-Pad2) -> Net-(J18-Pad2)
- R17 pad 1: /rp2040/GPIO09/12 -> Net-(R17-Pad1)
- R17 pad 2: Net-(J11-Pad3) -> Net-(J18-Pad6)
- R22 pad 1: +3V3 -> Net-(J17-Pad1)
- R22 pad 2: /rp2040/RUN(RES)/30 -> Net-(D7-Pad2)
- R23 pad 1: Net-(C3-Pad1) -> +15V
- R23 pad 2: Net-(J13-Pad3) -> Vbatt
- R24 pad 1: Net-(C3-Pad1) -> Vbatt
- R24 pad 2: Net-(J13-Pad1) -> GND
- R35 pad 1: Net-(J18-Pad1) -> Net-(C10-Pad1)
- R35 pad 2: Net-(D13-Pad2) -> Net-(J20-Pad3)
- R36 pad 1: +5V -> Net-(C10-Pad1)
- R36 pad 2: Net-(Q1-Pad3) -> Net-(J20-Pad1)
- R37 pad 1: Net-(J19-Pad1) -> Net-(C10-Pad1)
- R37 pad 2: Vbatt -> Net-(D12-Pad2)
- R38 pad 1: Vbatt -> Net-(R38-Pad1)
- R38 pad 2: GND -> +3.3VA
- R39 pad 1: Net-(R39-Pad1) -> +3.3VA
- R39 pad 2: /Sheet61861092/drib_in -> Net-(D14-Pad2)
- R4 pad 1: Net-(R4-Pad1) -> Net-(C2-Pad1)
- R4 pad 2: Net-(D3-Pad2) -> Net-(R4-Pad2)
- R40 pad 1: Net-(R40-Pad1) -> +3.3VA
- R40 pad 2: /Sheet61861092/kick_in -> /Sheet63625160/SCL_1
- R41 pad 1: Net-(J21-Pad1) -> +3.3VA
- R41 pad 2: Net-(R41-Pad2) -> /Sheet63625160/SDA_1
- R42 pad 1: Net-(K1-Pad1) -> Net-(R42-Pad1)
- R42 pad 2: Net-(R42-Pad2) -> Net-(D15-Pad2)
- R43 pad 1: Net-(C13-Pad1) -> Net-(C12-Pad1)
- R43 pad 2: Net-(D15-Pad2) -> +3.3VA
- R44 pad 2: +3.3VA -> Vcc1
- R45 pad 1: +3.3VA -> Vcc1
- R45 pad 2: Net-(D17-Pad2) -> /LineTrimmer/SCL
- R46 pad 1: +3.3VA -> Vcc1
- R46 pad 2: /Sheet63625160/SCL_1 -> /LineTrimmer/SDA
- R47 pad 1: +3.3VA -> Net-(R47-Pad1)
- R47 pad 2: /Sheet63625160/SDA_1 -> Net-(D17-Pad2)
- R48 pad 1: Net-(R48-Pad1) -> RESET
- R48 pad 2: Net-(D18-Pad2) -> Vcc1
- R49 pad 1: Net-(C15-Pad1) -> /rp2040/RUN(RES)/30
- R49 pad 2: +3.3VA -> +3V3
- R5 pad 1: Net-(J3-Pad6) -> Net-(C2-Pad1)
- R5 pad 2: GND -> Net-(R5-Pad2)
- R50 pad 2: Vcc1 -> Net-(R50-Pad2)
- R51 pad 1: Vcc1 -> ADC_VREF
- R51 pad 2: /LineTrimmer/SCL -> +3V3
- R52 pad 1: Vcc1 -> Net-(C23-Pad1)
- R52 pad 2: /LineTrimmer/SDA -> ADC_VREF
- R53 pad 2: Net-(D20-Pad2) -> USB_DP
- R54 pad 1: RESET -> Net-(R54-Pad1)
- R54 pad 2: Vcc1 -> USB_DM
- R55 pad 1: /rp2040/RUN(RES)/30 -> QSPI_SS
- R56 pad 2: Net-(R56-Pad2) -> QSPI_SS
- R6 pad 1: Net-(C1-Pad1) -> Net-(R5-Pad2)
- R6 pad 2: Net-(R6-Pad2) -> Net-(D4-Pad2)
- R7 pad 1: Net-(J3-Pad5) -> Net-(R7-Pad1)
- R7 pad 2: GND -> /rp2040/GPIO00/01
- R8 pad 1: Net-(C1-Pad1) -> Net-(R5-Pad2)
- R8 pad 2: Net-(R10-Pad1) -> /rp2040/GPIO01/02
- RV1 pad 1: Net-(R41-Pad2) -> Net-(D19-Pad2)
- RV1 pad 2: Net-(J21-Pad2) -> Net-(J28-Pad1)
- RV1 pad 3: Net-(J21-Pad3) -> Net-(J28-Pad1)
- RV2 pad 1: Net-(D22-Pad2) -> Net-(D19-Pad2)
- RV2 pad 2: Net-(J33-Pad1) -> Net-(J28-Pad2)
- RV2 pad 3: Net-(J33-Pad1) -> Net-(J28-Pad2)
- RV3 pad 1: Net-(D22-Pad2) -> Net-(D19-Pad2)
- RV3 pad 2: Net-(J33-Pad2) -> Net-(J28-Pad3)
- RV3 pad 3: Net-(J33-Pad2) -> Net-(J28-Pad3)
- RV4 pad 1: Net-(D22-Pad2) -> Net-(D19-Pad2)
- RV4 pad 2: Net-(J33-Pad3) -> Net-(J28-Pad4)
- RV4 pad 3: Net-(J33-Pad3) -> Net-(J28-Pad4)
- RV5 pad 1: Net-(D22-Pad2) -> Net-(D19-Pad2)
- RV5 pad 2: Net-(J33-Pad4) -> Line5
- RV5 pad 3: Net-(J33-Pad4) -> Line5
- SW1 pad 1: Net-(J4-Pad3) -> Net-(R4-Pad2)
- SW1 pad 2: Net-(J4-Pad1) -> GND
- SW2 pad 1: Net-(J4-Pad3) -> /rp2040/RUN(RES)/30
- SW2 pad 2: Net-(J4-Pad4) -> GND
- SW3 pad 1: Net-(F1-Pad2) -> Net-(J19-Pad3)
- SW3 pad 2: Net-(J1-Pad2) -> Net-(J19-Pad1)
- SW4 pad 1: Net-(R6-Pad2) -> Net-(J19-Pad3)
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
Commit message: fix: main xbee
Parts:
- removed C26, C27: 0.1u, Capacitor_SMD:C_0603_1608Metric_Pad1.08x0.95mm_HandSolder
- removed D17: LED(OSWT1608), 0.main.robot:LED_SMLE13WBC8W1
- removed D18, D19: RSX101VAM-30, Diode_SMD:D_0805_2012Metric_Pad1.15x1.40mm_HandSolder
- removed R50: 1k, Resistor_SMD:R_0603_1608Metric_Pad0.98x0.95mm_HandSolder
- removed R51: 200R, Resistor_SMD:R_0603_1608Metric_Pad0.98x0.95mm_HandSolder
- removed R52: 1R, Resistor_SMD:R_0603_1608Metric_Pad0.98x0.95mm_HandSolder
- removed R53, R54: 27.4R, Resistor_SMD:R_0603_1608Metric_Pad0.98x0.95mm_HandSolder
- removed R55: 10kR, Resistor_SMD:R_0603_1608Metric_Pad0.98x0.95mm_HandSolder
- removed R56: 1kR, Resistor_SMD:R_0603_1608Metric_Pad0.98x0.95mm_HandSolder
- removed SW8: BOOTSEL, 0.main.robot:TVAF06-A020B-R
- removed U11: RP2040, rp2040:RP2040_hand
- removed U12: W25Q128JVS, rp2040:W25Q16-128JV-SOIC
- added J29: Trimmer, 0.main.robot:JSTS6B-ZRLFSN, F.Cu at (53.1, 81.3)
- added R25: 120, Resistor_SMD:R_0603_1608Metric_Pad0.98x0.95mm_HandSolder, F.Cu at (117.2, 46.6)
- added R26: 120, Resistor_SMD:R_0603_1608Metric_Pad0.98x0.95mm_HandSolder, F.Cu at (68.9, 74.6)
- added R27: 120, Resistor_SMD:R_0603_1608Metric_Pad0.98x0.95mm_HandSolder, F.Cu at (112.8, 46.6)
- added R28: 47k, Resistor_SMD:R_0603_1608Metric_Pad0.98x0.95mm_HandSolder, F.Cu at (96.7, 71.1)
- added R29: 47k, Resistor_SMD:R_0603_1608Metric_Pad0.98x0.95mm_HandSolder, F.Cu at (137.3, 31.7)
- added R30: 470, Resistor_SMD:R_0603_1608Metric_Pad0.98x0.95mm_HandSolder, F.Cu at (119.3, 41.6)
- added R31: 47k, Resistor_SMD:R_0603_1608Metric_Pad0.98x0.95mm_HandSolder, F.Cu at (178.6, 27.2)
- added R32: 470, Resistor_SMD:R_0603_1608Metric_Pad0.98x0.95mm_HandSolder, F.Cu at (166.9, 39.8)
- added R33: 47k, Resistor_SMD:R_0603_1608Metric_Pad0.98x0.95mm_HandSolder, F.Cu at (173.9, 29.7)
- added R34: 47k, Resistor_SMD:R_0603_1608Metric_Pad0.98x0.95mm_HandSolder, F.Cu at (169.1, 35.2)
- C11: value 0.1u -> 10u
- C12, C15, C7: value 10u -> 0.1u
- C16, C21: value 0.1u -> 1uF
- C2: value 10u -> 10uF
- C20, C23: value 1uF -> 0.1u
- C4: value 10uF -> 10u
- D10: value LED3_Y -> RSX101VAM-30TR; footprint 0.main.robot:LED_SMLE13WBC8W1 -> Diode_SMD:D_0805_2012Metric_Pad1.15x1.40mm_HandSolder
- D11: value LED4_B -> LED(OSWT1608); footprint 0.main.robot:LED_SMLE13WBC8W1 -> LED_SMD:LED_0603_1608Metric_Pad1.05x0.95mm_HandSolder
- D12: footprint 0.main.robot:LED_SMLE13WBC8W1 -> LED_SMD:LED_0603_1608Metric_Pad1.05x0.95mm_HandSolder
- D14: footprint LED_SMD:LED_0603_1608Metric_Pad1.05x0.95mm_HandSolder -> 0.main.robot:LED_SMLE13WBC8W1
- D15: value LED(OSWT1608) -> RSX101VAM-30; footprint LED_SMD:LED_0603_1608Metric_Pad1.05x0.95mm_HandSolder -> Diode_SMD:D_0805_2012Metric_Pad1.15x1.40mm_HandSolder
- D16: value RSX101VAM-30TR -> RSX101VAM-30
- D3: value RSSI -> RSX101VAM-30TR; footprint LED_SMD:LED_0603_1608Metric_Pad1.05x0.95mm_HandSolder -> Diode_SMD:D_SMA
- D4: value RX -> LED; footprint LED_SMD:LED_0603_1608Metric_Pad1.05x0.95mm_HandSolder -> 0.main.robot:LED_SMLE13WBC8W1
- D5: value TX -> LED1_R; footprint LED_SMD:LED_0603_1608Metric_Pad1.05x0.95mm_HandSolder -> 0.main.robot:LED_SMLE13WBC8W1
- D6: value RSX101VAM-30TR -> LED2_G; footprint Diode_SMD:D_SMA -> 0.main.robot:LED_SMLE13WBC8W1
- D7: value LED -> LED3_Y
- D8: value LED1_R -> LED4_B
- D9: value LED2_G -> LED(OSWT1608)
- J10: value Drib -> MD2; footprint Connector_JST:JST_XH_B2B-XH-A_1x02_P2.50mm_Vertical -> Connector_JST:JST_XH_S2B-XH-A-1_1x02_P2.50mm_Horizontal
- J11: value I2C_0 -> Drib; footprint 0.main.robot:JSTB4B-ZR -> Connector_JST:JST_XH_B2B-XH-A_1x02_P2.50mm_Vertical
- J12: value SW1 -> I2C_0; footprint 0.main.robot:JSTB6B-ZR -> 0.main.robot:JSTB4B-ZR
- J13: value I2C_1 -> SW1; footprint 0.main.robot:JSTB4B-ZR -> 0.main.robot:JSTB6B-ZR
- J14: value drib-kick -> I2C_1
- J16: value I2C_2 -> drib-kick
- J17: value 5V OUT -> I2C_2; footprint Connector_JST:JST_XH_B2B-XH-A_1x02_P2.50mm_Vertical -> 0.main.robot:JSTB4B-ZR
- J18: value LINE -> 5V OUT; footprint 0.main.robot:JSTB8B-ZR -> Connector_JST:JST_XH_B2B-XH-A_1x02_P2.50mm_Vertical
- J19: value SW1 -> LINE; footprint 0.main.robot:JSTS6B-ZRLFSN -> 0.main.robot:JSTB8B-ZR
- J20: value I2C/IMU -> SW1; footprint 0.main.robot:JSTB4B-ZR -> 0.main.robot:JSTS6B-ZRLFSN
- J21: value ICSP -> I2C/IMU; footprint 0.main.robot:JSTB6B-ZR -> 0.main.robot:JSTB4B-ZR
- J22: value MD1 -> ICSP; footprint 0.main.robot:JSTB4B-ZR -> 0.main.robot:JSTB6B-ZR
- J23, J9: value MD2 -> MD1
- J24: value MD3 -> MD2
- J25: value MD4 -> MD3
- J26: value I2C/OLED -> MD4
- J27: value ICSP -> I2C/OLED; footprint 0.main.robot:JSTB6B-ZR -> 0.main.robot:JSTB4B-ZR
- J28: value Trimmer -> ICSP; footprint 0.main.robot:JSTS6B-ZRLFSN -> 0.main.robot:JSTB6B-ZR
- J4: value Serial3/OpenMV -> XBee
- J5: value Power IN -> Serial3/OpenMV; footprint Connector_JST:JST_VH_B2P-VH-B_1x02_P3.96mm_Vertical -> 0.main.robot:JSTB4B-ZR
- J6: value LED -> Power IN; footprint 0.main.robot:JSTB6B-ZR -> Connector_JST:JST_VH_B2P-VH-B_1x02_P3.96mm_Vertical
- J7: value Kicker -> LED; footprint Connector_JST:JST_XH_B2B-XH-A_1x02_P2.50mm_Vertical -> 0.main.robot:JSTB6B-ZR
- J8: value MD1 -> Kicker; footprint Connector_JST:JST_XH_S2B-XH-A-1_1x02_P2.50mm_Horizontal -> Connector_JST:JST_XH_B2B-XH-A_1x02_P2.50mm_Vertical
- R11: value 47k -> 1k; footprint Resistor_SMD:R_0603_1608Metric_Pad0.98x0.95mm_HandSolder -> Resistor_THT:R_Axial_DIN0204_L3.6mm_D1.6mm_P5.08mm_Horizontal
- R13: value 10k -> 330; footprint Resistor_SMD:R_0603_1608Metric_Pad0.98x0.95mm_HandSolder -> Resistor_THT:R_Axial_DIN0204_L3.6mm_D1.6mm_P5.08mm_Horizontal
- R15, R19: value 10k -> 470
- R16, R21, R4: value 10k -> 47k
- R18: value 1k -> 470; footprint Resistor_THT:R_Axial_DIN0204_L3.6mm_D1.6mm_P5.08mm_Horizontal -> Resistor_SMD:R_0603_1608Metric_Pad0.98x0.95mm_HandSolder
- R2: value 470 -> 5.1kR
- R20: value 330 -> 47k; footprint Resistor_THT:R_Axial_DIN0204_L3.6mm_D1.6mm_P5.08mm_Horizontal -> Resistor_SMD:R_0603_1608Metric_Pad0.98x0.95mm_HandSolder
- R22, R37, R39: value 470 -> 47k
- R24: value 10k -> 120
- R3: value 5.1kR -> 10k
- R35, R40: value 47k -> 470
- R36, R41: value 47k -> 10k
- R42: value 470 -> 1k
- R43: value 10k -> 1k
- R44: value 47k -> 200R
- R45: value 47k -> 1R
- R46: value 47k -> 27.4R
- R47: value 470 -> 27.4R
- R48: value 10k -> 10kR
- R49: value 1k -> 1kR
- R6, R9: value 470 -> 10k
- SW2: value Reset -> GOAL; footprint 0.main.robot:THAU13-AB-R -> 0.main.robot:MFS101D-14-Z
- SW3: value GOAL -> START; footprint 0.main.robot:MFS101D-14-Z -> 0.main.robot:SW_NKK_B-12CCPRM
- SW4: value START -> AUX1; footprint 0.main.robot:SW_NKK_B-12CCPRM -> Button_Switch_THT:SW_DIP_SPSTx02_Slide_9.78x7.26mm_W7.62mm_P2.54mm
- SW5: value AUX1 -> IMU SET; footprint Button_Switch_THT:SW_DIP_SPSTx02_Slide_9.78x7.26mm_W7.62mm_P2.54mm -> 0.main.robot:TVAF06-A020B-R
- SW6: value IMU SET -> RESET
- SW7: value RESET -> BOOTSEL
- U1: value XBEE-S2C -> AZ1117CH-3.3; footprint 0.main.robot:XBEE-S2C -> Package_TO_SOT_SMD:SOT-223-3_TabPin2
- U10: value ATmega328P-AU -> W25Q128JVS; footprint Package_QFP:TQFP-32_7x7mm_P0.8mm -> rp2040:W25Q16-128JV-SOIC
- U2: value AZ1117CH-3.3 -> 74HC32; footprint Package_TO_SOT_SMD:SOT-223-3_TabPin2 -> 0.main.robot:SOP14W
- U3: value AZ1117CH-3.3 -> 74HC04; footprint Package_TO_SOT_SMD:SOT-223-3_TabPin2 -> 0.main.robot:SOP14W
- U4: value 74HC32 -> OKL-T_3-W12N-C; footprint 0.main.robot:SOP14W -> 0.main.robot:OKL-T3-W12N-C
- U5: value 74HC04 -> PCF8574PW; footprint 0.main.robot:SOP14W -> Package_SO:TSSOP-20_4.4x6.5mm_P0.65mm
- U6: value OKL-T_3-W12N-C -> AE-BNO055; footprint 0.main.robot:OKL-T3-W12N-C -> 0.main.robot:AE-BNO055
- U7: value PCF8574PW -> ATmega328P-AU; footprint Package_SO:TSSOP-20_4.4x6.5mm_P0.65mm -> Package_QFP:TQFP-32_7x7mm_P0.8mm
- U8: value AE-BNO055 -> ATmega328P-AU; footprint 0.main.robot:AE-BNO055 -> Package_QFP:TQFP-32_7x7mm_P0.8mm
- U9: value ATmega328P-AU -> RP2040; footprint Package_QFP:TQFP-32_7x7mm_P0.8mm -> rp2040:RP2040_hand
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Connections:
- C11 pad 1: +3.3VA -> Vcc1
- C12 pad 1: Net-(C12-Pad1) -> Vcc1
- C13 pad 1: Vcc1 -> RESET
- C14 pad 1: Vcc1 -> +1V1
- C15 pad 1: RESET -> +1V1
- C17 pad 1: +1V1 -> +3V3
- C18 pad 1: +1V1 -> +3V3
- C2 pad 1: Net-(C2-Pad1) -> +3V3
- C2 pad 2: Net-(C2-Pad2) -> GND
- C21 pad 1: +3V3 -> Net-(C21-Pad1)
- C23 pad 1: Net-(C23-Pad1) -> +3V3
- C3 pad 1: +5V -> GND
- C3 pad 2: Net-(C2-Pad2) -> /rp2040/RUN(RES)/30
- C4 pad 1: +3V3 -> +15V
- C5 pad 1: GND -> +5V
- C5 pad 2: /rp2040/RUN(RES)/30 -> Net-(C5-Pad2)
- C6 pad 1: +15V -> Vbatt
- C7 pad 1: +5V -> Net-(C7-Pad1)
- C7 pad 2: Net-(C7-Pad2) -> GND
- C8 pad 1: Vbatt -> Net-(C7-Pad1)
- C9 pad 1: Net-(C10-Pad1) -> +3.3VA
- D10 pad 1: Net-(D10-Pad1) -> +3.3VA
- D10 pad 2: Net-(D10-Pad2) -> +3V3
- D11 pad 1: Net-(D10-Pad1) -> GND
- D13 pad 2: +3V3 -> Net-(C10-Pad1)
- D15 pad 1: GND -> Vcc1
- D15 pad 2: Net-(D15-Pad2) -> RESET
- D16 pad 1: +3.3VA -> Vcc1
- D16 pad 2: Net-(C12-Pad1) -> Net-(D16-Pad2)
- D3 pad 1: GND -> +3V3
- D3 pad 2: Net-(D3-Pad2) -> /rp2040/RUN(RES)/30
- D5 pad 1: GND -> Net-(D5-Pad1)
- D6 pad 1: +3V3 -> Net-(D5-Pad1)
- D6 pad 2: /rp2040/RUN(RES)/30 -> Net-(D6-Pad2)
- D7 pad 1: GND -> Net-(D5-Pad1)
- D8 pad 1: Net-(D10-Pad1) -> Net-(D5-Pad1)
- D9 pad 1: Net-(D10-Pad1) -> GND
- J10 pad 1: +15V -> GND
- J10 pad 2: GND -> +15V
- J11 pad 1: /rp2040/GPIO05/07 -> +15V
- J11 pad 2: +3V3 -> GND
- J12 pad 1: /rp2040/GPIO03/05 -> /rp2040/GPIO05/07
- J12 pad 2: /rp2040/GPIO06/09 -> +3V3
- J12 pad 3: +3V3 -> /rp2040/GPIO04/06
- J12 pad 4: /rp2040/GPIO02/04 -> GND
- J13 pad 1: /rp2040/GPIO05/07 -> /rp2040/GPIO03/05
- J13 pad 2: +3V3 -> /rp2040/GPIO06/09
- J13 pad 3: /rp2040/GPIO04/06 -> +3V3
- J13 pad 4: GND -> /rp2040/GPIO02/04
- J14 pad 1: /rp2040/GPIO13/17 -> /rp2040/GPIO05/07
- J14 pad 2: GND -> +3V3
- J14 pad 3: /rp2040/GPIO12/16 -> /rp2040/GPIO04/06
- J15 pad 1: +15V -> /rp2040/GPIO13/17
- J15 pad 3: +15V -> /rp2040/GPIO12/16
- J16 pad 1: /rp2040/GPIO05/07 -> +15V
- J16 pad 2: +3V3 -> GND
- J16 pad 3: /rp2040/GPIO04/06 -> +15V
- J17 pad 1: Net-(J17-Pad1) -> /rp2040/GPIO05/07
- J17 pad 2: Net-(C7-Pad2) -> +3V3
- J18 pad 2: Net-(J18-Pad2) -> Net-(C5-Pad2)
- J19 pad 6: GND -> Net-(J19-Pad6)
- J20 pad 2: Net-(C10-Pad1) -> Net-(J20-Pad2)
- J20 pad 4: GND -> Net-(J20-Pad4)
- J21 pad 2: +3.3VA -> Net-(C7-Pad1)
- J21 pad 4: Net-(J21-Pad4) -> GND
- J22 pad 1: Net-(J21-Pad4) -> Net-(J22-Pad1)
- J22 pad 2: Net-(J21-Pad1) -> +3.3VA
- J22 pad 3: Net-(J21-Pad4) -> Net-(J22-Pad3)
- J22 pad 4: Net-(J21-Pad3) -> Net-(J22-Pad4)
- J23 pad 1: Net-(J23-Pad1) -> Net-(J22-Pad4)
- J23 pad 2: Net-(J23-Pad2) -> Net-(J22-Pad1)
- J23 pad 3: Net-(J23-Pad1) -> Net-(J22-Pad4)
- J23 pad 4: Net-(J23-Pad4) -> Net-(J22-Pad3)
- J26 pad 1: /LineTrimmer/SCL -> Net-(J26-Pad1)
- J26 pad 2: Vcc1 -> Net-(J26-Pad2)
- J26 pad 3: /LineTrimmer/SDA -> Net-(J26-Pad1)
- J26 pad 4: GND -> Net-(J26-Pad4)
- J27 pad 1: Net-(J27-Pad1) -> /LineTrimmer/SCL
- J27 pad 3: Net-(J27-Pad3) -> /LineTrimmer/SDA
- J27 pad 4: Net-(J27-Pad4) -> GND
- J28 pad 2: Net-(J28-Pad2) -> Vcc1
- J28 pad 5: Line5 -> RESET
- J28 pad 6: Net-(D19-Pad2) -> GND
- J4 pad 1: /rp2040/GPIO08/11 -> /rp2040/GPIO00/01
- J4 pad 3: Net-(J4-Pad3) -> /rp2040/GPIO01/02
- J5 pad 1: GND -> /rp2040/GPIO08/11
- J5 pad 2: +15V -> +5V
- J6 pad 1: /rp2040/GPIO26/31 -> GND
- J6 pad 2: unconnected-(J6-Pad2) -> +15V
- J7 pad 1: +15V -> /rp2040/GPIO26/31
- J7 pad 2: GND -> unconnected-(J7-Pad2)
- J8 pad 1: GND -> +15V
- J8 pad 2: +15V -> GND
- JP1 pad 2: Net-(J19-Pad5) -> Net-(J20-Pad5)
- JP3 pad 1: Net-(D10-Pad1) -> Net-(D5-Pad1)
- Q2 pad 3: Net-(J18-Pad4) -> Net-(J19-Pad4)
- R10 pad 1: /rp2040/GPIO09/12 -> Net-(R10-Pad1)
- R10 pad 2: Net-(J4-Pad3) -> Net-(J19-Pad6)
- R11 pad 1: +3V3 -> Net-(R11-Pad1)
- R11 pad 2: /rp2040/RUN(RES)/30 -> Net-(R11-Pad2)
- R12 pad 1: +3V3 -> Net-(R12-Pad1)
- R12 pad 2: /rp2040/GPIO05/07 -> Net-(J19-Pad3)
- R13 pad 1: +3V3 -> GND
- R13 pad 2: /rp2040/GPIO04/06 -> Net-(R11-Pad1)
- R14 pad 1: Net-(R14-Pad1) -> +5V
- R14 pad 2: Net-(J18-Pad1) -> Net-(Q1-Pad3)
- R15 pad 1: Net-(R15-Pad1) -> Net-(J18-Pad1)
- R15 pad 2: Net-(J18-Pad2) -> Net-(D4-Pad2)
- R16 pad 1: Net-(R16-Pad1) -> +15V
- R16 pad 2: Net-(J18-Pad5) -> Vbatt
- R17 pad 1: Net-(R17-Pad1) -> Vbatt
- R17 pad 2: Net-(J18-Pad6) -> GND
- R18 pad 1: Net-(R18-Pad1) -> Net-(J20-Pad2)
- R19 pad 1: Net-(R19-Pad1) -> Net-(J20-Pad5)
- R19 pad 2: Net-(J18-Pad3) -> Net-(R19-Pad2)
- R2 pad 1: Net-(R2-Pad1) -> Net-(J1-Pad5)
- R2 pad 2: Net-(D3-Pad2) -> GND
- R20 pad 1: GND -> Net-(C7-Pad1)
- R20 pad 2: Net-(R18-Pad1) -> Net-(R20-Pad2)
- R21 pad 1: +5V -> Net-(C7-Pad1)
- R21 pad 2: Net-(Q1-Pad3) -> Net-(R21-Pad2)
- R22 pad 1: Net-(J17-Pad1) -> Net-(C7-Pad1)
- R22 pad 2: Net-(D7-Pad2) -> Net-(R22-Pad2)
- R23 pad 1: +15V -> Net-(C7-Pad1)
- R23 pad 2: Vbatt -> Net-(R23-Pad2)
- R24 pad 1: Vbatt -> Net-(R24-Pad1)
- R24 pad 2: GND -> Net-(D5-Pad2)
- R3 pad 1: Net-(J1-Pad5) -> /rp2040/GPIO09/12
- R3 pad 2: GND -> Net-(J5-Pad3)
- R35 pad 1: Net-(C10-Pad1) -> Net-(R35-Pad1)
- R35 pad 2: Net-(J20-Pad3) -> Net-(D12-Pad2)
- R36 pad 2: Net-(J20-Pad1) -> +3.3VA
- R37 pad 1: Net-(C10-Pad1) -> Net-(R37-Pad1)
- R37 pad 2: Net-(D12-Pad2) -> Vcc1
- R38 pad 1: Net-(R38-Pad1) -> Vcc1
- R38 pad 2: +3.3VA -> /LineTrimmer/SCL
- R39 pad 1: +3.3VA -> Vcc1
- R39 pad 2: Net-(D14-Pad2) -> /LineTrimmer/SDA
- R4 pad 1: Net-(C2-Pad1) -> +3V3
- R4 pad 2: Net-(R4-Pad2) -> /rp2040/RUN(RES)/30
- R40 pad 1: +3.3VA -> Net-(R40-Pad1)
- R40 pad 2: /Sheet63625160/SCL_1 -> Net-(D14-Pad2)
- R41 pad 1: +3.3VA -> RESET
- R41 pad 2: /Sheet63625160/SDA_1 -> Vcc1
- R42 pad 1: Net-(R42-Pad1) -> /rp2040/RUN(RES)/30
- R42 pad 2: Net-(D15-Pad2) -> +3V3
- R43 pad 1: Net-(C12-Pad1) -> Net-(R43-Pad1)
- R43 pad 2: +3.3VA -> Net-(R43-Pad2)
- R44 pad 1: Net-(R44-Pad1) -> ADC_VREF
- R44 pad 2: Vcc1 -> +3V3
- R45 pad 1: Vcc1 -> Net-(C21-Pad1)
- R45 pad 2: /LineTrimmer/SCL -> ADC_VREF
- R46 pad 1: Vcc1 -> Net-(R46-Pad1)
- R46 pad 2: /LineTrimmer/SDA -> USB_DP
- R47 pad 2: Net-(D17-Pad2) -> USB_DM
- R48 pad 1: RESET -> QSPI_SS
- R48 pad 2: Vcc1 -> +3V3
- R49 pad 1: /rp2040/RUN(RES)/30 -> Net-(R49-Pad1)
- R49 pad 2: +3V3 -> QSPI_SS
- R5 pad 1: Net-(C2-Pad1) -> +3V3
- R5 pad 2: Net-(R5-Pad2) -> /rp2040/GPIO05/07
- R6 pad 1: Net-(R5-Pad2) -> +3V3
- R6 pad 2: Net-(D4-Pad2) -> /rp2040/GPIO04/06
- R7 pad 2: /rp2040/GPIO00/01 -> Net-(J19-Pad1)
- R8 pad 1: Net-(R5-Pad2) -> Net-(R8-Pad1)
- R8 pad 2: /rp2040/GPIO01/02 -> Net-(J19-Pad2)
- R9 pad 1: /rp2040/GPIO00/01 -> Net-(R9-Pad1)
- R9 pad 2: Net-(D5-Pad2) -> Net-(J19-Pad5)
- RV1 pad 1: Net-(D19-Pad2) -> Net-(D16-Pad2)
- RV1 pad 2: Net-(J28-Pad1) -> Net-(J29-Pad1)
- RV1 pad 3: Net-(J28-Pad1) -> Net-(J29-Pad1)
- RV2 pad 1: Net-(D19-Pad2) -> Net-(D16-Pad2)
- RV2 pad 2: Net-(J28-Pad2) -> Net-(J29-Pad2)
- RV2 pad 3: Net-(J28-Pad2) -> Net-(J29-Pad2)
- RV3 pad 1: Net-(D19-Pad2) -> Net-(D16-Pad2)
- RV3 pad 2: Net-(J28-Pad3) -> Net-(J29-Pad3)
- RV3 pad 3: Net-(J28-Pad3) -> Net-(J29-Pad3)
- RV4 pad 1: Net-(D19-Pad2) -> Net-(D16-Pad2)
- RV4 pad 2: Net-(J28-Pad4) -> Net-(J29-Pad4)
- RV4 pad 3: Net-(J28-Pad4) -> Net-(J29-Pad4)
- RV5 pad 1: Net-(D19-Pad2) -> Net-(D16-Pad2)
- SW1 pad 1: Net-(R4-Pad2) -> /rp2040/RUN(RES)/30
- SW2 pad 1: /rp2040/RUN(RES)/30 -> Net-(J20-Pad3)
- SW2 pad 2: GND -> Net-(J20-Pad1)
- SW3 pad 1: Net-(J19-Pad3) -> Net-(J20-Pad3)
- SW3 pad 2: Net-(J19-Pad1) -> Net-(J20-Pad4)
- SW4 pad 1: Net-(J19-Pad3) -> GND
- SW4 pad 2: Net-(J19-Pad4) -> GND
- SW4 pad 3: GND -> Net-(R20-Pad2)
- SW4 pad 4: Net-(R25-Pad2) -> Net-(R21-Pad2)
- SW5 pad 1: GND -> Net-(R22-Pad2)
- SW6 pad 1: Net-(R29-Pad2) -> GND
- SW6 pad 2: GND -> RESET
- SW7 pad 2: RESET -> Net-(R49-Pad1)
- U1 pad 1: Net-(C2-Pad1) -> GND
- U1 pad 2: Net-(R5-Pad2) -> +3V3
- U1 pad 3: Net-(R7-Pad1) -> Net-(C1-Pad1)
- U10 pad 1: unconnected-(U10-Pad1) -> QSPI_SS
- U10 pad 2: unconnected-(U10-Pad2) -> QSPI_SD1
- U10 pad 3: GND -> QSPI_SD2
- U10 pad 4: Vcc1 -> GND
- U10 pad 5: GND -> QSPI_SD0
- U10 pad 6: Vcc1 -> QSPI_CLK
- U10 pad 7: Net-(U10-Pad7) -> QSPI_SD3
- U10 pad 8: Net-(U10-Pad8) -> +3V3
- U2 pad 1: GND -> /rp2040/GPIO20/26
- U2 pad 2: Net-(C2-Pad1) -> Net-(U2-Pad11)
- U2 pad 3: +5V -> /rp2040/GPIO28/34
- U3 pad 1: GND -> Net-(R7-Pad1)
- U3 pad 2: +3V3 -> /rp2040/GPIO16/21
- U3 pad 3: Net-(C1-Pad1) -> Net-(R8-Pad1)
- U4 pad 1: /rp2040/GPIO20/26 -> GND
- U4 pad 10: /rp2040/GPIO19/25 -> unconnected-(U4-Pad10)
- U4 pad 11: Net-(U4-Pad11) -> unconnected-(U4-Pad11)
- U4 pad 12: Net-(U4-Pad12) -> unconnected-(U4-Pad12)
- U4 pad 2: Net-(U4-Pad11) -> +15V
- U4 pad 3: /rp2040/GPIO28/34 -> GND
- U4 pad 4: /rp2040/GPIO16/21 -> Net-(J18-Pad1)
- U4 pad 5: /rp2040/GPIO18/24 -> Net-(J18-Pad1)
- U4 pad 6: Net-(U4-Pad12) -> Net-(R11-Pad2)
- U4 pad 8: Net-(U4-Pad13) -> unconnected-(U4-Pad8)
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
Commit message: ToF
Parts:
- removed J28: ICSP, 0.main.robot:JSTB6B-ZR
- removed J29: Trimmer, 0.main.robot:JSTS6B-ZRLFSN
- J12: value I2C_0 -> SW1; footprint 0.main.robot:JSTB4B-ZR -> 0.main.robot:JSTB6B-ZR
- J13: value SW1 -> I2C_1; footprint 0.main.robot:JSTB6B-ZR -> 0.main.robot:JSTB4B-ZR
- J14: value I2C_1 -> drib-kick
- J16: value drib-kick -> I2C_2
- J17: value I2C_2 -> 5V OUT; footprint 0.main.robot:JSTB4B-ZR -> Connector_JST:JST_XH_B2B-XH-A_1x02_P2.50mm_Vertical
- J18: value 5V OUT -> LINE; footprint Connector_JST:JST_XH_B2B-XH-A_1x02_P2.50mm_Vertical -> 0.main.robot:JSTB8B-ZR
- J19: value LINE -> SW1; footprint 0.main.robot:JSTB8B-ZR -> 0.main.robot:JSTS6B-ZRLFSN
- J20: value SW1 -> ICSP; footprint 0.main.robot:JSTS6B-ZRLFSN -> 0.main.robot:JSTB6B-ZR
- J21: value I2C/IMU -> MD1
- J22: value ICSP -> MD2; footprint 0.main.robot:JSTB6B-ZR -> 0.main.robot:JSTB4B-ZR
- J23: value MD1 -> MD3
- J24: value MD2 -> MD4
- J25: value MD3 -> I2C/OLED
- J26: value MD4 -> ICSP; footprint 0.main.robot:JSTB4B-ZR -> 0.main.robot:JSTB6B-ZR
- J27: value I2C/OLED -> Trimmer; footprint 0.main.robot:JSTB4B-ZR -> 0.main.robot:JSTS6B-ZRLFSN
- moved J25 160.2 mm to (22.5, 99.5)
- moved J26 147.2 mm to (25.5, 84.6)
- moved R23 89.7 mm to (58.9, 62.9)
- moved R12 86.0 mm to (50.1, 67.4)
- moved D9 84.9 mm to (50.1, 64.9)
- moved J20 80.5 mm to (120.6, 21.7)
- moved R24 75.3 mm to (63.3, 60.4)
- moved SW1 74.3 mm to (52.3, 60.8)
- moved J18 67.9 mm to (18.1, 55.5)
- moved R2 65.7 mm to (66.1, 55.0)
- moved J16 65.6 mm to (44.5, 55.0)
- moved D8 63.2 mm to (59.0, 57.8)
- moved J13 62.4 mm to (53.6, 55.0)
- moved R29 58.4 mm to (81.0, 47.5)
- moved R30 58.2 mm to (63.3, 57.8)
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Connections:
- C7 pad 1: Net-(C7-Pad1) -> +3V3
- C8 pad 1: Net-(C7-Pad1) -> +3V3
- J12 pad 1: /rp2040/GPIO05/07 -> /rp2040/GPIO03/05
- J12 pad 2: +3V3 -> /rp2040/GPIO06/09
- J12 pad 3: /rp2040/GPIO04/06 -> +3V3
- J12 pad 4: GND -> /rp2040/GPIO02/04
- J13 pad 1: /rp2040/GPIO03/05 -> SCL_IMU
- J13 pad 2: /rp2040/GPIO06/09 -> +3V3
- J13 pad 3: +3V3 -> SDA_IMU
- J13 pad 4: /rp2040/GPIO02/04 -> GND
- J14 pad 1: /rp2040/GPIO05/07 -> /rp2040/GPIO13/17
- J14 pad 2: +3V3 -> GND
- J14 pad 3: /rp2040/GPIO04/06 -> /rp2040/GPIO12/16
- J15 pad 1: /rp2040/GPIO13/17 -> +15V
- J15 pad 3: /rp2040/GPIO12/16 -> +15V
- J16 pad 1: +15V -> SCL_IMU
- J16 pad 2: GND -> +3V3
- J16 pad 3: +15V -> SDA_IMU
- J17 pad 1: /rp2040/GPIO05/07 -> Net-(J17-Pad1)
- J17 pad 2: +3V3 -> Net-(C5-Pad2)
- J18 pad 2: Net-(C5-Pad2) -> Net-(J18-Pad2)
- J19 pad 6: Net-(J19-Pad6) -> GND
- J20 pad 2: Net-(J20-Pad2) -> +3.3VA
- J20 pad 5: Net-(J20-Pad5) -> Net-(C10-Pad1)
- J21 pad 1: Net-(J21-Pad1) -> Net-(J20-Pad4)
- J21 pad 2: Net-(C7-Pad1) -> Net-(J20-Pad1)
- J21 pad 3: Net-(J21-Pad3) -> Net-(J20-Pad4)
- J21 pad 4: GND -> Net-(J20-Pad3)
- J22 pad 2: +3.3VA -> Net-(J22-Pad2)
- J22 pad 3: Net-(J22-Pad3) -> Net-(J22-Pad1)
- J23 pad 1: Net-(J22-Pad4) -> Net-(J23-Pad1)
- J23 pad 2: Net-(J22-Pad1) -> Net-(J23-Pad2)
- J23 pad 3: Net-(J22-Pad4) -> Net-(J23-Pad1)
- J23 pad 4: Net-(J22-Pad3) -> Net-(J23-Pad4)
- J25 pad 1: Net-(J25-Pad1) -> /LineTrimmer/SCL
- J25 pad 2: Net-(J25-Pad2) -> Vcc1
- J25 pad 3: Net-(J25-Pad1) -> /LineTrimmer/SDA
- J25 pad 4: Net-(J25-Pad4) -> GND
- J26 pad 2: Net-(J26-Pad2) -> Vcc1
- J26 pad 3: Net-(J26-Pad1) -> Net-(J26-Pad3)
- J27 pad 1: /LineTrimmer/SCL -> Net-(J27-Pad1)
- J27 pad 2: Vcc1 -> Net-(J27-Pad2)
- J27 pad 3: /LineTrimmer/SDA -> Net-(J27-Pad3)
- J27 pad 4: GND -> Net-(J27-Pad4)
- JP1 pad 2: Net-(J20-Pad5) -> Net-(J19-Pad5)
- Q2 pad 3: Net-(J19-Pad4) -> Net-(J18-Pad4)
- R10 pad 2: Net-(J19-Pad6) -> Net-(J18-Pad6)
- R12 pad 2: Net-(J19-Pad3) -> Net-(J18-Pad3)
- R15 pad 1: Net-(J18-Pad1) -> Net-(J17-Pad1)
- R18 pad 1: Net-(J20-Pad2) -> Net-(J19-Pad2)
- R19 pad 1: Net-(J20-Pad5) -> Net-(J19-Pad5)
- R20 pad 1: Net-(C7-Pad1) -> +3V3
- R21 pad 1: Net-(C7-Pad1) -> +3V3
- R22 pad 1: Net-(C7-Pad1) -> +3V3
- R23 pad 1: Net-(C7-Pad1) -> +3V3
- R28 pad 1: Net-(C7-Pad1) -> +3V3
- R28 pad 2: Net-(J21-Pad3) -> SDA_IMU
- R29 pad 1: Net-(C7-Pad1) -> +3V3
- R29 pad 2: Net-(J21-Pad1) -> SCL_IMU
- R30 pad 1: Net-(C7-Pad1) -> +3V3
- R5 pad 2: /rp2040/GPIO05/07 -> SCL_IMU
- R6 pad 2: /rp2040/GPIO04/06 -> SDA_IMU
- R7 pad 2: Net-(J19-Pad1) -> Net-(J18-Pad1)
- R8 pad 2: Net-(J19-Pad2) -> Net-(J18-Pad2)
- R9 pad 2: Net-(J19-Pad5) -> Net-(J18-Pad5)
- RV1 pad 2: Net-(J29-Pad1) -> Net-(J27-Pad1)
- RV1 pad 3: Net-(J29-Pad1) -> Net-(J27-Pad1)
- RV2 pad 2: Net-(J29-Pad2) -> Net-(J27-Pad2)
- RV2 pad 3: Net-(J29-Pad2) -> Net-(J27-Pad2)
- RV3 pad 2: Net-(J29-Pad3) -> Net-(J27-Pad3)
- RV3 pad 3: Net-(J29-Pad3) -> Net-(J27-Pad3)
- RV4 pad 2: Net-(J29-Pad4) -> Net-(J27-Pad4)
- RV4 pad 3: Net-(J29-Pad4) -> Net-(J27-Pad4)
- SW2 pad 1: Net-(J20-Pad3) -> Net-(J19-Pad3)
- SW2 pad 2: Net-(J20-Pad1) -> Net-(J19-Pad1)
- SW3 pad 1: Net-(J20-Pad3) -> Net-(J19-Pad3)
- SW3 pad 2: Net-(J20-Pad4) -> Net-(J19-Pad4)
- SW3 pad 5: Net-(J20-Pad3) -> Net-(J19-Pad3)
- U4 pad 4: Net-(J18-Pad1) -> Net-(J17-Pad1)
- U4 pad 5: Net-(J18-Pad1) -> Net-(J17-Pad1)
- U5 pad 14: Net-(J20-Pad2) -> Net-(J19-Pad2)
- U5 pad 2: Net-(J21-Pad1) -> SCL_IMU
- U5 pad 4: Net-(J21-Pad3) -> SDA_IMU
- U5 pad 5: Net-(C7-Pad1) -> +3V3
- U6 pad 1: Net-(C7-Pad1) -> +3V3
- U6 pad 3: Net-(J21-Pad3) -> SDA_IMU
- U6 pad 4: Net-(J21-Pad1) -> SCL_IMU
- U7 pad 1: Net-(J24-Pad2) -> Net-(J22-Pad2)
- U7 pad 11: Net-(J25-Pad2) -> Net-(J23-Pad2)
- U7 pad 12: Net-(J25-Pad4) -> Net-(J23-Pad4)
- U7 pad 13: Net-(J25-Pad1) -> Net-(J23-Pad1)
- U7 pad 14: Net-(J26-Pad1) -> Net-(J24-Pad1)
- U7 pad 15: Net-(J22-Pad4) -> Net-(J20-Pad4)
- U7 pad 16: Net-(J22-Pad1) -> Net-(J20-Pad1)
- U7 pad 17: Net-(J22-Pad3) -> Net-(J20-Pad3)
- U7 pad 2: Net-(J24-Pad4) -> Net-(J22-Pad4)
- U7 pad 23: Net-(J26-Pad2) -> Net-(J24-Pad2)
- U7 pad 24: Net-(J26-Pad4) -> Net-(J24-Pad4)
- U7 pad 32: Net-(J24-Pad1) -> Net-(J22-Pad1)
- U8 pad 15: Net-(J28-Pad4) -> Net-(J26-Pad4)
- U8 pad 16: Net-(J28-Pad1) -> Net-(J26-Pad1)
- U8 pad 17: Net-(J28-Pad3) -> Net-(J26-Pad3)
- U8 pad 23: Net-(J29-Pad1) -> Net-(J27-Pad1)
- U8 pad 24: Net-(J29-Pad2) -> Net-(J27-Pad2)
- U8 pad 25: Net-(J29-Pad3) -> Net-(J27-Pad3)
- U8 pad 26: Net-(J29-Pad4) -> Net-(J27-Pad4)
- U9 pad 6: /rp2040/GPIO04/06 -> SDA_IMU
- U9 pad 7: /rp2040/GPIO05/07 -> SCL_IMU
