File: kicad/M1n-test/M1n-test.kicad_sch (KiCad schematic)
At the start: 1 part

Commit message: no message
Parts:
- added J1: Conn_01x01, M1n:SMTWE2025MTJ, symbol Connector_Generic:Conn_01x01
- added J3: I2C, symbol Connector_Generic:Conn_01x04
- added J4: Serial, symbol Connector_Generic:Conn_01x04
- added J5: USB, symbol Connector_Generic:Conn_01x04
- added R1, R2, R3, R4: 2k, Resistor_SMD:R_0603_1608Metric_Pad0.98x0.95mm_HandSolder, symbol Device:R
- added SW1: SW_SPDT, symbol Switch:SW_SPDT
- added SW2, SW3: SW_Push, symbol Switch:SW_Push
- J2: renamed from J?; footprint 121991190 -> M1n:121991190
Connections:
- net RST: now reaches J2.10
- net RST: now also SW2.1
- net +5V: now reaches J2.2
- net +5V: now also J2.4, J5.2 (Pin_2)
- net ISP_TX: now reaches J2.40
- net ISP_TX: now also J4.1 (Pin_1), J5.1 (Pin_1)
- net ISP_RX: now reaches J2.42
- net ISP_RX: now also SW1.2 (B)
- net BOOT: now reaches J2.53
- net BOOT: now also SW3.1
- net GND: now reaches J2.6
- net GND: now also J2.76 (MP1), J2.77 (MP2), J2.8, J3.4 (Pin_4), J4.4 (Pin_4), J5.4 (Pin_4), SW2.2, SW3.2
- net IO_10: now reaches J2.65
- net IO_10: now also R1.2
- net IO_11: now reaches J2.67
- net IO_11: now also R2.1
- net +3V3: now reaches J2.73
- net +3V3: now also J3.2 (Pin_2), J4.2 (Pin_2)
- new net: J4.3 (Pin_3), R3.2
- new net: J5.3 (Pin_3), R4.2
- new net: J3.3 (Pin_3), R2.2
- new net: J3.1 (Pin_1), R1.1
- new net: R3.1, SW1.3 (C)
- new net: R4.1, SW1.1 (A)
