File: kicad/vison-boad/vison-boad.kicad_sch (KiCad schematic)
At the start: 21 parts, among them J1 USB_C_Receptacle_USB2.0, J2 Wio Terminal, J3 UART, J4 to main, SW1 BTN_UP, SW2 BTN_UP, U1 RP2040_Stamp, U2 M1n-break, U3 M1n-break, U4 M1n-break, U5 M1n-break, U6 M1n-break

Commit message: no message
Parts:
- added D3: LED_PWR, 0.main.robot:LED_SMLE13WBC8W1, symbol Device:D_Small
- added D4: LED, 0.main.robot:LED_SMLE13WBC8W1, symbol Device:LED
- added J4: I2C_0, 0.main.robot:JSTB4B-ZR, symbol Connector_Generic:Conn_01x04
- added J5: pin_test, Connector_PinHeader_2.54mm:PinHeader_1x01_P2.54mm_Vertical, symbol Connector_Generic:Conn_01x01
- added R4: 1K, Resistor_SMD:R_0603_1608Metric_Pad0.98x0.95mm_HandSolder, symbol Device:R_Small
- added R7: 470, Resistor_SMD:R_0603_1608Metric_Pad0.98x0.95mm_HandSolder, symbol Device:R
- added SW3: M1n_RST, Button_Switch_SMD:Panasonic_EVQPUJ_EVQPUA, symbol Switch:SW_SPST
- R2, R3: footprint Resistor_SMD:R_0603_1608Metric -> Resistor_SMD:R_0603_1608Metric_Pad0.98x0.95mm_HandSolder
- SW1: value BTN_UP -> BOOTSET
- SW2: value BTN_UP -> RST
- renumbered J4 to J6, R4 to R5, R5 to R6, R6 to R8, R7 to R9, U3 to U2, U2 to U3, U5 to U4, U4 to U5
Connections:
- net +3.3V: now also D3.2 (A); no longer J2.1 (Pin_1), J6.4 (Pin_4), J6.5 (Pin_5), R8.2, R9.2
- net +5V: now also J2.2 (Pin_2), J2.4 (Pin_4), J6.4 (Pin_4), R8.2, R9.2, J4.2 (Pin_2)
- net GND: now also J6.5 (Pin_5), D4.1 (K), J4.4 (Pin_4), J5.1 (Pin_1), R4.2, SW3.1 (A)
- net SCL_0: now also J4.1 (Pin_1)
- net SDA_0: now also J4.3 (Pin_3)
- net at U1.26 (GPIO25): now also R7.2
- net M1n_RST: now reaches U2.13 (RST)
- net M1n_RST: now also U3.13 (RST), U4.13 (RST), U5.13 (RST), U6.13 (RST), SW3.2 (B)
- new net: D4.2 (A), R7.1
- new net: D3.1 (K), R4.1
Other:
- moved on the sheet: U2, U3, U4, U6

Commit message: no message
Parts:
- added J5: NEO PIXEL, 0.main.robot:JSTB4B-ZR, symbol Connector_Generic:Conn_01x04
- J4: renamed from J5; footprint Connector_PinHeader_2.54mm:PinHeader_1x01_P2.54mm_Vertical -> Connector_Pin:Pin_D0.7mm_L6.5mm_W1.8mm_FlatFork
- renumbered J4 to J7
Connections:
- net +3.3V: now also J3.2 (Pin_2), J7.2 (Pin_2), R8.2, R9.2, U1.34 (3.3V)
- net +5V: now also J5.2 (Pin_2); no longer J3.2 (Pin_2), J7.2 (Pin_2), R8.2, R9.2
- net GND: now also J5.4 (Pin_4)
- net NEO PIXEL: now reaches U1.22 (GPIO21)
- net NEO PIXEL: now also J5.3 (Pin_3)
- net SCL_0 renamed I2C_0.SCL
- net SCL_1 renamed I2C_1.SCL
- net SDA_0 renamed I2C_0.SDA
- net SDA_1 renamed I2C_1.SDA
- no-connect marks 2 -> 234
Other:
- moved on the sheet: J3, J7, R1, R6, R8, R9, SW1, SW2

Commit message: bus
Connections:
- net +3.3V: no longer D3.2 (A)
- net +5V: now also D3.2 (A)
- net USB_D+ renamed USB.D+
- net USB_D- renamed USB.D-
Other:
- moved on the sheet: D3, R4

Commit message: update
Connections:
- net +3.3V: now also D3.2 (A)
- net +5V: no longer D3.2 (A)
Other:
- moved on the sheet: D3, R4
Changed lines of the file:
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@@
     (stroke (width 0) (type default) (color 0 0 0 0))
   )
-  (wire (pts (xy 260.35 104.14) (xy 264.16 104.14))
+  (wire (pts (xy 102.87 52.07) (xy 106.68 52.07))
     (stroke (width 0) (type solid) (color 0 0 0 0))
   )
@@
     (stroke (width 0) (type default) (color 0 0 0 0))
   )
-  (wire (pts (xy 241.3 104.14) (xy 241.3 102.87))
+  (wire (pts (xy 83.82 52.07) (xy 83.82 50.8))
     (stroke (width 0) (type solid) (color 0 0 0 0))
   )
@@
     (stroke (width 0) (type default) (color 0 0 0 0))
   )
-  (wire (pts (xy 264.16 104.14) (xy 264.16 105.41))
+  (wire (pts (xy 106.68 52.07) (xy 106.68 53.34))
     (stroke (width 0) (type solid) (color 0 0 0 0))
   )
@@
     (stroke (width 0) (type default) (color 0 0 0 0))
   )
-  (wire (pts (xy 250.19 104.14) (xy 255.27 104.14))
+  (wire (pts (xy 92.71 52.07) (xy 97.79 52.07))
     (stroke (width 0) (type solid) (color 0 0 0 0))
   )
@@
     (stroke (width 0) (type default) (color 0 0 0 0))
   )
-  (wire (pts (xy 241.3 104.14) (xy 245.11 104.14))
+  (wire (pts (xy 83.82 52.07) (xy 87.63 52.07))
     (stroke (width 0) (type solid) (color 0 0 0 0))
   )
@@
     (pin "9")
   )
-  (symbol (lib_id "power:+5V") (at 241.3 102.87 0) (unit 1)
-    (in_bom yes) (on_board yes)
-    (property "Reference" "#PWR?" (id 0) (at 241.3 106.68 0)
-      (effects (font (size 1.27 1.27)) hide)
-    )
-    (property "Value" "+5V" (id 1) (at 241.3 102.87 0)
-      (effects (font (size 1.27 1.27)) (justify left))
-    )
-    (property "Footprint" "" (id 2) (at 241.3 102.87 0)
-      (effects (font (size 1.27 1.27)) hide)
-    )
-    (property "Datasheet" "" (id 3) (at 241.3 102.87 0)
-      (effects (font (size 1.27 1.27)) hide)
-    )
-    (pin "1")
-  )
   (symbol (lib_id "Device:R") (at 128.27 72.39 180) (unit 1)
     (in_bom yes) (on_board yes) (fields_autoplaced)
@@
     (pin "1")
   )
-  (symbol (lib_id "power:GND") (at 264.16 105.41 0) (unit 1)
+  (symbol (lib_id "power:+3.3V") (at 83.82 50.8 0) (unit 1)
+    (in_bom yes) (on_board yes) (fields_autoplaced)
+    (property "Reference" "#PWR0101" (id 0) (at 83.82 54.61 0)
+      (effects (font (size 1.27 1.27)) hide)
+    )
+    (property "Value" "+3.3V" (id 1) (at 83.82 47.2242 0))
+    (property "Footprint" "" (id 2) (at 83.82 50.8 0)
+      (effects (font (size 1.27 1.27)) hide)
+    )
+    (property "Datasheet" "" (id 3) (at 83.82 50.8 0)
+      (effects (font (size 1.27 1.27)) hide)
+    )
+    (pin "1")
+  )
+  (symbol (lib_id "power:GND") (at 106.68 53.34 0) (unit 1)
     (in_bom yes) (on_board yes)
-    (property "Reference" "#PWR017" (id 0) (at 264.16 111.76 0)
-      (effects (font (size 1.27 1.27)) hide)
-    )
-    (property "Value" "GND" (id 1) (at 264.16 109.22 0))
-    (property "Footprint" "" (id 2) (at 264.16 105.41 0))
-    (property "Datasheet" "" (id 3) (at 264.16 105.41 0))
+    (property "Reference" "#PWR017" (id 0) (at 106.68 59.69 0)
+      (effects (font (size 1.27 1.27)) hide)
+    )
+    (property "Value" "GND" (id 1) (at 106.68 57.15 0))
+    (property "Footprint" "" (id 2) (at 106.68 53.34 0))
+    (property "Datasheet" "" (id 3) (at 106.68 53.34 0))
     (pin "1")
   )
@@
     (pin "2")
   )
-  (symbol (lib_id "Device:D_Small") (at 247.65 104.14 0) (mirror y) (unit 1)
+  (symbol (lib_id "Device:D_Small") (at 90.17 52.07 0) (mirror y) (unit 1)
     (in_bom yes) (on_board yes)
-    (property "Reference" "D3" (id 0) (at 247.65 101.6 0))
-    (property "Value" "LED_PWR" (id 1) (at 247.65 106.68 0))
-    (property "Footprint" "0.main.robot:LED_SMLE13WBC8W1" (id 2) (at 247.65 104.14 90)
-      (effects (font (size 1.27 1.27)) hide)
-    )
-    (property "Datasheet" "~" (id 3) (at 247.65 104.14 90)
+    (property "Reference" "D3" (id 0) (at 90.17 49.53 0))
+    (property "Value" "LED_PWR" (id 1) (at 90.17 54.61 0))
+    (property "Footprint" "0.main.robot:LED_SMLE13WBC8W1" (id 2) (at 90.17 52.07 90)
+      (effects (font (size 1.27 1.27)) hide)
+    )
+    (property "Datasheet" "~" (id 3) (at 90.17 52.07 90)
       (effects (font (size 1.27 1.27)) hide)
     )
@@
     (pin "1")
   )
-  (symbol (lib_id "Device:R_Small") (at 257.81 104.14 90) (unit 1)
+  (symbol (lib_id "Device:R_Small") (at 100.33 52.07 90) (unit 1)
     (in_bom yes) (on_board yes)
-    (property "Reference" "R4" (id 0) (at 255.27 102.87 90)
+    (property "Reference" "R4" (id 0) (at 97.79 50.8 90)
       (effects (font (size 1.27 1.27)) (justify left))
     )
-    (property "Value" "1K" (id 1) (at 260.35 102.87 90)
+    (property "Value" "1K" (id 1) (at 102.87 50.8 90)
       (effects (font (size 1.27 1.27)) (justify right))
     )
-    (property "Footprint" "Resistor_SMD:R_0603_1608Metric_Pad0.98x0.95mm_HandSolder" (id 2) (at 257.81 104.14 0)
-      (effects (font (size 1.27 1.27)) hide)
-    )
-    (property "Datasheet" "~" (id 3) (at 257.81 104.14 0)
+    (property "Footprint" "Resistor_SMD:R_0603_1608Metric_Pad0.98x0.95mm_HandSolder" (id 2) (at 100.33 52.07 0)
+      (effects (font (size 1.27 1.27)) hide)
+    )
+    (property "Datasheet" "~" (id 3) (at 100.33 52.07 0)
       (effects (font (size 1.27 1.27)) hide)
     )
@@
       (reference "#PWR043") (unit 1) (value "+3.3V") (footprint "")
     )
-    (path "/4de8ff2c-5080-4d6a-ae63-3bad634e166b"
-      (reference "#PWR?") (unit 1) (value "+5V") (footprint "")
+    (path "/69511ecc-98a6-425a-880c-bb666c52f4db"
+      (reference "#PWR0101") (unit 1) (value "+3.3V") (footprint "")
     )
     (path "/31be8863-1987-4197-85f1-2ca80d5b7afb"

Commit message: fix: vison-boad
Parts:
- SW2: value RST -> RESET
Changed lines of the file:
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@@
     (in_bom yes) (on_board yes)
     (property "Reference" "SW2" (id 0) (at 129.54 102.87 0))
-    (property "Value" "RST" (id 1) (at 129.54 103.0224 0)
+    (property "Value" "RESET" (id 1) (at 129.54 103.0224 0)
       (effects (font (size 1.27 1.27)) hide)
     )
@@
     )
     (path "/432125bd-57fb-4d04-a3f3-c4c3c8c4d863"
-      (reference "SW2") (unit 1) (value "RST") (footprint "Button_Switch_SMD:Panasonic_EVQPUJ_EVQPUA")
+      (reference "SW2") (unit 1) (value "RESET") (footprint "Button_Switch_SMD:Panasonic_EVQPUJ_EVQPUA")
     )
     (path "/d36c93f4-34a2-4864-ad4d-c61de23a7361"
