File: kicad/power/power.kicad_pcb (KiCad board)
At the start: 2 copper layers, 5 parts, among them J1 Power IN, J2 Power OUT, SW1 SW_SPST

Commit message: power
Parts:
- added R1: 3k, Resistor_SMD:R_0603_1608Metric_Pad0.98x0.95mm_HandSolder, B.Cu at (109.5, 89.5)
- D1, F1, J1: moved to B.Cu
- J2: footprint Connector_JST:JST_VH_B2P-VH-B_1x02_P3.96mm_Vertical -> Connector_JST:JST_VH_B2PS-VH_1x02_P3.96mm_Horizontal; moved to B.Cu
- moved J2 37.2 mm to (106.5, 85.8)
- moved D1 32.4 mm to (107.5, 89.5), turned to 90 degrees
- moved SW1 24.0 mm to (120.0, 80.0)
- moved J1 14.4 mm to (135.0, 86.1), turned to 90 degrees
- moved F1 7.23 mm to (120.0, 96.5), turned to -90 degrees
Connections:
- net Net-(D1-Pad1) renamed GND
Routing:
- net GND: track 0.00 -> 36.7 mm
- net Net-(F1-Pad2): track 0.00 -> 29.3 mm
- net Net-(J1-Pad2): track 0.00 -> 15.5 mm
- net Net-(F1-Pad1): track 0.00 -> 15.2 mm
- net Net-(D1-Pad2): track 0.00 -> 2.02 mm
- net (no net): vias 0 -> 4
- added copper zone on B.Cu, net GND
- added copper zone on F.Cu, net GND
Other:
- board outline added: 40 x 30 mm

Commit message: no message
Parts:
- removed SW1: SW_SPST, 0.main.robot:SW_SPST_POWER
- added J2: OLED_in, 0.main.robot:JSTS4B-ZRLFSN, F.Cu at (115.0, 75.0)
- added J3: SW_Power, Connector_JST:JST_VH_B2PS-VH_1x02_P3.96mm_Horizontal, B.Cu at (113.0, 85.8)
- added J4: OLED_out, Connector_PinSocket_2.54mm:PinSocket_1x04_P2.54mm_Vertical, F.Cu at (118.8, 80.0)
- moved D1 8.50 mm to (99.0, 89.5)
- moved J5 8.50 mm to (98.0, 85.8)
- moved R1 8.50 mm to (101.0, 89.5)
- moved F1 5.00 mm to (115.0, 96.5)
- moved J1 2.50 mm to (135.0, 88.6)
- renumbered J2 to J5
Routing:
- net GND: track 36.7 -> 47.3 mm
- net Net-(J2-Pad4): track 0.00 -> 5.68 mm
- net Net-(J2-Pad1): track 0.00 -> 5.67 mm
- net Net-(J2-Pad3): track 0.00 -> 5.24 mm
- net Net-(J2-Pad2): track 0.00 -> 5.24 mm
- net Net-(F1-Pad2): track 29.3 -> 24.3 mm
- net Net-(J1-Pad2): track 15.5 -> 19.7 mm
- net Net-(F1-Pad1): track 15.2 -> 13.6 mm
Other:
- board size 40 x 30 mm -> 50 x 30 mm

Commit message: fix: power
Parts:
- removed J3: SW_Power, Connector_JST:JST_VH_B2PS-VH_1x02_P3.96mm_Horizontal
- removed J4: OLED_out, Connector_PinSocket_2.54mm:PinSocket_1x04_P2.54mm_Vertical
- removed J5: Power OUT, Connector_JST:JST_VH_B2PS-VH_1x02_P3.96mm_Horizontal
- added SW1: SW_SPST, 0.main.robot:SW_SPST_POWER, F.Cu at (100.0, 90.0)
- D1, J1, R1: moved to F.Cu
- F1: footprint 0.main.robot:FUSE_20mm -> 0.main.robot:FUSE_35222; moved to F.Cu
- J2: value OLED_in -> Power OUT; footprint 0.main.robot:JSTS4B-ZRLFSN -> Connector_PinHeader_2.54mm:PinHeader_2x05_P2.54mm_Vertical
- moved F1 20.0 mm to (110.0, 77.2), turned to 180 degrees
- moved J1 15.2 mm to (120.0, 86.4), turned to -90 degrees
- moved D1 11.9 mm to (110.0, 94.0)
- moved J2 11.3 mm to (115.1, 63.7), turned to -90 degrees
- moved R1 9.66 mm to (110.0, 86.0), turned to -90 degrees
Connections:
- J2 pad 1: Net-(J2-Pad1) -> GND
- J2 pad 2: Net-(J2-Pad2) -> Net-(F1-Pad1)
- J2 pad 3: Net-(J2-Pad3) -> GND
- J2 pad 4: Net-(J2-Pad4) -> Net-(F1-Pad1)
Routing:
- net GND: track 47.3 -> 0.00 mm
- net Net-(F1-Pad2): track 24.3 -> 0.00 mm
- net Net-(J1-Pad2): track 19.7 -> 0.00 mm
- net Net-(F1-Pad1): track 13.6 -> 0.00 mm
- net Net-(J2-Pad4): track 5.68 -> 0.00 mm
- net Net-(J2-Pad1): track 5.67 -> 0.00 mm
- net Net-(J2-Pad3): track 5.24 -> 0.00 mm
- net Net-(J2-Pad2): track 5.24 -> 0.00 mm
- net Net-(D1-Pad2): track 2.02 -> 0.00 mm
- net (no net): vias 4 -> 0
- removed copper zone on B.Cu, net GND
- removed copper zone on F.Cu, net GND
Other:
- board size 50 x 30 mm -> 51.7 x 40 mm

Commit message: Power基板できた
Routing:
- net GND: track 0.00 -> 50.4 mm, vias 0 -> 1
- net Net-(F1-Pad1): track 0.00 -> 36.5 mm
- net Net-(D1-Pad2): track 0.00 -> 29.7 mm
- net Net-(J1-Pad2): track 0.00 -> 21.5 mm
- net Net-(F1-Pad2): track 0.00 -> 8.86 mm
- added copper zone on B.Cu, net GND
Changed lines of the file:
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@@
   (gr_arc (start 100 62.239071) (mid 100.585786 60.824857) (end 102 60.239071) (layer "Edge.Cuts") (width 0.2))
   (target plus (at 85 105) (size 5) (width 0.1) (layer "Edge.Cuts"))
+  (segment (start 110 94.875) (end 110.375 95.25) (width 0.25) (layer "F.Cu") (net 1))
+  (segment (start 110.375 95.25) (end 112.395 95.25) (width 0.25) (layer "F.Cu") (net 1))
+  (via (at 112.395 95.25) (size 0.8) (drill 0.4) (layers "F.Cu" "B.Cu") (net 1))
+  (segment (start 120 86.4) (end 119.952528 86.352528) (width 2) (layer "B.Cu") (net 1))
+  (segment (start 119.952528 77.329083) (end 120.53 76.751611) (width 2) (layer "B.Cu") (net 1))
+  (segment (start 119.952528 86.352528) (end 119.952528 77.329083) (width 2) (layer "B.Cu") (net 1))
+  (segment (start 117.4295 70.817889) (end 117.4295 65.291098) (width 2) (layer "B.Cu") (net 1))
+  (segment (start 112.395 94.005) (end 120 86.4) (width 0.25) (layer "B.Cu") (net 1))
+  (segment (start 112.395 95.25) (end 112.395 94.005) (width 0.25) (layer "B.Cu") (net 1))
+  (segment (start 115.863402 63.725) (end 115.08 63.725) (width 2) (layer "B.Cu") (net 1))
+  (segment (start 117.4295 65.291098) (end 115.863402 63.725) (width 2) (layer "B.Cu") (net 1))
+  (segment (start 104.92 63.725) (end 115.08 63.725) (width 2) (layer "B.Cu") (net 1))
+  (segment (start 120.53 73.918389) (end 117.4295 70.817889) (width 2) (layer "B.Cu") (net 1))
+  (segment (start 120.53 76.751611) (end 120.53 73.918389) (width 2) (layer "B.Cu") (net 1))
+  (segment (start 99.08 93.125) (end 110 93.125) (width 0.25) (layer "F.Cu") (net 2))
+  (segment (start 99.0305 86.9125) (end 97.0995 88.8435) (width 0.25) (layer "F.Cu") (net 2))
+  (segment (start 97.0995 91.1445) (end 99.08 93.125) (width 0.25) (layer "F.Cu") (net 2))
+  (segment (start 97.0995 88.8435) (end 97.0995 91.1445) (width 0.25) (layer "F.Cu") (net 2))
+  (segment (start 110 86.9125) (end 99.0305 86.9125) (width 0.25) (layer "F.Cu") (net 2))
+  (segment (start 110.5607 84.5268) (end 110 85.0875) (width 0.9516) (layer "F.Cu") (net 3))
+  (segment (start 117.11 70.6453) (end 114.3803 70.6453) (width 2) (layer "F.Cu") (net 3))
+  (segment (start 107.46 66.265) (end 110 66.265) (width 2) (layer "F.Cu") (net 3))
+  (segment (start 117.11 75.335) (end 117.11 70.6453) (width 2) (layer "F.Cu") (net 3))
+  (segment (start 110 66.265) (end 112.54 66.265) (width 2) (layer "F.Cu") (net 3))
+  (segment (start 114.3803 70.6453) (end 110 66.265) (width 2) (layer "F.Cu") (net 3))
+  (segment (start 112.54 66.265) (end 115.08 66.265) (width 2) (layer "F.Cu") (net 3))
+  (segment (start 117.11 77.9775) (end 117.11 75.335) (width 2) (layer "F.Cu") (net 3))
+  (segment (start 110.5607 84.5268) (end 117.11 77.9775) (width 2) (layer "F.Cu") (net 3))
+  (segment (start 104.92 66.265) (end 107.46 66.265) (width 2) (layer "F.Cu") (net 3))
+  (segment (start 102.89 77.3477) (end 100 80.2377) (width 2) (layer "B.Cu") (net 4))
+  (segment (start 102.89 75.335) (end 102.89 77.3477) (width 2) (layer "B.Cu") (net 4))
+  (segment (start 100 83) (end 100 80.2377) (width 2) (layer "B.Cu") (net 4))
+  (segment (start 120 93.6) (end 115.3886 93.6) (width 2) (layer "F.Cu") (net 5))
+  (segment (start 115.3886 93.6) (end 111.7886 90) (width 2) (layer "F.Cu") (net 5))
+  (segment (start 111.7886 90) (end 100 90) (width 2) (layer "F.Cu") (net 5))
+  (zone (net 1) (net_name "GND") (layer "B.Cu") (hatch edge 0.508)
+    (connect_pads (clearance 0.508))
+    (min_thickness 0.254) (filled_areas_thickness no)
+    (fill yes (thermal_gap 0.508) (thermal_bridge_width 0.508))
+    (polygon
+      (pts
+        (xy 137.16 101.6)
+        (xy 83.82 101.6)
+        (xy 83.82 58.42)
+        (xy 137.16 58.42)
+      )
+    )
+  )
   (group "" (id 1413ff2a-3607-4a20-8e54-9442547fe19e)
     (members
