File: kicad/power/power.kicad_pcb (KiCad board)
At the start: 2 copper layers, 51.7 x 40 mm, 6 parts, among them J1 Power IN, J2 Power OUT, SW1 SW_SPST

Commit message: fix: main
Parts:
- added G***: LOGO, 0.main.robot:MMA_Logo, B.Cu at (110.0, 91.9)
Other:
- board text added: "Mar.2023 A.Saeki"
